File: lab/minifrank_rm1p2/amp.kicad_sch (KiCad schematic)
At the start: 20 parts, among them U9 LM358

Commit message: MiniFRANK RM1P2 1.01
Other:
- title: MiniFRANK RM1 -> MiniFRANK RM1P2
Changed lines of the file:
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@@
 	(paper "A4")
 	(title_block
-		(title "MiniFRANK RM1")
-		(date "2025-05-19")
+		(title "MiniFRANK RM1P2")
+		(date "2025-05-24")
 		(rev "${VERSION}")
 		(company "Mikhail Matveev")
