File: lab/nyx2/rp2350a.kicad_sch (KiCad schematic)
At the start: 33 parts, among them U1 RP2350, U2 ESP-PSRAM32, U3 W25Q128JVS, Y1 ASE-12MHz

Commit message: Nyx2 1.04
Parts:
- added J6: PSRAM CE Pin, FRANK:Jumper (solder, 3 pins), symbol Connector:Conn_01x03_Pin
Connections:
- net GPIO19: now also J6.3 (Pin_3)
- net GPIO8: now also J6.1 (Pin_1); no longer R7.1, U2.1 (~{CE})
- new net PSRAM_CE: J6.2 (Pin_2), R7.1, U2.1 (~{CE})
Changed lines of the file:
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@@
 	(title_block
 		(title "${NAME}")
-		(date "2025-05-07")
+		(date "2025-05-24")
 		(rev "${VERSION}")
 		(company "Mikhail Matveev")
@@
 	(wire
 		(pts
+			(xy 114.3 125.73) (xy 125.73 125.73)
+		)
+		(stroke
+			(width 0)
+			(type default)
+		)
+	)
+	(wire
+		(pts
 			(xy 265.43 21.59) (xy 265.43 20.32)
 		)
@@
 	(wire
 		(pts
+			(xy 114.3 128.27) (xy 125.73 128.27)
+		)
+		(stroke
+			(width 0)
+			(type default)
+		)
+	)
+	(wire
+		(pts
 			(xy 33.02 34.29) (xy 38.1 34.29)
 		)
@@
 	(wire
 		(pts
+			(xy 114.3 123.19) (xy 125.73 123.19)
+		)
+		(stroke
+			(width 0)
+			(type default)
+		)
+	)
+	(wire
+		(pts
 			(xy 130.81 49.53) (xy 138.43 49.53)
 		)
@@
 		)
 	)
-	(label "GPIO8"
-		(at 86.36 115.57 0)
+	(label "XIN"
+		(at 66.04 45.72 180)
 		(effects
 			(font
 				(size 1.27 1.27)
 			)
-			(justify left bottom)
+			(justify right bottom)
 		)
 	)
-	(label "XIN"
-		(at 66.04 45.72 180)
+	(label "QSPI_SCLK"
+		(at 137.16 97.79 0)
 		(effects
 			(font
 				(size 1.27 1.27)
 			)
-			(justify right bottom)
+			(justify left bottom)
 		)
 	)
-	(label "QSPI_SCLK"
-		(at 137.16 97.79 0)
+	(label "PSRAM_CE"
+		(at 86.36 115.57 0)
 		(effects
 			(font
@@
 		)
 	)
+	(label "GPIO19"
+		(at 125.73 128.27 180)
+		(effects
+			(font
+				(size 1.27 1.27)
+			)
+			(justify right bottom)
+		)
+	)
 	(label "QSPI_SD1"
 		(at 86.36 128.27 0)
@@
 		)
 	)
+	(label "GPIO8"
+		(at 125.73 123.19 180)
+		(effects
+			(font
+				(size 1.27 1.27)
+			)
+			(justify right bottom)
+		)
+	)
 	(label "QSPI_SD0"
 		(at 137.16 86.36 0)
@@
 		)
 	)
+	(label "PSRAM_CE"
+		(at 125.73 125.73 180)
+		(effects
+			(font
+				(size 1.27 1.27)
+			)
+			(justify right bottom)
+		)
+	)
 	(label "QSPI_SCLK"
 		(at 86.36 118.11 0)
@@
 					(unit 1)
 				)
+			)
+		)
+	)
+	(symbol
+		(lib_id "Connector:Conn_01x03_Pin")
+		(at 109.22 125.73 0)
+		(unit 1)
+		(exclude_from_sim no)
+		(in_bom yes)
+		(on_board yes)
+		(dnp no)
+		(fields_autoplaced yes)
+		(property "Reference" "J6"
+			(at 109.855 118.11 0)
+			(effects
+				(font
+					(size 1.27 1.27)
+				)
+			)
+		)
+		(property "Value" "PSRAM CE Pin"
+			(at 109.855 120.65 0)
+			(effects
+				(font
+					(size 1.27 1.27)
+				)
+			)
+		)
+		(property "Footprint" "FRANK:Jumper (solder, 3 pins)"
+			(at 109.22 125.73 0)
+			(effects
+				(font
+					(size 1.27 1.27)
+				)
+				(hide yes)
+			)
+		)
+		(property "Datasheet" "~"
+			(at 109.22 125.73 0)
+			(effects
+				(font
+					(size 1.27 1.27)
+				)
+				(hide yes)
+			)
+		)
+		(property "Description" "Generic connector, single row, 01x03, script generated"
+			(at 109.22 125.73 0)
+			(effects
+				(font
+					(size 1.27 1.27)
+				)
+				(hide yes)
+			)
+		)
+		(pin "3"
+		)
+		(pin "2"
+		)
+		(pin "1"
+		)
+		(instances
+			(project ""
+				(path "/8c0b3d8b-46d3-4173-ab1e-a61765f77d61/aade15f9-043c-45d2-91a1-54a1b11ea0a5"
+					(reference "J6")
+					(unit 1)
+				)
