File: hardware/turbofrank_rm1p2/turbofrank_rm1p2.kicad_pcb (KiCad board)
At the start: 4 copper layers, 99.5 x 99.5 mm, 247 parts, among them J1 PWR, J10 D-SUB 9 Male, J11 SS-52100-004, J12 DC3RX19JA2, J13 USB4215-03-A, J14 RCA-103, J15 D-SUB 9 Male, J16 D-SUB 15 Female, J17 Pin Header 1x08, J2 D-SUB 9 Male, J3 USB4215-03-A, J4 0475710001, J5 104031-0811, J6 PAM L, J7 PAM R, J8 PJ-320D, J9 PJ-320D, Q1 BC850, Q2 BC850, Q3 BC850, U1 USBLC6-2SC6, U10 MAX232CSE+, U11 SN74CBT3257CDR, U12 PAM8403D, U13 LM358, U14 TDA1387T, U15 JFC95101, U16 JFC95101, U17 74HC595, U18 74HC595, U19 74HC74, U2 74HC4052D, U3 NCP1117 3.3, U4 USBLC6-2SC6, U5 RP2350, U6 ESP-PSRAM32, U7 W25Q128JVS, U8 W25Q128JVSIQ, U9 RP2040, Y1 ASE-12MHz, Y2 12 MHz, Y3 3.58 Mhz

Commit message: Update turbofrank_rm1p2.kicad_pcb
Routing:
- net /GPIO17: track 67.9 -> 136.0 mm, vias 2 -> 3
Changed lines of the file:
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@@
+	)
+	(segment
+		(start 189.75 134)
+		(end 190.5 133.25)
+		(width 0.2)
+		(layer "F.Cu")
+		(net 23)
 	)
 	(segment
@@
 	)
 	(segment
+		(start 192.125 133.625)
+		(end 192.125 134.4725)
+		(width 0.2)
+		(layer "F.Cu")
+		(net 23)
+	)
+	(segment
+		(start 191.75 133.25)
+		(end 192.125 133.625)
+		(width 0.2)
+		(layer "F.Cu")
+		(net 23)
+	)
+	(segment
+		(start 192.125 134.4725)
+		(end 192 134.5975)
+		(width 0.2)
+		(layer "F.Cu")
+		(net 23)
+	)
+	(segment
 		(start 191.0125 79.4375)
 		(end 185.307888 79.4375)
@@
 		(start 185.307888 79.4375)
 		(end 182.898694 77.028306)
+		(width 0.2)
+		(layer "F.Cu")
+		(net 23)
+	)
+	(segment
+		(start 190.5 133.25)
+		(end 191.75 133.25)
 		(width 0.2)
 		(layer "F.Cu")
@@
 	)
 	(via
+		(at 192.125 133.625)
+		(size 0.6)
+		(drill 0.35)
+		(layers "F.Cu" "B.Cu")
+		(net 23)
+	)
+	(via
 		(at 133.679 82.805)
 		(size 0.6)
@@
 	)
 	(segment
+		(start 182.425 76.425)
+		(end 187.5 81.5)
+		(width 0.2)
+		(layer "B.Cu")
+		(net 23)
+	)
+	(segment
+		(start 191.966 119.261211)
+		(end 191.966 123.306388)
+		(width 0.2)
+		(layer "B.Cu")
+		(net 23)
+	)
+	(segment
+		(start 182.425 75.034)
+		(end 182.425 76.425)
+		(width 0.2)
+		(layer "B.Cu")
+		(net 23)
+	)
+	(segment
+		(start 193.477211 92)
+		(end 193.477211 117.75)
+		(width 0.2)
+		(layer "B.Cu")
+		(net 23)
+	)
+	(segment
 		(start 180.835 73.897)
 		(end 139.955 73.897)
@@
 	)
 	(segment
+		(start 191.966 123.306388)
+		(end 192.415 123.755388)
+		(width 0.2)
+		(layer "B.Cu")
+		(net 23)
+	)
+	(segment
 		(start 135.077 81.407)
 		(end 133.679 82.805)
@@
 	)
 	(segment
+		(start 192.415 133.335)
+		(end 192.125 133.625)
+		(width 0.2)
+		(layer "B.Cu")
+		(net 23)
+	)
+	(segment
+		(start 192.415 123.755388)
+		(end 192.415 133.335)
+		(width 0.2)
+		(layer "B.Cu")
+		(net 23)
+	)
+	(segment
+		(start 193.477211 117.75)
+		(end 191.966 119.261211)
+		(width 0.2)
+		(layer "B.Cu")
+		(net 23)
+	)
+	(segment
+		(start 192.125 133.625)
+		(end 192 133.75)
+		(width 0.2)
+		(layer "B.Cu")
+		(net 23)
+	)
+	(segment
 		(start 182.425 75.034)
 		(end 182.425 74.43)
 		(width 0.2)
 		(layer "B.Cu")
+		(net 23)
+	)
+	(segment
+		(start 187.5 86.022789)
+		(end 193.477211 92)
+		(width 0.2)
+		(layer "B.Cu")
+		(net 23)
+	)
+	(segment
+		(start 187.5 81.5)
+		(end 187.5 86.022789)
+		(width 0.2)
+		(layer "B.Cu")

Commit message: TF WIP
Parts:
- moved R76 84.0 mm to (143.2, 56.0)
- moved C58 83.1 mm to (143.2, 52.0), turned to -90 degrees
- moved R77 69.7 mm to (144.8, 76.5), turned to 0 degrees
- moved C56 68.4 mm to (144.8, 62.8)
- moved C55 68.3 mm to (148.5, 63.2)
- moved C59 67.5 mm to (144.0, 74.5), turned to 0 degrees
- moved R71 66.3 mm to (143.7, 59.8), turned to 180 degrees
- moved R75 65.5 mm to (147.8, 76.2)
- moved R69 64.7 mm to (153.6, 70.0), turned to 90 degrees
- moved R68 63.8 mm to (151.3, 61.0), turned to 0 degrees
- moved U13 63.3 mm to (149.1, 71.2)
- moved C53 63.1 mm to (145.0, 69.2), turned to 90 degrees
- moved R63 62.9 mm to (154.3, 61.0)
- moved R72 62.3 mm to (151.6, 66.2), turned to 0 degrees
- moved R67 62.0 mm to (153.0, 64.0), turned to 0 degrees
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Routing:
- net /GPIO17: track 136.0 -> 9.44 mm, vias 3 -> 1
- net /GPIO18: track 77.2 -> 8.01 mm, vias 2 -> 1
- net /RP2350A/~{USB_BOOT}: track 62.2 -> 0.00 mm, vias 4 -> 0
- net /GPIO16: track 65.2 -> 11.0 mm, vias 2 -> 1
- net VBUS: track 529.3 -> 582.6 mm, vias 51 -> 50
- net /GPIO19: track 59.1 -> 8.06 mm, vias 6 -> 0
- net /GPIO15: track 109.8 -> 150.0 mm
- net /GPIO9: track 118.3 -> 78.4 mm
- net /GPIO14: track 112.9 -> 148.7 mm
- net /GPIO27: track 48.3 -> 13.7 mm
- net Net-(R21-Pad1): track 6.56 -> 40.8 mm
- net /GPIO28: track 47.6 -> 18.5 mm
- net Net-(R20-Pad1): track 8.14 -> 36.9 mm
- net /GPIO26: track 43.2 -> 15.1 mm
- net /RP2_RUN: track 45.1 -> 19.0 mm
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
Commit message: TF WIP
Routing:
- net /GPIO17: track 9.44 -> 158.7 mm, vias 1 -> 3
- net /GPIO16: track 11.0 -> 156.0 mm, vias 1 -> 7
- net /TS_L: track 0.00 -> 126.5 mm, vias 0 -> 5
- net /GPIO19: track 8.06 -> 116.4 mm, vias 0 -> 7
- net /TS_R: track 0.00 -> 97.3 mm, vias 0 -> 2
- net /GPIO18: track 8.01 -> 92.8 mm, vias 1 -> 2
- net /GPIO26: track 15.1 -> 94.8 mm, vias 0 -> 5
- net /GPIO28: track 18.5 -> 92.1 mm, vias 0 -> 5
- net /Audio Out/TS/YM_BC1: track 0.00 -> 64.0 mm
- net /LOAD_IN: track 0.00 -> 60.3 mm, vias 0 -> 2
- net /RP2350A/~{USB_BOOT}: track 0.00 -> 59.2 mm, vias 0 -> 2
- net /Audio Out/TS/DA0: track 0.00 -> 57.2 mm
- net /AMP_IN_L: track 0.00 -> 55.9 mm, vias 0 -> 4
- net /GPIO27: track 13.7 -> 68.4 mm, vias 0 -> 4
- net /Audio Out/TS/YM_BDIR: track 0.00 -> 53.8 mm, vias 0 -> 3
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Other:
- outline, holes or cut-outs redrawn
