File: hardware/turbofrank_rm1p2/audio.kicad_sch (KiCad schematic)
At the start: 3 parts, among them J7 PAM L, J8 PAM R, J9 PJ-320D

Commit message: TF WIP
Parts:
- J6: renamed from J7; footprint FRANK:Connector Female ZH 1.50mm (2 pins) -> FRANK:Connector Female 1.25 JST 2P
- J7: renamed from J8; footprint FRANK:Connector Female ZH 1.50mm (2 pins) -> FRANK:Connector Female 1.25 JST 2P
- renumbered J9 to J8
Changed lines of the file:
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@@
 		(on_board yes)
 		(dnp no)
-		(property "Reference" "#PWR030"
+		(property "Reference" "#PWR029"
 			(at 175.26 119.38 0)
 			(effects
@@
 			(project "minifrank_rm1p2"
 				(path "/8c0b3d8b-46d3-4173-ab1e-a61765f77d61/765ae3f7-f5ac-49b6-99ac-a22ffc934361"
-					(reference "#PWR030")
+					(reference "#PWR029")
 					(unit 1)
 				)
@@
 		(on_board yes)
 		(dnp no)
-		(property "Reference" "J9"
+		(property "Reference" "J8"
 			(at 193.8019 100.1303 0)
 			(effects
@@
 			(project "minifrank_rm1p2"
 				(path "/8c0b3d8b-46d3-4173-ab1e-a61765f77d61/765ae3f7-f5ac-49b6-99ac-a22ffc934361"
-					(reference "J9")
+					(reference "J8")
 					(unit 1)
 				)
@@
 		(on_board yes)
 		(dnp no)
-		(property "Reference" "J8"
+		(property "Reference" "J7"
 			(at 170.815 69.85 0)
 			(effects
@@
 			)
 		)
-		(property "Footprint" "FRANK:Connector Female ZH 1.50mm (2 pins)"
+		(property "Footprint" "FRANK:Connector Female 1.25 JST 2P"
 			(at 170.18 74.93 0)
 			(effects
@@
 			(project "minifrank_rm1p2"
 				(path "/8c0b3d8b-46d3-4173-ab1e-a61765f77d61/765ae3f7-f5ac-49b6-99ac-a22ffc934361"
-					(reference "J8")
+					(reference "J7")
 					(unit 1)
 				)
@@
 		(on_board yes)
 		(dnp no)
-		(property "Reference" "J7"
+		(property "Reference" "J6"
 			(at 170.815 58.42 0)
 			(effects
@@
 			)
 		)
-		(property "Footprint" "FRANK:Connector Female ZH 1.50mm (2 pins)"
+		(property "Footprint" "FRANK:Connector Female 1.25 JST 2P"
 			(at 170.18 63.5 0)
 			(effects
@@
 			(project "minifrank_rm1p2"
 				(path "/8c0b3d8b-46d3-4173-ab1e-a61765f77d61/765ae3f7-f5ac-49b6-99ac-a22ffc934361"
-					(reference "J7")
-					(unit 1)
-				)
+					(reference "J6")
+					(unit 1)
+				)
