File: hardware/turbofrank_rm1p2/rp2350a.kicad_sch (KiCad schematic)
At the start: 31 parts, among them U5 RP2350, U6 ESP-PSRAM32, U7 W25Q128JVS, Y1 ASE-12MHz

Commit message: TF WIP
Parts:
- R25: value 33 -> 33R; footprint FRANK:Resistor (0805) -> FRANK:Resistor (0402)
- R26, R27, R31: footprint FRANK:Resistor (0805) -> FRANK:Resistor (0402)
Changed lines of the file:
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@@
 			)
 		)
-		(property "Value" "33"
+		(property "Value" "33R"
 			(at 128.143 47.752 0)
 			(effects
@@
 			)
 		)
-		(property "Footprint" "FRANK:Resistor (0805)"
+		(property "Footprint" "FRANK:Resistor (0402)"
 			(at 127 51.308 90)
 			(effects
@@
 		(on_board yes)
 		(dnp no)
-		(property "Reference" "#PWR079"
+		(property "Reference" "#PWR078"
 			(at 104.14 64.77 0)
 			(effects
@@
 			(project "frank_rm2-2350A"
 				(path "/8c0b3d8b-46d3-4173-ab1e-a61765f77d61/0b3076e2-1497-4f02-953d-15a48298b1c3"
-					(reference "#PWR079")
+					(reference "#PWR078")
 					(unit 1)
 				)
@@
 			)
 		)
-		(property "Footprint" "FRANK:Resistor (0805)"
+		(property "Footprint" "FRANK:Resistor (0402)"
 			(at 229.87 52.832 90)
 			(effects
@@
 		(on_board yes)
 		(dnp no)
-		(property "Reference" "#PWR074"
+		(property "Reference" "#PWR073"
 			(at 128.27 39.37 0)
 			(effects
@@
 			(project "frank_rm2-2350A"
 				(path "/8c0b3d8b-46d3-4173-ab1e-a61765f77d61/0b3076e2-1497-4f02-953d-15a48298b1c3"
-					(reference "#PWR074")
+					(reference "#PWR073")
 					(unit 1)
 				)
@@
 		(on_board yes)
 		(dnp no)
-		(property "Reference" "#PWR083"
+		(property "Reference" "#PWR082"
 			(at 41.91 132.08 0)
 			(effects
@@
 			(project "valera-2350A"
 				(path "/8c0b3d8b-46d3-4173-ab1e-a61765f77d61/0b3076e2-1497-4f02-953d-15a48298b1c3"
-					(reference "#PWR083")
+					(reference "#PWR082")
 					(unit 1)
 				)
@@
 		(on_board yes)
 		(dnp no)
-		(property "Reference" "#PWR075"
+		(property "Reference" "#PWR074"
 			(at 276.86 40.64 0)
 			(effects
@@
 			(project "frank_rm2-2350A"
 				(path "/8c0b3d8b-46d3-4173-ab1e-a61765f77d61/0b3076e2-1497-4f02-953d-15a48298b1c3"
-					(reference "#PWR075")
+					(reference "#PWR074")
 					(unit 1)
 				)
@@
 		(on_board yes)
 		(dnp no)
-		(property "Reference" "#PWR081"
+		(property "Reference" "#PWR080"
 			(at 111.76 101.6 0)
 			(effects
@@
 			(project "frank_rm2-2350A"
 				(path "/8c0b3d8b-46d3-4173-ab1e-a61765f77d61/0b3076e2-1497-4f02-953d-15a48298b1c3"
-					(reference "#PWR081")
+					(reference "#PWR080")
 					(unit 1)
 				)
@@
 		(on_board yes)
 		(dnp no)
-		(property "Reference" "#PWR086"
+		(property "Reference" "#PWR085"
 			(at 182.88 163.83 0)
 			(effects
@@
 			(project "frank_rm2-2350A"
 				(path "/8c0b3d8b-46d3-4173-ab1e-a61765f77d61/0b3076e2-1497-4f02-953d-15a48298b1c3"
-					(reference "#PWR086")
+					(reference "#PWR085")
 					(unit 1)
 				)
@@
 		(on_board yes)
 		(dnp no)
-		(property "Reference" "#PWR072"
+		(property "Reference" "#PWR071"
 			(at 199.39 22.86 0)
 			(effects
@@
 			(project "frank_rm2-2350A"
 				(path "/8c0b3d8b-46d3-4173-ab1e-a61765f77d61/0b3076e2-1497-4f02-953d-15a48298b1c3"
-					(reference "#PWR072")
+					(reference "#PWR071")
 					(unit 1)
 				)
@@
 			)
 		)
-		(property "Footprint" "FRANK:Resistor (0805)"
+		(property "Footprint" "FRANK:Resistor (0402)"
 			(at 229.87 61.722 90)
 			(effects
@@
 		(on_board yes)
 		(dnp no)
-		(property "Reference" "#PWR090"
+		(property "Reference" "#PWR089"
 			(at 77.47 194.31 0)
 			(effects
@@
 			(project "frank_rm2-2350A"
 				(path "/8c0b3d8b-46d3-4173-ab1e-a61765f77d61/0b3076e2-1497-4f02-953d-15a48298b1c3"
-					(reference "#PWR090")
+					(reference "#PWR089")
 					(unit 1)
 				)
@@
 		(on_board yes)
 		(dnp no)
-		(property "Reference" "#PWR073"
+		(property "Reference" "#PWR072"
 			(at 25.4 33.02 0)
 			(effects
@@
 			(project "frank_rm2-2350A"
 				(path "/8c0b3d8b-46d3-4173-ab1e-a61765f77d61/0b3076e2-1497-4f02-953d-15a48298b1c3"
-					(reference "#PWR073")
+					(reference "#PWR072")
 					(unit 1)
 				)
@@
 		(on_board yes)
 		(dnp no)
-		(property "Reference" "#PWR084"
+		(property "Reference" "#PWR083"
 			(at 62.23 142.24 0)
 			(effects
@@
 			(project "valera-2350A"
 				(path "/8c0b3d8b-46d3-4173-ab1e-a61765f77d61/0b3076e2-1497-4f02-953d-15a48298b1c3"
-					(reference "#PWR084")
+					(reference "#PWR083")
 					(unit 1)
 				)
@@
 		(on_board yes)
 		(dnp no)
-		(property "Reference" "#PWR071"
+		(property "Reference" "#PWR070"
 			(at 160.02 22.86 0)
 			(effects
@@
 			(project "frank_rm2-2350A"
 				(path "/8c0b3d8b-46d3-4173-ab1e-a61765f77d61/0b3076e2-1497-4f02-953d-15a48298b1c3"
-					(reference "#PWR071")
+					(reference "#PWR070")
 					(unit 1)
 				)
@@
 		(on_board yes)
 		(dnp no)
-		(property "Reference" "#PWR087"
+		(property "Reference" "#PWR086"
 			(at 83.82 166.37 0)
 			(effects
@@
 			(project "frank_rm2-2350A"
 				(path "/8c0b3d8b-46d3-4173-ab1e-a61765f77d61/0b3076e2-1497-4f02-953d-15a48298b1c3"
-					(reference "#PWR087")
+					(reference "#PWR086")
 					(unit 1)
 				)
@@
 		(dnp no)
 		(fields_autoplaced yes)
-		(property "Reference" "#PWR089"
+		(property "Reference" "#PWR088"
 			(at 149.86 182.88 0)
 			(effects
@@
 			(project "frank_rm2-2350A"
 				(path "/8c0b3d8b-46d3-4173-ab1e-a61765f77d61/0b3076e2-1497-4f02-953d-15a48298b1c3"
-					(reference "#PWR089")
+					(reference "#PWR088")
 					(unit 1)
 				)
@@
 		(dnp no)
 		(fields_autoplaced yes)
-		(property "Reference" "#PWR077"
+		(property "Reference" "#PWR076"
 			(at 25.4 63.5 0)
 			(effects
@@
 			(project ""
 				(path "/8c0b3d8b-46d3-4173-ab1e-a61765f77d61/0b3076e2-1497-4f02-953d-15a48298b1c3"
-					(reference "#PWR077")
+					(reference "#PWR076")
 					(unit 1)
 				)
@@
 		(on_board yes)
 		(dnp no)
-		(property "Reference" "#PWR076"
+		(property "Reference" "#PWR075"
 			(at 92.71 50.8 0)
 			(effects
@@
 			(project "frank_rm2-2350A"
 				(path "/8c0b3d8b-46d3-4173-ab1e-a61765f77d61/0b3076e2-1497-4f02-953d-15a48298b1c3"
-					(reference "#PWR076")
+					(reference "#PWR075")
 					(unit 1)
 				)
@@
 		(on_board yes)
 		(dnp no)
-		(property "Reference" "#PWR080"
+		(property "Reference" "#PWR079"
 			(at 92.71 83.82 0)
 			(effects
@@
 			(project "frank_rm2-2350A"
 				(path "/8c0b3d8b-46d3-4173-ab1e-a61765f77d61/0b3076e2-1497-4f02-953d-15a48298b1c3"
-					(reference "#PWR080")
+					(reference "#PWR079")
 					(unit 1)
 				)
@@
 		(dnp no)
 		(fields_autoplaced yes)
-		(property "Reference" "#PWR082"
+		(property "Reference" "#PWR081"
 			(at 73.66 101.6 0)
 			(effects
@@
 			(project "valera-2350A"
 				(path "/8c0b3d8b-46d3-4173-ab1e-a61765f77d61/0b3076e2-1497-4f02-953d-15a48298b1c3"
-					(reference "#PWR082")
+					(reference "#PWR081")
 					(unit 1)
 				)
@@
 		(on_board yes)
 		(dnp no)
-		(property "Reference" "#PWR078"
+		(property "Reference" "#PWR077"
 			(at 138.43 66.04 0)
 			(effects
@@
 			(project "frank_rm2-2350A"
 				(path "/8c0b3d8b-46d3-4173-ab1e-a61765f77d61/0b3076e2-1497-4f02-953d-15a48298b1c3"
-					(reference "#PWR078")
+					(reference "#PWR077")
 					(unit 1)
 				)
@@
 		(dnp no)
 		(fields_autoplaced yes)
-		(property "Reference" "#PWR088"
+		(property "Reference" "#PWR087"
 			(at 129.54 182.88 0)
 			(effects
@@
 			(project "frank_rm2-2350A"
 				(path "/8c0b3d8b-46d3-4173-ab1e-a61765f77d61/0b3076e2-1497-4f02-953d-15a48298b1c3"
-					(reference "#PWR088")
+					(reference "#PWR087")
 					(unit 1)
 				)
@@
 			)
 		)
-		(property "Footprint" "FRANK:Resistor (0805)"
+		(property "Footprint" "FRANK:Resistor (0402)"
 			(at 41.91 175.768 90)
 			(effects
@@
 		(on_board yes)
 		(dnp no)
-		(property "Reference" "#PWR085"
+		(property "Reference" "#PWR084"
 			(at 77.47 152.4 0)
 			(effects
@@
 			(project "frank_rm2-2350A"
 				(path "/8c0b3d8b-46d3-4173-ab1e-a61765f77d61/0b3076e2-1497-4f02-953d-15a48298b1c3"
-					(reference "#PWR085")
+					(reference "#PWR084")
 					(unit 1)
 				)

Commit message: TurboFRANK RM1P2 HW 1.00
Parts:
- S4: value TS-1233 -> Boot 2350
Changed lines of the file:
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@@
 	(title_block
 		(title "${NAME} ${MODEL}")
-		(date "2025-07-22")
+		(date "2025-07-25")
 		(rev "${VERSION}")
 		(company "Mikhail Matveev")
@@
 			)
 		)
-		(property "Value" "TS-1233"
+		(property "Value" "Boot 2350"
 			(at 113.03 91.4399 90)
 			(effects
