File: lab/frank_rm1p2/tda.kicad_sch (KiCad schematic)
At the start: 6 parts, among them U12 TDA1387T

Commit message: FRANK RM1P2 HW 1.01
Parts:
- renumbered R64 to R62, R65 to R63
Changed lines of the file:
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@@
 	(title_block
 		(title "${NAME} ${MODEL}")
-		(date "2025-08-12")
+		(date "${DATE}")
 		(rev "${VERSION}")
 		(company "Mikhail Matveev")
@@
 		(dnp no)
 		(fields_autoplaced yes)
-		(property "Reference" "#PWR0132"
+		(property "Reference" "#PWR0130"
 			(at 166.37 82.55 0)
 			(effects
@@
 			(project "minifrank_rm1p2"
 				(path "/8c0b3d8b-46d3-4173-ab1e-a61765f77d61/765ae3f7-f5ac-49b6-99ac-a22ffc934361/0dccd710-fd54-4e53-9f08-059759dd7a75"
-					(reference "#PWR0132")
+					(reference "#PWR0130")
 					(unit 1)
 				)
@@
 		(on_board yes)
 		(dnp no)
-		(property "Reference" "R65"
+		(property "Reference" "R63"
 			(at 184.15 97.79 90)
 			(effects
@@
 			)
 		)
-		(property "Datasheet" "https://www.vishay.com/docs/28952/mcs0402at-mct0603at-mcu0805at-mca1206at.pdf"
+		(property "Datasheet" "~"
 			(at 186.69 97.79 0)
 			(effects
@@
 			(project "minifrank_rm1p2"
 				(path "/8c0b3d8b-46d3-4173-ab1e-a61765f77d61/765ae3f7-f5ac-49b6-99ac-a22ffc934361/0dccd710-fd54-4e53-9f08-059759dd7a75"
-					(reference "R65")
+					(reference "R63")
 					(unit 1)
 				)
@@
 		(dnp no)
 		(fields_autoplaced yes)
-		(property "Reference" "#PWR0134"
+		(property "Reference" "#PWR0132"
 			(at 186.69 109.22 0)
 			(effects
@@
 			(project "minifrank_rm1p2"
 				(path "/8c0b3d8b-46d3-4173-ab1e-a61765f77d61/765ae3f7-f5ac-49b6-99ac-a22ffc934361/0dccd710-fd54-4e53-9f08-059759dd7a75"
-					(reference "#PWR0134")
+					(reference "#PWR0132")
 					(unit 1)
 				)
@@
 		(dnp no)
 		(fields_autoplaced yes)
-		(property "Reference" "#PWR0131"
+		(property "Reference" "#PWR0129"
 			(at 186.69 68.58 0)
 			(effects
@@
 			(project "minifrank_rm1p2"
 				(path "/8c0b3d8b-46d3-4173-ab1e-a61765f77d61/765ae3f7-f5ac-49b6-99ac-a22ffc934361/0dccd710-fd54-4e53-9f08-059759dd7a75"
-					(reference "#PWR0131")
+					(reference "#PWR0129")
 					(unit 1)
 				)
@@
 	)
 	(symbol
+		(lib_name "R_Small_1")
 		(lib_id "Device:R_Small")
 		(at 186.69 80.01 180)
@@
 		(on_board yes)
 		(dnp no)
-		(property "Reference" "R64"
+		(property "Reference" "R62"
 			(at 184.15 80.01 90)
 			(effects
@@
 			)
 		)
-		(property "Datasheet" "https://www.vishay.com/docs/28952/mcs0402at-mct0603at-mcu0805at-mca1206at.pdf"
+		(property "Datasheet" "~"
 			(at 186.69 80.01 0)
 			(effects
@@
 			(project "minifrank_rm1p2"
 				(path "/8c0b3d8b-46d3-4173-ab1e-a61765f77d61/765ae3f7-f5ac-49b6-99ac-a22ffc934361/0dccd710-fd54-4e53-9f08-059759dd7a75"
-					(reference "R64")
+					(reference "R62")
 					(unit 1)
 				)
@@
 		(dnp no)
 		(fields_autoplaced yes)
-		(property "Reference" "#PWR0133"
+		(property "Reference" "#PWR0131"
 			(at 116.84 109.22 0)
 			(effects
@@
 			(project "minifrank_rm1p2"
 				(path "/8c0b3d8b-46d3-4173-ab1e-a61765f77d61/765ae3f7-f5ac-49b6-99ac-a22ffc934361/0dccd710-fd54-4e53-9f08-059759dd7a75"
-					(reference "#PWR0133")
+					(reference "#PWR0131")
 					(unit 1)
 				)
@@
 		(dnp no)
 		(fields_autoplaced yes)
-		(property "Reference" "#PWR0136"
+		(property "Reference" "#PWR0134"
 			(at 166.37 121.92 0)
 			(effects
@@
 			(project "minifrank_rm1p2"
 				(path "/8c0b3d8b-46d3-4173-ab1e-a61765f77d61/765ae3f7-f5ac-49b6-99ac-a22ffc934361/0dccd710-fd54-4e53-9f08-059759dd7a75"
-					(reference "#PWR0136")
+					(reference "#PWR0134")
 					(unit 1)
 				)
@@
 		(dnp no)
 		(fields_autoplaced yes)
-		(property "Reference" "#PWR0135"
+		(property "Reference" "#PWR0133"
 			(at 157.48 121.92 0)
 			(effects
@@
 			(project "minifrank_rm1p2"
 				(path "/8c0b3d8b-46d3-4173-ab1e-a61765f77d61/765ae3f7-f5ac-49b6-99ac-a22ffc934361/0dccd710-fd54-4e53-9f08-059759dd7a75"
-					(reference "#PWR0135")
+					(reference "#PWR0133")
 					(unit 1)
 				)
@@
 		(dnp no)
 		(fields_autoplaced yes)
-		(property "Reference" "#PWR0137"
+		(property "Reference" "#PWR0135"
 			(at 176.53 121.92 0)
 			(effects
@@
 			(project "minifrank_rm1p2"
 				(path "/8c0b3d8b-46d3-4173-ab1e-a61765f77d61/765ae3f7-f5ac-49b6-99ac-a22ffc934361/0dccd710-fd54-4e53-9f08-059759dd7a75"
-					(reference "#PWR0137")
+					(reference "#PWR0135")
 					(unit 1)
 				)
