File: lab/minifrank_rm1p2h/power.kicad_sch (KiCad schematic)
At the start: 13 parts, among them J4 USB4215-03-A, U1 NCP1117 3.3, U2 USBLC6-2SC6

Commit message: MiniFRANK RM1P2H HW 1.0
Parts:
- R7: AliExpress https://www.vishay.com/docs/28952/mcs0402at-mct0603at-mcu08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 -> https://www.aliexpress.com/item/1005005945735199.html
- S2: AliExpress (none) -> https://www.aliexpress.com/item/4000685483225.html
- U2: AliExpress (none) -> https://www.aliexpress.com/item/1005006883533480.html
Changed lines of the file:
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@@
 	(title_block
 		(title "${NAME} ${MODEL}")
-		(date "2025-07-30")
+		(date "2025-08-01")
 		(rev "${VERSION}")
 		(company "Mikhail Matveev")
@@
 			)
 		)
+		(property "AliExpress" "https://www.aliexpress.com/item/1005006883533480.html"
+			(at 148.59 90.17 0)
+			(effects
+				(font
+					(size 1.27 1.27)
+				)
+				(hide yes)
+			)
+		)
 		(pin "2"
 		)
@@
 			)
 		)
-		(property "AliExpress" "https://www.vishay.com/docs/28952/mcs0402at-mct0603at-mcu0805at-mca1206at.pdf"
+		(property "AliExpress" "https://www.aliexpress.com/item/1005005945735199.html"
 			(at 193.04 119.38 0)
 			(effects
@@
 			(at 143.51 76.2 0)
 			(effects
+				(font
+					(size 1.27 1.27)
+				)
+				(hide yes)
+			)
+		)
+		(property "AliExpress" "https://www.aliexpress.com/item/4000685483225.html"
+			(at 143.51 76.2 0)
+			(effects
