File: hardware/turbofrank/turbofrank.kicad_pcb (KiCad board)
At the start: 2 copper layers, 99 x 99 mm, 219 parts, among them J1 UART, J10 PAM L, J11 PAM R, J12 PJ-320D, J13 PJ-320D, J14 Rasberry Pi Pico, J15 RP2040-Zero, J16 SS-52100-004, J17 D-SUB 15 Female, J18 Pin Header 1x08, J19 RCA-103, J2 PWR, J20 D-SUB 9 Male, J21 USB HUB Data, J3 USB4215, J4 MDC-036, J5 0475710001, J6 104031-0811, J7 D-SUB 9 Male, J8 D-SUB 9 Male, J9 DC3RX19JA2, Q1 BC850, Q2 BC850, Q3 BC850, U1 NCP1117 3.3, U10 PAM8403D, U11 LM358, U12 TDA1387T, U2 ESP-PSRAM32, U3 MAX232CSE+, U4 JFC95101, U5 JFC95101, U6 74HC595, U7 74HC595, U8 74HC74, U9 MW7211A, X1 3.58 MHz

Commit message: PCB updated
Parts:
- turned JP2 to 180 degrees
Routing:
- net /GPIO27: track 245.9 -> 225.8 mm
- net /GPIO0: track 116.6 -> 105.3 mm, vias 3 -> 1
- net /USB Hub/DM_IN: track 87.6 -> 78.2 mm
- net Net-(C34-Pad1): track 159.2 -> 150.1 mm, vias 4 -> 6
- net /USB Hub/DP_IN: track 91.1 -> 82.8 mm
- net /GPIO1: track 105.2 -> 100.0 mm
- net /GPIO12: track 59.3 -> 54.6 mm
- net Net-(C28-Pad2): track 100.6 -> 96.2 mm
- net /Composite/CVBS: track 17.3 -> 13.1 mm
- net VBUS: track 775.3 -> 771.9 mm
- net /GPIO21: track 119.6 -> 116.8 mm
- net /TS_L: track 111.4 -> 108.7 mm
- net /GPIO5: track 45.3 -> 42.6 mm
- net /Audio Out/TS/A1: track 9.18 -> 6.73 mm
- net /GPIO11: track 30.9 -> 28.7 mm
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