File: lab/frank_one/ps2.kicad_sch (KiCad schematic)
At the start: 14 parts, among them J4 MDC-036

Commit message: FRANK Fastbeta PWT, One WIP
Parts:
- C27: renamed from C3; footprint FRANK:Capacitor (0805) -> FRANK:Capacitor (0603)
- R32: renamed from R10; footprint FRANK:Resistor (0805) -> FRANK:Resistor (0603)
- R33: renamed from R13; footprint FRANK:Resistor (0805) -> FRANK:Resistor (0603)
- R34: renamed from R12; footprint FRANK:Resistor (0805) -> FRANK:Resistor (0603)
- R35: renamed from R15; footprint FRANK:Resistor (0805) -> FRANK:Resistor (0603)
- R36: renamed from R9; footprint FRANK:Resistor (0805) -> FRANK:Resistor (0603)
- R37: renamed from R14; footprint FRANK:Resistor (0805) -> FRANK:Resistor (0603)
- R38: renamed from R11; footprint FRANK:Resistor (0805) -> FRANK:Resistor (0603)
- R39: renamed from R16; footprint FRANK:Resistor (0805) -> FRANK:Resistor (0603)
- renumbered D2 to D4, D3 to D5, D1 to D6, D4 to D7, J4 to J13
Changed lines of the file:
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@@
 		(on_board yes)
 		(dnp no)
-		(property "Reference" "R10"
+		(property "Reference" "R32"
 			(at 151.13 74.93 90)
 			(effects
@@
 			)
 		)
-		(property "Footprint" "FRANK:Resistor (0805)"
+		(property "Footprint" "FRANK:Resistor (0603)"
 			(at 155.448 74.93 90)
 			(effects
@@
 			(project "frank_m2"
 				(path "/8c0b3d8b-46d3-4173-ab1e-a61765f77d61/0d431c2a-21fb-40ea-8f7b-9d17d283876a"
-					(reference "R10")
+					(reference "R32")
 					(unit 1)
 				)
@@
 		(on_board yes)
 		(dnp no)
-		(property "Reference" "C3"
+		(property "Reference" "C27"
 			(at 64.516 97.028 0)
 			(effects
@@
 			)
 		)
-		(property "Footprint" "FRANK:Capacitor (0805)"
+		(property "Footprint" "FRANK:Capacitor (0603)"
 			(at 70.8152 101.6 0)
 			(effects
@@
 			(project "frank_m2"
 				(path "/8c0b3d8b-46d3-4173-ab1e-a61765f77d61/0d431c2a-21fb-40ea-8f7b-9d17d283876a"
-					(reference "C3")
+					(reference "C27")
 					(unit 1)
 				)
@@
 		(on_board yes)
 		(dnp no)
-		(property "Reference" "#PWR025"
+		(property "Reference" "#PWR0106"
 			(at 209.55 73.66 0)
 			(effects
@@
 			(project "frank_m2"
 				(path "/8c0b3d8b-46d3-4173-ab1e-a61765f77d61/0d431c2a-21fb-40ea-8f7b-9d17d283876a"
-					(reference "#PWR025")
+					(reference "#PWR0106")
 					(unit 1)
 				)
@@
 		(on_board yes)
 		(dnp no)
-		(property "Reference" "R11"
+		(property "Reference" "R38"
 			(at 217.17 80.264 90)
 			(effects
@@
 			)
 		)
-		(property "Footprint" "FRANK:Resistor (0805)"
+		(property "Footprint" "FRANK:Resistor (0603)"
 			(at 217.17 84.328 90)
 			(effects
@@
 			(project "frank_m2"
 				(path "/8c0b3d8b-46d3-4173-ab1e-a61765f77d61/0d431c2a-21fb-40ea-8f7b-9d17d283876a"
-					(reference "R11")
+					(reference "R38")
 					(unit 1)
 				)
@@
 		(dnp no)
 		(fields_autoplaced yes)
-		(property "Reference" "J4"
+		(property "Reference" "J13"
 			(at 97.8077 82.55 0)
 			(effects
@@
 			(project "frank_m2"
 				(path "/8c0b3d8b-46d3-4173-ab1e-a61765f77d61/0d431c2a-21fb-40ea-8f7b-9d17d283876a"
-					(reference "J4")
+					(reference "J13")
 					(unit 1)
 				)
@@
 		(on_board yes)
 		(dnp no)
-		(property "Reference" "R13"
+		(property "Reference" "R33"
 			(at 151.13 102.87 90)
 			(effects
@@
 			)
 		)
-		(property "Footprint" "FRANK:Resistor (0805)"
+		(property "Footprint" "FRANK:Resistor (0603)"
 			(at 155.448 102.87 90)
 			(effects
@@
 			(project "frank_m2"
 				(path "/8c0b3d8b-46d3-4173-ab1e-a61765f77d61/0d431c2a-21fb-40ea-8f7b-9d17d283876a"
-					(reference "R13")
+					(reference "R33")
 					(unit 1)
 				)
@@
 		(on_board yes)
 		(dnp no)
-		(property "Reference" "D1"
+		(property "Reference" "D6"
 			(at 227.33 74.93 0)
 			(effects
@@
 			(project "frank_m2"
 				(path "/8c0b3d8b-46d3-4173-ab1e-a61765f77d61/0d431c2a-21fb-40ea-8f7b-9d17d283876a"
-					(reference "D1")
+					(reference "D6")
 					(unit 1)
 				)
@@
 		(on_board yes)
 		(dnp no)
-		(property "Reference" "D4"
+		(property "Reference" "D7"
 			(at 227.33 104.14 0)
 			(effects
@@
 			(project "frank_m2"
 				(path "/8c0b3d8b-46d3-4173-ab1e-a61765f77d61/0d431c2a-21fb-40ea-8f7b-9d17d283876a"
-					(reference "D4")
+					(reference "D7")
 					(unit 1)
 				)
@@
 		(on_board yes)
 		(dnp no)
-		(property "Reference" "R14"
+		(property "Reference" "R37"
 			(at 207.01 102.87 90)
 			(effects
@@
 			)
 		)
-		(property "Footprint" "FRANK:Resistor (0805)"
+		(property "Footprint" "FRANK:Resistor (0603)"
 			(at 211.328 102.87 90)
 			(effects
@@
 			(project "frank_m2"
 				(path "/8c0b3d8b-46d3-4173-ab1e-a61765f77d61/0d431c2a-21fb-40ea-8f7b-9d17d283876a"
-					(reference "R14")
+					(reference "R37")
 					(unit 1)
 				)
@@
 		(on_board yes)
 		(dnp no)
-		(property "Reference" "R15"
+		(property "Reference" "R35"
 			(at 161.29 109.474 90)
 			(effects
@@
 			)
 		)
-		(property "Footprint" "FRANK:Resistor (0805)"
+		(property "Footprint" "FRANK:Resistor (0603)"
 			(at 161.29 113.538 90)
 			(effects
@@
 			(project "frank_m2"
 				(path "/8c0b3d8b-46d3-4173-ab1e-a61765f77d61/0d431c2a-21fb-40ea-8f7b-9d17d283876a"
-					(reference "R15")
+					(reference "R35")
 					(unit 1)
 				)
@@
 		(dnp no)
 		(fields_autoplaced yes)
-		(property "Reference" "#PWR027"
+		(property "Reference" "#PWR0108"
 			(at 224.79 64.77 0)
 			(effects
@@
 			(project "frank_m2"
 				(path "/8c0b3d8b-46d3-4173-ab1e-a61765f77d61/0d431c2a-21fb-40ea-8f7b-9d17d283876a"
-					(reference "#PWR027")
+					(reference "#PWR0108")
 					(unit 1)
 				)
@@
 		(on_board yes)
 		(dnp no)
-		(property "Reference" "#PWR030"
+		(property "Reference" "#PWR0101"
 			(at 127 92.71 0)
 			(effects
@@
 			(project "frank_m2"
 				(path "/8c0b3d8b-46d3-4173-ab1e-a61765f77d61/0d431c2a-21fb-40ea-8f7b-9d17d283876a"
-					(reference "#PWR030")
+					(reference "#PWR0101")
 					(unit 1)
 				)
@@
 		(on_board yes)
 		(dnp no)
-		(property "Reference" "D3"
+		(property "Reference" "D5"
 			(at 171.45 104.14 0)
 			(effects
@@
 			(project "frank_m2"
 				(path "/8c0b3d8b-46d3-4173-ab1e-a61765f77d61/0d431c2a-21fb-40ea-8f7b-9d17d283876a"
-					(reference "D3")
+					(reference "D5")
 					(unit 1)
 				)
@@
 		(dnp no)
 		(fields_autoplaced yes)
-		(property "Reference" "#PWR035"
+		(property "Reference" "#PWR0109"
 			(at 224.79 93.98 0)
 			(effects
@@
 			(project "frank_m2"
 				(path "/8c0b3d8b-46d3-4173-ab1e-a61765f77d61/0d431c2a-21fb-40ea-8f7b-9d17d283876a"
-					(reference "#PWR035")
+					(reference "#PWR0109")
 					(unit 1)
 				)
@@
 		(on_board yes)
 		(dnp no)
-		(property "Reference" "#PWR032"
+		(property "Reference" "#PWR0107"
 			(at 209.55 102.87 0)
 			(effects
@@
 			(project "frank_m2"
 				(path "/8c0b3d8b-46d3-4173-ab1e-a61765f77d61/0d431c2a-21fb-40ea-8f7b-9d17d283876a"
-					(reference "#PWR032")
+					(reference "#PWR0107")
 					(unit 1)
 				)
@@
 		(dnp no)
 		(fields_autoplaced yes)
-		(property "Reference" "#PWR034"
+		(property "Reference" "#PWR0105"
 			(at 168.91 93.98 0)
 			(effects
@@
 			(project "frank_m2"
 				(path "/8c0b3d8b-46d3-4173-ab1e-a61765f77d61/0d431c2a-21fb-40ea-8f7b-9d17d283876a"
-					(reference "#PWR034")
+					(reference "#PWR0105")
 					(unit 1)
 				)
@@
 		(dnp no)
 		(fields_autoplaced yes)
-		(property "Reference" "#PWR028"
+		(property "Reference" "#PWR0104"
 			(at 168.91 66.04 0)
 			(effects
@@
 			(project "frank_m2"
 				(path "/8c0b3d8b-46d3-4173-ab1e-a61765f77d61/0d431c2a-21fb-40ea-8f7b-9d17d283876a"
-					(reference "#PWR028")
+					(reference "#PWR0104")
 					(unit 1)
 				)
@@
 		(on_board yes)
 		(dnp no)
-		(property "Reference" "R12"
+		(property "Reference" "R34"
 			(at 161.29 81.534 90)
 			(effects
@@
 			)
 		)
-		(property "Footprint" "FRANK:Resistor (0805)"
+		(property "Footprint" "FRANK:Resistor (0603)"
 			(at 161.29 85.598 90)
 			(effects
@@
 			(project "frank_m2"
 				(path "/8c0b3d8b-46d3-4173-ab1e-a61765f77d61/0d431c2a-21fb-40ea-8f7b-9d17d283876a"
-					(reference "R12")
+					(reference "R34")
 					(unit 1)
 				)
@@
 		(on_board yes)
 		(dnp no)
-		(property "Reference" "#PWR029"
+		(property "Reference" "#PWR099"
 			(at 71.12 92.71 0)
 			(effects
@@
 			(project "frank_m2"
 				(path "/8c0b3d8b-46d3-4173-ab1e-a61765f77d61/0d431c2a-21fb-40ea-8f7b-9d17d283876a"
-					(reference "#PWR029")
+					(reference "#PWR099")
 					(unit 1)
 				)
@@
 		(on_board yes)
 		(dnp no)
-		(property "Reference" "D2"
+		(property "Reference" "D4"
 			(at 171.45 76.2 0)
 			(effects
@@
 			(project "frank_m2"
 				(path "/8c0b3d8b-46d3-4173-ab1e-a61765f77d61/0d431c2a-21fb-40ea-8f7b-9d17d283876a"
-					(reference "D2")
+					(reference "D4")
 					(unit 1)
 				)
@@
 		(on_board yes)
 		(dnp no)
-		(property "Reference" "#PWR026"
+		(property "Reference" "#PWR0102"
 			(at 153.67 74.93 0)
 			(effects
@@
 			(project "frank_m2"
 				(path "/8c0b3d8b-46d3-4173-ab1e-a61765f77d61/0d431c2a-21fb-40ea-8f7b-9d17d283876a"
-					(reference "#PWR026")
+					(reference "#PWR0102")
 					(unit 1)
 				)
@@
 		(on_board yes)
 		(dnp no)
-		(property "Reference" "#PWR033"
+		(property "Reference" "#PWR0100"
 			(at 69.85 106.68 0)
 			(effects
@@
 			(project "frank_m2"
 				(path "/8c0b3d8b-46d3-4173-ab1e-a61765f77d61/0d431c2a-21fb-40ea-8f7b-9d17d283876a"
-					(reference "#PWR033")
+					(reference "#PWR0100")
 					(unit 1)
 				)
@@
 		(on_board yes)
 		(dnp no)
-		(property "Reference" "R9"
+		(property "Reference" "R36"
 			(at 207.01 73.66 90)
 			(effects
@@
 			)
 		)
-		(property "Footprint" "FRANK:Resistor (0805)"
+		(property "Footprint" "FRANK:Resistor (0603)"
 			(at 211.328 73.66 90)
 			(effects
@@
 			(project "frank_m2"
 				(path "/8c0b3d8b-46d3-4173-ab1e-a61765f77d61/0d431c2a-21fb-40ea-8f7b-9d17d283876a"
-					(reference "R9")
+					(reference "R36")
 					(unit 1)
 				)
@@
 		(on_board yes)
 		(dnp no)
-		(property "Reference" "R16"
+		(property "Reference" "R39"
 			(at 217.17 109.474 90)
 			(effects
@@
 			)
 		)
-		(property "Footprint" "FRANK:Resistor (0805)"
+		(property "Footprint" "FRANK:Resistor (0603)"
 			(at 217.17 113.538 90)
 			(effects
@@
 			(project "frank_m2"
 				(path "/8c0b3d8b-46d3-4173-ab1e-a61765f77d61/0d431c2a-21fb-40ea-8f7b-9d17d283876a"
-					(reference "R16")
+					(reference "R39")
 					(unit 1)
 				)
@@
 		(on_board yes)
 		(dnp no)
-		(property "Reference" "#PWR031"
+		(property "Reference" "#PWR0103"
 			(at 153.67 102.87 0)
 			(effects
@@
 			(project "frank_m2"
 				(path "/8c0b3d8b-46d3-4173-ab1e-a61765f77d61/0d431c2a-21fb-40ea-8f7b-9d17d283876a"
-					(reference "#PWR031")
-					(unit 1)
-				)
+					(reference "#PWR0103")
+					(unit 1)
+				)

Commit message: FRANK One HW 1.01
Other:
- title: FRANK M2 -> ${NAME} ${MODEL} (${BOARD})
Changed lines of the file:
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@@
 	(paper "A4")
 	(title_block
-		(title "FRANK M2")
-		(date "2025-08-20")
-		(rev "1.04")
+		(title "${NAME} ${MODEL} (${BOARD})")
+		(date "${DATE}")
+		(rev "${VERSION}")
 		(company "Mikhail Matveev")
 		(comment 1 "https://github.com/xtremespb/frank")
