File: lab/frank_one/tape.kicad_sch (KiCad schematic)
At the start: 11 parts, among them J9 PJ-320D, Q1 BC850, Q2 BC850

Commit message: Boards WIP
Parts:
- renumbered C3 to C4, C4 to C5, J9 to J10, R13 to R10, R14 to R11, R15 to R12, R11 to R8, R12 to R9

Commit message: FRANK Fastbeta PWT, One WIP
Parts:
- C3: renamed from C5; footprint FRANK:Capacitor (0805) -> FRANK:Capacitor (0603)
- C4: footprint FRANK:Capacitor (0805) -> FRANK:Capacitor (0603)
- R10: footprint FRANK:Resistor (0805) -> FRANK:Resistor (0603)
- R11: renamed from R9; footprint FRANK:Resistor (0805) -> FRANK:Resistor (0603)
- R7: renamed from R12; footprint FRANK:Resistor (0805) -> FRANK:Resistor (0603)
- R8: renamed from R11; footprint FRANK:Resistor (0805) -> FRANK:Resistor (0603)
- R9: renamed from R8; footprint FRANK:Resistor (0805) -> FRANK:Resistor (0603)
- renumbered J10 to J9, Q2 to Q1, Q1 to Q2
Changed lines of the file:
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@@
 		(dnp no)
 		(fields_autoplaced yes)
-		(property "Reference" "#PWR038"
+		(property "Reference" "#PWR031"
 			(at 158.75 125.73 0)
 			(effects
@@
 			(project "minifrank_rm1"
 				(path "/8c0b3d8b-46d3-4173-ab1e-a61765f77d61/8f57fa0b-80dc-4c8c-9148-33c48d230b70"
-					(reference "#PWR038")
+					(reference "#PWR031")
 					(unit 1)
 				)
@@
 			)
 		)
-		(property "Footprint" "FRANK:Resistor (0805)"
+		(property "Footprint" "FRANK:Resistor (0603)"
 			(at 165.1 98.298 90)
 			(effects
@@
 		(dnp no)
 		(fields_autoplaced yes)
-		(property "Reference" "#PWR037"
+		(property "Reference" "#PWR030"
 			(at 125.73 125.73 0)
 			(effects
@@
 			(project "minifrank_rm1"
 				(path "/8c0b3d8b-46d3-4173-ab1e-a61765f77d61/8f57fa0b-80dc-4c8c-9148-33c48d230b70"
-					(reference "#PWR037")
+					(reference "#PWR030")
 					(unit 1)
 				)
@@
 		(dnp no)
 		(fields_autoplaced yes)
-		(property "Reference" "R9"
+		(property "Reference" "R11"
 			(at 179.07 83.8199 0)
 			(effects
@@
 			)
 		)
-		(property "Footprint" "FRANK:Resistor (0805)"
+		(property "Footprint" "FRANK:Resistor (0603)"
 			(at 174.752 85.09 90)
 			(effects
@@
 			(project "minifrank_rm1"
 				(path "/8c0b3d8b-46d3-4173-ab1e-a61765f77d61/8f57fa0b-80dc-4c8c-9148-33c48d230b70"
-					(reference "R9")
+					(reference "R11")
 					(unit 1)
 				)
@@
 		(on_board yes)
 		(dnp no)
-		(property "Reference" "J10"
+		(property "Reference" "J9"
 			(at 97.0281 105.2103 0)
 			(effects
@@
 			(project "minifrank_rm1"
 				(path "/8c0b3d8b-46d3-4173-ab1e-a61765f77d61/8f57fa0b-80dc-4c8c-9148-33c48d230b70"
-					(reference "J10")
+					(reference "J9")
 					(unit 1)
 				)
@@
 		(on_board yes)
 		(dnp no)
-		(property "Reference" "C5"
+		(property "Reference" "C3"
 			(at 130.81 100.33 90)
 			(effects
@@
 			)
 		)
-		(property "Footprint" "FRANK:Capacitor (0805)"
+		(property "Footprint" "FRANK:Capacitor (0603)"
 			(at 133.35 103.1748 0)
 			(effects
@@
 			(project "minifrank_rm1"
 				(path "/8c0b3d8b-46d3-4173-ab1e-a61765f77d61/8f57fa0b-80dc-4c8c-9148-33c48d230b70"
-					(reference "C5")
+					(reference "C3")
 					(unit 1)
 				)
@@
 		(dnp no)
 		(fields_autoplaced yes)
-		(property "Reference" "#PWR036"
+		(property "Reference" "#PWR029"
 			(at 115.57 111.76 0)
 			(effects
@@
 			(project "minifrank_rm1"
 				(path "/8c0b3d8b-46d3-4173-ab1e-a61765f77d61/8f57fa0b-80dc-4c8c-9148-33c48d230b70"
-					(reference "#PWR036")
+					(reference "#PWR029")
 					(unit 1)
 				)
@@
 		(dnp no)
 		(fields_autoplaced yes)
-		(property "Reference" "R11"
+		(property "Reference" "R8"
 			(at 140.97 97.79 90)
 			(effects
@@
 			)
 		)
-		(property "Footprint" "FRANK:Resistor (0805)"
+		(property "Footprint" "FRANK:Resistor (0603)"
 			(at 140.97 105.918 90)
 			(effects
@@
 			(project "minifrank_rm1"
 				(path "/8c0b3d8b-46d3-4173-ab1e-a61765f77d61/8f57fa0b-80dc-4c8c-9148-33c48d230b70"
-					(reference "R11")
+					(reference "R8")
 					(unit 1)
 				)
@@
 		(dnp no)
 		(fields_autoplaced yes)
-		(property "Reference" "#PWR035"
+		(property "Reference" "#PWR034"
 			(at 198.12 90.17 0)
 			(effects
@@
 			(project "minifrank_rm1"
 				(path "/8c0b3d8b-46d3-4173-ab1e-a61765f77d61/8f57fa0b-80dc-4c8c-9148-33c48d230b70"
-					(reference "#PWR035")
+					(reference "#PWR034")
 					(unit 1)
 				)
@@
 		(dnp no)
 		(fields_autoplaced yes)
-		(property "Reference" "#PWR039"
+		(property "Reference" "#PWR032"
 			(at 176.53 125.73 0)
 			(effects
@@
 			(project "minifrank_rm1"
 				(path "/8c0b3d8b-46d3-4173-ab1e-a61765f77d61/8f57fa0b-80dc-4c8c-9148-33c48d230b70"
-					(reference "#PWR039")
+					(reference "#PWR032")
 					(unit 1)
 				)
@@
 		(dnp no)
 		(fields_autoplaced yes)
-		(property "Reference" "#PWR034"
+		(property "Reference" "#PWR033"
 			(at 181.61 74.93 0)
 			(effects
@@
 			(project "minifrank_rm1"
 				(path "/8c0b3d8b-46d3-4173-ab1e-a61765f77d61/8f57fa0b-80dc-4c8c-9148-33c48d230b70"
-					(reference "#PWR034")
+					(reference "#PWR033")
 					(unit 1)
 				)
@@
 			)
 		)
-		(property "Footprint" "FRANK:Capacitor (0805)"
+		(property "Footprint" "FRANK:Capacitor (0603)"
 			(at 192.7352 86.36 0)
 			(effects
@@
 		(dnp no)
 		(fields_autoplaced yes)
-		(property "Reference" "R12"
+		(property "Reference" "R7"
 			(at 127.508 114.3578 0)
 			(effects
@@
 			)
 		)
-		(property "Footprint" "FRANK:Resistor (0805)"
+		(property "Footprint" "FRANK:Resistor (0603)"
 			(at 123.952 115.57 90)
 			(effects
@@
 			(project "minifrank_rm1"
 				(path "/8c0b3d8b-46d3-4173-ab1e-a61765f77d61/8f57fa0b-80dc-4c8c-9148-33c48d230b70"
-					(reference "R12")
+					(reference "R7")
 					(unit 1)
 				)
@@
 		(dnp no)
 		(fields_autoplaced yes)
-		(property "Reference" "Q2"
+		(property "Reference" "Q1"
 			(at 161.0614 103.3053 0)
 			(effects
@@
 			(project "minifrank_rm1"
 				(path "/8c0b3d8b-46d3-4173-ab1e-a61765f77d61/8f57fa0b-80dc-4c8c-9148-33c48d230b70"
-					(reference "Q2")
+					(reference "Q1")
 					(unit 1)
 				)
@@
 		(dnp no)
 		(fields_autoplaced yes)
-		(property "Reference" "R8"
+		(property "Reference" "R9"
 			(at 161.29 83.8199 0)
 			(effects
@@
 			)
 		)
-		(property "Footprint" "FRANK:Resistor (0805)"
+		(property "Footprint" "FRANK:Resistor (0603)"
 			(at 156.972 85.09 90)
 			(effects
@@
 			(project "minifrank_rm1"
 				(path "/8c0b3d8b-46d3-4173-ab1e-a61765f77d61/8f57fa0b-80dc-4c8c-9148-33c48d230b70"
-					(reference "R8")
+					(reference "R9")
 					(unit 1)
 				)
@@
 		(dnp no)
 		(fields_autoplaced yes)
-		(property "Reference" "Q1"
+		(property "Reference" "Q2"
 			(at 178.8414 95.6853 0)
 			(effects
@@
 			(project "minifrank_rm1"
 				(path "/8c0b3d8b-46d3-4173-ab1e-a61765f77d61/8f57fa0b-80dc-4c8c-9148-33c48d230b70"
-					(reference "Q1")
-					(unit 1)
-				)
+					(reference "Q2")
+					(unit 1)
+				)

Commit message: FRANK One HW 1.01
Other:
- title: ${NAME} ${MODEL} -> ${NAME} ${MODEL} (${BOARD})
Changed lines of the file:
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@@
 	(paper "A4")
 	(title_block
-		(title "${NAME} ${MODEL}")
+		(title "${NAME} ${MODEL} (${BOARD})")
 		(date "${DATE}")
 		(rev "${VERSION}")
