File: lab/tinyfrank_rm1p2/ps2.kicad_sch (KiCad schematic)
At the start: 14 parts, among them J7 MDC-036

Commit message: TinyFRANK WIP
Parts:
- renumbered J7 to J6
Changed lines of the file:
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@@
 		(on_board yes)
 		(dnp no)
-		(property "Reference" "#PWR062"
+		(property "Reference" "#PWR059"
 			(at 209.55 73.66 0)
 			(effects
@@
 			(project "frank_m2"
 				(path "/8c0b3d8b-46d3-4173-ab1e-a61765f77d61/e95ab524-4f6c-414a-a124-e627805404c7"
-					(reference "#PWR062")
+					(reference "#PWR059")
 					(unit 1)
 				)
@@
 		(dnp no)
 		(fields_autoplaced yes)
-		(property "Reference" "J7"
+		(property "Reference" "J6"
 			(at 97.8077 82.55 0)
 			(effects
@@
 			(project "frank_m2"
 				(path "/8c0b3d8b-46d3-4173-ab1e-a61765f77d61/e95ab524-4f6c-414a-a124-e627805404c7"
-					(reference "J7")
+					(reference "J6")
 					(unit 1)
 				)
@@
 		(dnp no)
 		(fields_autoplaced yes)
-		(property "Reference" "#PWR064"
+		(property "Reference" "#PWR061"
 			(at 224.79 64.77 0)
 			(effects
@@
 			(project "frank_m2"
 				(path "/8c0b3d8b-46d3-4173-ab1e-a61765f77d61/e95ab524-4f6c-414a-a124-e627805404c7"
-					(reference "#PWR064")
+					(reference "#PWR061")
 					(unit 1)
 				)
@@
 		(on_board yes)
 		(dnp no)
-		(property "Reference" "#PWR057"
+		(property "Reference" "#PWR054"
 			(at 127 92.71 0)
 			(effects
@@
 			(project "frank_m2"
 				(path "/8c0b3d8b-46d3-4173-ab1e-a61765f77d61/e95ab524-4f6c-414a-a124-e627805404c7"
-					(reference "#PWR057")
+					(reference "#PWR054")
 					(unit 1)
 				)
@@
 		(dnp no)
 		(fields_autoplaced yes)
-		(property "Reference" "#PWR065"
+		(property "Reference" "#PWR062"
 			(at 224.79 93.98 0)
 			(effects
@@
 			(project "frank_m2"
 				(path "/8c0b3d8b-46d3-4173-ab1e-a61765f77d61/e95ab524-4f6c-414a-a124-e627805404c7"
-					(reference "#PWR065")
+					(reference "#PWR062")
 					(unit 1)
 				)
@@
 		(on_board yes)
 		(dnp no)
-		(property "Reference" "#PWR063"
+		(property "Reference" "#PWR060"
 			(at 209.55 102.87 0)
 			(effects
@@
 			(project "frank_m2"
 				(path "/8c0b3d8b-46d3-4173-ab1e-a61765f77d61/e95ab524-4f6c-414a-a124-e627805404c7"
-					(reference "#PWR063")
+					(reference "#PWR060")
 					(unit 1)
 				)
@@
 		(dnp no)
 		(fields_autoplaced yes)
-		(property "Reference" "#PWR061"
+		(property "Reference" "#PWR058"
 			(at 168.91 93.98 0)
 			(effects
@@
 			(project "frank_m2"
 				(path "/8c0b3d8b-46d3-4173-ab1e-a61765f77d61/e95ab524-4f6c-414a-a124-e627805404c7"
-					(reference "#PWR061")
+					(reference "#PWR058")
 					(unit 1)
 				)
@@
 		(dnp no)
 		(fields_autoplaced yes)
-		(property "Reference" "#PWR060"
+		(property "Reference" "#PWR057"
 			(at 168.91 66.04 0)
 			(effects
@@
 			(project "frank_m2"
 				(path "/8c0b3d8b-46d3-4173-ab1e-a61765f77d61/e95ab524-4f6c-414a-a124-e627805404c7"
-					(reference "#PWR060")
+					(reference "#PWR057")
 					(unit 1)
 				)
@@
 		(on_board yes)
 		(dnp no)
-		(property "Reference" "#PWR055"
+		(property "Reference" "#PWR052"
 			(at 71.12 92.71 0)
 			(effects
@@
 			(project "frank_m2"
 				(path "/8c0b3d8b-46d3-4173-ab1e-a61765f77d61/e95ab524-4f6c-414a-a124-e627805404c7"
-					(reference "#PWR055")
+					(reference "#PWR052")
 					(unit 1)
 				)
@@
 		(on_board yes)
 		(dnp no)
-		(property "Reference" "#PWR058"
+		(property "Reference" "#PWR055"
 			(at 153.67 74.93 0)
 			(effects
@@
 			(project "frank_m2"
 				(path "/8c0b3d8b-46d3-4173-ab1e-a61765f77d61/e95ab524-4f6c-414a-a124-e627805404c7"
-					(reference "#PWR058")
+					(reference "#PWR055")
 					(unit 1)
 				)
@@
 		(on_board yes)
 		(dnp no)
-		(property "Reference" "#PWR056"
+		(property "Reference" "#PWR053"
 			(at 69.85 106.68 0)
 			(effects
@@
 			(project "frank_m2"
 				(path "/8c0b3d8b-46d3-4173-ab1e-a61765f77d61/e95ab524-4f6c-414a-a124-e627805404c7"
-					(reference "#PWR056")
+					(reference "#PWR053")
 					(unit 1)
 				)
@@
 		(on_board yes)
 		(dnp no)
-		(property "Reference" "#PWR059"
+		(property "Reference" "#PWR056"
 			(at 153.67 102.87 0)
 			(effects
@@
 			(project "frank_m2"
 				(path "/8c0b3d8b-46d3-4173-ab1e-a61765f77d61/e95ab524-4f6c-414a-a124-e627805404c7"
-					(reference "#PWR059")
-					(unit 1)
-				)
+					(reference "#PWR056")
+					(unit 1)
+				)
