File: lab/tinyfrank_rm1p2/tape.kicad_sch (KiCad schematic)
At the start: 11 parts, among them Q1 BC850, Q2 BC850

Commit message: TinyFRANK RM1P2 1.00
Parts:
- renumbered AJ1 to J7
Changed lines of the file:
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@@
 		(on_board yes)
 		(dnp no)
-		(property "Reference" "AJ1"
+		(property "Reference" "J7"
 			(at 97.0281 102.6703 0)
 			(effects
@@
 			(project "38NJU24"
 				(path "/8c0b3d8b-46d3-4173-ab1e-a61765f77d61/e3ca564e-da9b-40b5-a06b-378e9f062223"
-					(reference "AJ1")
+					(reference "J7")
 					(unit 1)
 				)
