File: lab/tinyfrank_rm1p2/tinyfrank_rm1p2.kicad_pcb (KiCad board)
At the start: 2 copper layers, 68 x 37.5 mm, 85 parts, among them J1 PWR, J2 676430910, J3 0475710001, J4 PJ-320D, J5 USB4215-03-A, J6 DC3RX19JA2, J7 MDC-036, U1 USBLC6-2SC6, U2 NCP1117 3.3, U3 ESP-PSRAM32, U4 W25Q128JVS, U5 RP2350, Y1 ASE-12MHz

Commit message: TinyFRANK WIP
Parts:
- removed the J1 at (56.8, 70.0)
- added AJ1: PJ-320D, FRANK:Jack (3.5mm, PJ-320D), F.Cu at (141.5, 59.5)
- added C27: 100n, FRANK:Capacitor (0402), F.Cu at (135.0, 60.8)
- added C28: 100n, FRANK:Capacitor (0402), F.Cu at (139.0, 71.5)
- added D6: 1N4148, FRANK:Diode (SOD-523), F.Cu at (137.5, 66.8)
- added Q1: BC850, FRANK:SOT-23, F.Cu at (133.6, 65.7)
- added Q2: BC850, FRANK:SOT-23, F.Cu at (136.2, 69.9)
- added R30: 100R, FRANK:Resistor (0402), F.Cu at (135.0, 58.8)
- added R31: 10K, FRANK:Resistor (0402), F.Cu at (135.0, 62.8)
- added R32: 10K, FRANK:Resistor (0402), F.Cu at (133.0, 68.8)
- added R33: 10K, FRANK:Resistor (0402), F.Cu at (133.0, 70.2)
- added R34: 1K, FRANK:Resistor (0402), F.Cu at (139.0, 69.1)
- moved R22 66.0 mm to (129.5, 84.0), turned to -90 degrees
- moved R24 64.8 mm to (129.5, 81.5), turned to 90 degrees
- moved R23 63.6 mm to (127.5, 84.0), turned to -90 degrees
- moved C1 63.3 mm to (138.5, 87.8), turned to -90 degrees
- moved R25 62.6 mm to (127.5, 81.5), turned to 90 degrees
- moved R26 60.7 mm to (125.5, 84.0), turned to -90 degrees
- moved R28 60.3 mm to (125.5, 81.5), turned to 90 degrees
- moved R27 58.5 mm to (123.5, 84.0), turned to -90 degrees
- moved R29 58.3 mm to (123.5, 81.5), turned to 90 degrees
- moved C26 44.3 mm to (127.8, 62.0)
- moved D2 37.4 mm to (121.2, 83.5), turned to 180 degrees
- moved S2 36.0 mm to (128.0, 88.8), turned to 180 degrees
- moved D5 35.6 mm to (122.0, 81.3), turned to -90 degrees
- moved D4 34.3 mm to (120.2, 81.3), turned to -90 degrees
- moved D3 33.2 mm to (118.5, 81.3), turned to -90 degrees
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- renumbered J2 to J1, J3 to J2, J4 to J3, J5 to J4, J6 to J5, J7 to J6

Commit message: TinyFRANK RM1P2 1.00
Parts:
- added G***: LOGO, FRANK:FRANK Logo, B.Cu at (138.0, 65.9)
- added JP4: Mouse (DATA), FRANK:Jumper (solder), B.Cu at (141.5, 72.3)
- added JP5: Mouse (CLK), FRANK:Jumper (solder), B.Cu at (145.2, 72.4)
- moved R5 53.5 mm to (153.8, 68.5), turned to -90 degrees
- moved C4 52.5 mm to (152.0, 68.0), turned to -90 degrees
- moved R9 51.9 mm to (151.1, 72.8)
- moved R8 50.5 mm to (151.1, 76.5)
- moved R7 50.4 mm to (151.1, 75.2)
- moved R6 50.3 mm to (151.1, 74.0)
- moved C6 46.7 mm to (150.0, 68.5), turned to 90 degrees
- moved C3 46.0 mm to (146.0, 68.0), turned to -90 degrees
- moved C5 44.1 mm to (148.0, 68.5), turned to 90 degrees
- moved R4 43.1 mm to (143.2, 67.0), turned to 180 degrees
- moved C14 2.78 mm to (161.6, 79.8)
- moved C20 2.28 mm to (169.6, 74.0), turned to -45 degrees
- moved C12 1.78 mm to (164.8, 83.2)
- moved C15 1.72 mm to (170.1, 71.3), turned to -45 degrees
- moved C9 1.51 mm to (177.2, 85.3)
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- renumbered AJ1 to J7
Connections:
- D4 pad 1: /GPIO14 -> /MS_CLK
- D5 pad 1: /GPIO15 -> /MS_DATA
- Q2 pad 3: /PGPIO22 -> /GPIO22
- R28 pad 2: /GPIO14 -> /MS_CLK
- R29 pad 2: /GPIO15 -> /MS_DATA
- R34 pad 2: /PGPIO22 -> /GPIO22
Routing:
- net +3V3: track 0.00 -> 134.2 mm, vias 0 -> 7
- net VBUS: track 0.00 -> 110.6 mm, vias 0 -> 3
- net /GPIO1: track 0.00 -> 73.2 mm, vias 0 -> 3
- net /GPIO0: track 0.00 -> 66.1 mm, vias 0 -> 3
- net /GPIO15: track 0.00 -> 44.8 mm, vias 0 -> 1
- net /GPIO19: track 0.00 -> 41.3 mm, vias 0 -> 4
- net Net-(S2-B): track 0.00 -> 40.0 mm, vias 0 -> 2
- net /GPIO14: track 0.00 -> 38.1 mm, vias 0 -> 1
- net /MS_CLK: track 0.00 -> 36.3 mm, vias 0 -> 2
- net /GPIO5: track 0.00 -> 33.9 mm, vias 0 -> 2
- net /GPIO3: track 0.00 -> 30.3 mm, vias 0 -> 2
- net +1V1: track 0.00 -> 27.5 mm
- net Net-(D1-K): track 0.00 -> 27.0 mm
- net /GPIO2: track 0.00 -> 25.7 mm, vias 0 -> 2
- net /RP2350A/QSPI_SD1: track 0.00 -> 25.4 mm
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- added copper zone on F.Cu, net +1V1
- added copper zone on B.Cu, net +3V3
- added copper zone on F.Cu, net +3V3
- added copper zone on B.Cu, net GND
- added copper zone on F.Cu, net GND
Other:
- outline, holes or cut-outs redrawn
- board text added: "${MODEL} HW ${VERSION}"
- board text added: "AUDIO OUT"
- board text added: "KB/BOOT"
- board text added: "PS/2"
- board text added: "TAPE IN"
- board text added: "rh1.tech"
