File: lab/frank_m1/frank_m1.kicad_sch (KiCad schematic)
At the start: 13 parts, among them J1 EXT Sound, J2 PWR, J3 UART

Commit message: FRANK M1 2.04
Parts:
- R1, R2, R3, R4: symbol Device:R -> FRANK:R
Other:
- title: ${NAME} ${VARIANT} -> ${NAME} ${MODEL}
Changed lines of the file:
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@@
 	(paper "A4")
 	(title_block
-		(title "${NAME} ${VARIANT}")
+		(title "${NAME} ${MODEL}")
 		(date "${DATE}")
 		(rev "${VERSION}")
@@
 		)
 	)
-	(label "PGPIO11"
+	(label "PGPIO13"
 		(at 25.4 87.63 0)
 		(effects
@@
 	)
 	(symbol
-		(lib_id "Device:R")
+		(lib_id "FRANK:R")
 		(at 242.57 67.31 270)
 		(unit 1)
@@
 	)
 	(symbol
-		(lib_id "Device:R")
+		(lib_id "FRANK:R")
 		(at 242.57 58.42 270)
 		(unit 1)
@@
 	)
 	(symbol
-		(lib_id "Device:R")
+		(lib_id "FRANK:R")
 		(at 200.66 58.42 270)
 		(unit 1)
@@
 	)
 	(symbol
-		(lib_id "Device:R")
+		(lib_id "FRANK:R")
 		(at 200.66 67.31 270)
 		(unit 1)

Commit message: FRANK M1 + TinyFRANK RM2 WIP
Parts:
- removed J1: EXT Sound, FRANK:PinHeader_2x10_P2.54mm_Vertical, symbol Connector_Generic:Conn_02x10_Odd_Even
- renumbered J3 to J1
Connections:
- net A_EXT is gone; now on net Z_VBUS: JP1.2
- net +3V3: now also JP1.10; no longer JP1.9
- net GND: now also JP1.9; no longer JP1.8
- net MONO_L: now also JP1.5; no longer JP1.6
- net MONO_R: now also JP1.8; no longer JP1.7
- net MSPUP3V3: now also JP1.3; no longer JP1.4
- net PGPIO22: now also JP1.7
- net SHND: now also JP1.4; no longer JP1.5
- net VBUS: no longer JP1.10
- net Z_VBUS: no longer JP1.3
- net A_TDA renamed AUDIOSW
- new net LOAD_IN: JP1.6
Other:
- sheet Audio Multiplexer ports: added AUDIOSW; removed EXT_L, EXT_R, J_EXT, J_TDA
- moved on the sheet: J1, J2, S1

Commit message: HW 2.05 WIP
Other:
- sheet Audio: file ../../hardware/frank_m1/audio.kicad_sch -> audio.kicad_sch
- sheet Audio Multiplexer: file ../../hardware/frank_m1/audio_multiplexer.kicad_sch -> audio_multiplexer.kicad_sch
- sheet Composite: file ../../hardware/frank_m1/composite.kicad_sch -> composite.kicad_sch
- sheet Display: file ../../hardware/frank_m1/display.kicad_sch -> display.kicad_sch
- sheet Gamepad 1: file ../../hardware/frank_m1/gamepad.kicad_sch -> gamepad.kicad_sch
- sheet Gamepad 2: file ../../hardware/frank_m1/gamepad.kicad_sch -> gamepad.kicad_sch
- sheet Micro SD: file ../../hardware/frank_m1/sd.kicad_sch -> sd.kicad_sch
- sheet PSRAM: file ../../hardware/frank_m1/psram.kicad_sch -> psram.kicad_sch
- sheet Tape In: file ../../hardware/frank_m1/tape.kicad_sch -> tape.kicad_sch
- sheet USB Stacked: file ../../hardware/frank_m1/usbstack.kicad_sch -> usbstack.kicad_sch
- sheet VGA: file ../../hardware/frank_m1/vga.kicad_sch -> vga.kicad_sch
- sheet Zero: file ../../hardware/frank_m1/zero.kicad_sch -> zero.kicad_sch
Changed lines of the file:
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@@
 			)
 		)
-		(property "Sheetfile" "../../hardware/frank_m1/tape.kicad_sch"
+		(property "Sheetfile" "tape.kicad_sch"
 			(at 69.85 78.0546 0)
 			(effects
@@
 			)
 		)
-		(property "Sheetfile" "../../hardware/frank_m1/display.kicad_sch"
+		(property "Sheetfile" "display.kicad_sch"
 			(at 38.1 98.3746 0)
 			(effects
@@
 			)
 		)
-		(property "Sheetfile" "../../hardware/frank_m1/composite.kicad_sch"
+		(property "Sheetfile" "composite.kicad_sch"
 			(at 38.1 122.5046 0)
 			(effects
@@
 			)
 		)
-		(property "Sheetfile" "../../hardware/frank_m1/vga.kicad_sch"
+		(property "Sheetfile" "vga.kicad_sch"
 			(at 38.1 76.7846 0)
 			(effects
@@
 			)
 		)
-		(property "Sheetfile" "../../hardware/frank_m1/zero.kicad_sch"
+		(property "Sheetfile" "zero.kicad_sch"
 			(at 142.24 161.8746 0)
 			(effects
@@
 			)
 		)
-		(property "Sheetfile" "../../hardware/frank_m1/psram.kicad_sch"
+		(property "Sheetfile" "psram.kicad_sch"
 			(at 69.85 97.1046 0)
 			(effects
@@
 			)
 		)
-		(property "Sheetfile" "../../hardware/frank_m1/audio.kicad_sch"
+		(property "Sheetfile" "audio.kicad_sch"
 			(at 105.41 71.7046 0)
 			(effects
@@
 			)
 		)
-		(property "Sheetfile" "../../hardware/frank_m1/gamepad.kicad_sch"
+		(property "Sheetfile" "gamepad.kicad_sch"
 			(at 105.41 130.1246 0)
 			(effects
@@
 			)
 		)
-		(property "Sheetfile" "../../hardware/frank_m1/gamepad.kicad_sch"
+		(property "Sheetfile" "gamepad.kicad_sch"
 			(at 105.41 145.3646 0)
 			(effects
@@
 			)
 		)
-		(property "Sheetfile" "../../hardware/frank_m1/audio_multiplexer.kicad_sch"
+		(property "Sheetfile" "audio_multiplexer.kicad_sch"
 			(at 105.41 97.1046 0)
 			(effects
@@
 			)
 		)
-		(property "Sheetfile" "../../hardware/frank_m1/usbstack.kicad_sch"
+		(property "Sheetfile" "usbstack.kicad_sch"
 			(at 69.85 67.8946 0)
 			(effects
@@
 			)
 		)
-		(property "Sheetfile" "../../hardware/frank_m1/sd.kicad_sch"
+		(property "Sheetfile" "sd.kicad_sch"
 			(at 105.41 114.8846 0)
 			(effects
