File: lab/frank_fastbeta_pwt/psram.kicad_sch (KiCad schematic)
At the start: 3 parts, among them U5 ESP-PSRAM32

Commit message: Boards WIP
Parts:
- renumbered C14 to C11, U5 to U4
Changed lines of the file:
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@@
 		(on_board yes)
 		(dnp no)
-		(property "Reference" "#PWR042"
+		(property "Reference" "#PWR047"
 			(at 148.59 111.76 0)
 			(effects
@@
 			(project "minifrank_rm1p2"
 				(path "/8c0b3d8b-46d3-4173-ab1e-a61765f77d61/69959616-34ef-45d1-8eb1-8ce60ead3b7b"
-					(reference "#PWR042")
+					(reference "#PWR047")
 					(unit 1)
 				)
@@
 		(dnp no)
 		(fields_autoplaced yes)
-		(property "Reference" "#PWR043"
+		(property "Reference" "#PWR048"
 			(at 158.75 83.82 0)
 			(effects
@@
 			(project "minifrank_rm1p2"
 				(path "/8c0b3d8b-46d3-4173-ab1e-a61765f77d61/69959616-34ef-45d1-8eb1-8ce60ead3b7b"
-					(reference "#PWR043")
+					(reference "#PWR048")
 					(unit 1)
 				)
@@
 		(dnp no)
 		(fields_autoplaced yes)
-		(property "Reference" "U5"
+		(property "Reference" "U4"
 			(at 142.24 91.4399 0)
 			(effects
@@
 			(project "minifrank_rm1p2"
 				(path "/8c0b3d8b-46d3-4173-ab1e-a61765f77d61/69959616-34ef-45d1-8eb1-8ce60ead3b7b"
-					(reference "U5")
+					(reference "U4")
 					(unit 1)
 				)
@@
 		(on_board yes)
 		(dnp no)
-		(property "Reference" "C14"
+		(property "Reference" "C11"
 			(at 131.191 86.4616 0)
 			(effects
@@
 			(project "minifrank_rm1p2"
 				(path "/8c0b3d8b-46d3-4173-ab1e-a61765f77d61/69959616-34ef-45d1-8eb1-8ce60ead3b7b"
-					(reference "C14")
+					(reference "C11")
 					(unit 1)
 				)
@@
 		(on_board yes)
 		(dnp no)
-		(property "Reference" "#PWR041"
+		(property "Reference" "#PWR046"
 			(at 128.27 101.6 0)
 			(effects
@@
 			(project "minifrank_rm1p2"
 				(path "/8c0b3d8b-46d3-4173-ab1e-a61765f77d61/69959616-34ef-45d1-8eb1-8ce60ead3b7b"
-					(reference "#PWR041")
+					(reference "#PWR046")
 					(unit 1)
 				)

Commit message: Board updates
Parts:
- renumbered U4 to U5
Changed lines of the file:
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@@
 		(on_board yes)
 		(dnp no)
-		(property "Reference" "#PWR047"
+		(property "Reference" "#PWR049"
 			(at 148.59 111.76 0)
 			(effects
@@
 			(project "minifrank_rm1p2"
 				(path "/8c0b3d8b-46d3-4173-ab1e-a61765f77d61/69959616-34ef-45d1-8eb1-8ce60ead3b7b"
-					(reference "#PWR047")
+					(reference "#PWR049")
 					(unit 1)
 				)
@@
 		(dnp no)
 		(fields_autoplaced yes)
-		(property "Reference" "#PWR048"
+		(property "Reference" "#PWR050"
 			(at 158.75 83.82 0)
 			(effects
@@
 			(project "minifrank_rm1p2"
 				(path "/8c0b3d8b-46d3-4173-ab1e-a61765f77d61/69959616-34ef-45d1-8eb1-8ce60ead3b7b"
-					(reference "#PWR048")
+					(reference "#PWR050")
 					(unit 1)
 				)
@@
 		(dnp no)
 		(fields_autoplaced yes)
-		(property "Reference" "U4"
+		(property "Reference" "U5"
 			(at 142.24 91.4399 0)
 			(effects
@@
 			(project "minifrank_rm1p2"
 				(path "/8c0b3d8b-46d3-4173-ab1e-a61765f77d61/69959616-34ef-45d1-8eb1-8ce60ead3b7b"
-					(reference "U4")
+					(reference "U5")
 					(unit 1)
 				)
@@
 		(on_board yes)
 		(dnp no)
-		(property "Reference" "#PWR046"
+		(property "Reference" "#PWR048"
 			(at 128.27 101.6 0)
 			(effects
@@
 			(project "minifrank_rm1p2"
 				(path "/8c0b3d8b-46d3-4173-ab1e-a61765f77d61/69959616-34ef-45d1-8eb1-8ce60ead3b7b"
-					(reference "#PWR046")
+					(reference "#PWR048")
 					(unit 1)
 				)
