File: hardware/frank_fastbeta_pwt/psram.kicad_sch (KiCad schematic)
At the start: 3 parts, among them U5 ESP-PSRAM32

Commit message: Board updates
Parts:
- renumbered C11 to C17
Changed lines of the file:
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@@
 		(on_board yes)
 		(dnp no)
-		(property "Reference" "#PWR049"
+		(property "Reference" "#PWR055"
 			(at 148.59 111.76 0)
 			(effects
@@
 			(project "minifrank_rm1p2"
 				(path "/8c0b3d8b-46d3-4173-ab1e-a61765f77d61/69959616-34ef-45d1-8eb1-8ce60ead3b7b"
-					(reference "#PWR049")
+					(reference "#PWR055")
 					(unit 1)
 				)
@@
 		(dnp no)
 		(fields_autoplaced yes)
-		(property "Reference" "#PWR050"
+		(property "Reference" "#PWR056"
 			(at 158.75 83.82 0)
 			(effects
@@
 			(project "minifrank_rm1p2"
 				(path "/8c0b3d8b-46d3-4173-ab1e-a61765f77d61/69959616-34ef-45d1-8eb1-8ce60ead3b7b"
-					(reference "#PWR050")
+					(reference "#PWR056")
 					(unit 1)
 				)
@@
 			)
 		)
+		(property "Sim.Device" ""
+			(at 151.13 92.71 0)
+			(effects
+				(font
+					(size 1.27 1.27)
+				)
+				(hide yes)
+			)
+		)
 		(pin "1"
 		)
@@
 		(on_board yes)
 		(dnp no)
-		(property "Reference" "C11"
+		(property "Reference" "C17"
 			(at 131.191 86.4616 0)
 			(effects
@@
 			)
 		)
-		(property "Datasheet" "https://eu.mouser.com/datasheet/2/40/KGM_X7R-3223212.pdf"
-			(at 128.27 87.63 0)
-			(effects
-				(font
-					(size 1.27 1.27)
-				)
-				(hide yes)
-			)
-		)
-		(property "Description" ""
+		(property "Datasheet" "~"
+			(at 128.27 87.63 0)
+			(effects
+				(font
+					(size 1.27 1.27)
+				)
+				(hide yes)
+			)
+		)
+		(property "Description" "Unpolarized capacitor"
 			(at 128.27 87.63 0)
 			(effects
@@
 		)
 		(property "Mouser Price/Stock" ""
+			(at 128.27 87.63 0)
+			(effects
+				(font
+					(size 1.27 1.27)
+				)
+				(hide yes)
+			)
+		)
+		(property "Sim.Device" ""
 			(at 128.27 87.63 0)
 			(effects
@@
 			(project "minifrank_rm1p2"
 				(path "/8c0b3d8b-46d3-4173-ab1e-a61765f77d61/69959616-34ef-45d1-8eb1-8ce60ead3b7b"
-					(reference "C11")
+					(reference "C17")
 					(unit 1)
 				)
@@
 			)
 		)
+		(property "Sim.Device" ""
+			(at 177.8 97.79 0)
+			(effects
+				(font
+					(size 1.27 1.27)
+				)
+				(hide yes)
+			)
+		)
 		(pin "1"
 		)
@@
 		(on_board yes)
 		(dnp no)
-		(property "Reference" "#PWR048"
+		(property "Reference" "#PWR054"
 			(at 128.27 101.6 0)
 			(effects
@@
 			(project "minifrank_rm1p2"
 				(path "/8c0b3d8b-46d3-4173-ab1e-a61765f77d61/69959616-34ef-45d1-8eb1-8ce60ead3b7b"
-					(reference "#PWR048")
+					(reference "#PWR054")
 					(unit 1)
 				)
