File: lab/frank_one_rm2/tape.kicad_sch (KiCad schematic)
At the start: 6 parts, among them J8 PJ-320D, U2 CD4069UBM

Commit message: Board updates
Parts:
- renumbered J8 to J9
Changed lines of the file:
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@@
 		(dnp no)
 		(fields_autoplaced yes)
-		(property "Reference" "#PWR030"
+		(property "Reference" "#PWR043"
 			(at 140.97 116.84 0)
 			(effects
@@
 			(project "frank_rm2"
 				(path "/8c0b3d8b-46d3-4173-ab1e-a61765f77d61/8f57fa0b-80dc-4c8c-9148-33c48d230b70"
-					(reference "#PWR030")
+					(reference "#PWR043")
 					(unit 1)
 				)
@@
 		(dnp no)
 		(fields_autoplaced yes)
-		(property "Reference" "#PWR034"
+		(property "Reference" "#PWR047"
 			(at 226.06 114.3 0)
 			(effects
@@
 			(project "frank_rm2"
 				(path "/8c0b3d8b-46d3-4173-ab1e-a61765f77d61/8f57fa0b-80dc-4c8c-9148-33c48d230b70"
-					(reference "#PWR034")
+					(reference "#PWR047")
 					(unit 1)
 				)
@@
 		(dnp no)
 		(fields_autoplaced yes)
-		(property "Reference" "#PWR033"
+		(property "Reference" "#PWR046"
 			(at 226.06 109.22 0)
 			(effects
@@
 			(project "frank_rm2"
 				(path "/8c0b3d8b-46d3-4173-ab1e-a61765f77d61/8f57fa0b-80dc-4c8c-9148-33c48d230b70"
-					(reference "#PWR033")
+					(reference "#PWR046")
 					(unit 1)
 				)
@@
 		(on_board yes)
 		(dnp no)
-		(property "Reference" "J8"
+		(property "Reference" "J9"
 			(at 72.8981 101.4003 0)
 			(effects
@@
 			(project "minifrank_rm1"
 				(path "/8c0b3d8b-46d3-4173-ab1e-a61765f77d61/8f57fa0b-80dc-4c8c-9148-33c48d230b70"
-					(reference "J8")
+					(reference "J9")
 					(unit 1)
 				)
@@
 		(dnp no)
 		(fields_autoplaced yes)
-		(property "Reference" "#PWR029"
+		(property "Reference" "#PWR042"
 			(at 91.44 107.95 0)
 			(effects
@@
 			(project "minifrank_rm1"
 				(path "/8c0b3d8b-46d3-4173-ab1e-a61765f77d61/8f57fa0b-80dc-4c8c-9148-33c48d230b70"
-					(reference "#PWR029")
+					(reference "#PWR042")
 					(unit 1)
 				)
@@
 		(on_board yes)
 		(dnp no)
-		(property "Reference" "#PWR031"
+		(property "Reference" "#PWR044"
 			(at 215.9 101.6 0)
 			(effects
@@
 			(project "frank_rm2"
 				(path "/8c0b3d8b-46d3-4173-ab1e-a61765f77d61/8f57fa0b-80dc-4c8c-9148-33c48d230b70"
-					(reference "#PWR031")
+					(reference "#PWR044")
 					(unit 1)
 				)
@@
 		(dnp no)
 		(fields_autoplaced yes)
-		(property "Reference" "#PWR032"
+		(property "Reference" "#PWR045"
 			(at 226.06 104.14 0)
 			(effects
@@
 			(project "frank_rm2"
 				(path "/8c0b3d8b-46d3-4173-ab1e-a61765f77d61/8f57fa0b-80dc-4c8c-9148-33c48d230b70"
-					(reference "#PWR032")
+					(reference "#PWR045")
 					(unit 1)
 				)

Commit message: FRANK One WIP
Parts:
- renumbered C3 to C2, J9 to J8, R11 to R6, R12 to R7, R13 to R8, U2 to U1
Connections:
- no-connect marks 4 -> 5
Changed lines of the file:
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@@
+	)
+	(no_connect
+		(at 85.09 96.52)
 	)
 	(no_connect
@@
 		(on_board yes)
 		(dnp no)
-		(property "Reference" "R12"
+		(property "Reference" "R7"
 			(at 119.634 105.156 90)
 			(effects
@@
 			(project "frank_rm2"
 				(path "/8c0b3d8b-46d3-4173-ab1e-a61765f77d61/8f57fa0b-80dc-4c8c-9148-33c48d230b70"
-					(reference "R12")
+					(reference "R7")
 					(unit 1)
 				)
@@
 		(dnp no)
 		(fields_autoplaced yes)
-		(property "Reference" "#PWR043"
+		(property "Reference" "#PWR034"
 			(at 140.97 116.84 0)
 			(effects
@@
 			(project "frank_rm2"
 				(path "/8c0b3d8b-46d3-4173-ab1e-a61765f77d61/8f57fa0b-80dc-4c8c-9148-33c48d230b70"
-					(reference "#PWR043")
+					(reference "#PWR034")
 					(unit 1)
 				)
@@
 		(dnp no)
 		(fields_autoplaced yes)
-		(property "Reference" "#PWR047"
+		(property "Reference" "#PWR038"
 			(at 226.06 114.3 0)
 			(effects
@@
 			(project "frank_rm2"
 				(path "/8c0b3d8b-46d3-4173-ab1e-a61765f77d61/8f57fa0b-80dc-4c8c-9148-33c48d230b70"
-					(reference "#PWR047")
+					(reference "#PWR038")
 					(unit 1)
 				)
@@
 		(dnp no)
 		(fields_autoplaced yes)
-		(property "Reference" "#PWR046"
+		(property "Reference" "#PWR037"
 			(at 226.06 109.22 0)
 			(effects
@@
 			(project "frank_rm2"
 				(path "/8c0b3d8b-46d3-4173-ab1e-a61765f77d61/8f57fa0b-80dc-4c8c-9148-33c48d230b70"
-					(reference "#PWR046")
+					(reference "#PWR037")
 					(unit 1)
 				)
@@
 		(dnp no)
 		(fields_autoplaced yes)
-		(property "Reference" "U2"
+		(property "Reference" "U1"
 			(at 185.42 91.44 0)
 			(effects
@@
 			(project "frank_rm2"
 				(path "/8c0b3d8b-46d3-4173-ab1e-a61765f77d61/8f57fa0b-80dc-4c8c-9148-33c48d230b70"
-					(reference "U2")
+					(reference "U1")
 					(unit 1)
 				)
@@
 		(on_board yes)
 		(dnp no)
-		(property "Reference" "J9"
+		(property "Reference" "J8"
 			(at 72.8981 101.4003 0)
 			(effects
@@
 			)
 		)
-		(property "Datasheet" "https://www.lcsc.com/datasheet/lcsc_datasheet_1810121716_Korean-Hroparts-Elec-PJ-320D-4A_C95562.pdf"
+		(property "Datasheet" "~"
 			(at 80.01 105.41 0)
 			(effects
@@
 		)
 		(pin "T"
+		)
+		(pin "RN"
 		)
 		(instances
@@
 			(project "minifrank_rm1"
 				(path "/8c0b3d8b-46d3-4173-ab1e-a61765f77d61/8f57fa0b-80dc-4c8c-9148-33c48d230b70"
-					(reference "J9")
+					(reference "J8")
 					(unit 1)
 				)
@@
 		(dnp no)
 		(fields_autoplaced yes)
-		(property "Reference" "#PWR042"
+		(property "Reference" "#PWR033"
 			(at 91.44 107.95 0)
 			(effects
@@
 			(project "minifrank_rm1"
 				(path "/8c0b3d8b-46d3-4173-ab1e-a61765f77d61/8f57fa0b-80dc-4c8c-9148-33c48d230b70"
-					(reference "#PWR042")
+					(reference "#PWR033")
 					(unit 1)
 				)
@@
 		(on_board yes)
 		(dnp no)
-		(property "Reference" "#PWR044"
+		(property "Reference" "#PWR035"
 			(at 215.9 101.6 0)
 			(effects
@@
 			(project "frank_rm2"
 				(path "/8c0b3d8b-46d3-4173-ab1e-a61765f77d61/8f57fa0b-80dc-4c8c-9148-33c48d230b70"
-					(reference "#PWR044")
+					(reference "#PWR035")
 					(unit 1)
 				)
@@
 		(dnp no)
 		(fields_autoplaced yes)
-		(property "Reference" "#PWR045"
+		(property "Reference" "#PWR036"
 			(at 226.06 104.14 0)
 			(effects
@@
 			(project "frank_rm2"
 				(path "/8c0b3d8b-46d3-4173-ab1e-a61765f77d61/8f57fa0b-80dc-4c8c-9148-33c48d230b70"
-					(reference "#PWR045")
+					(reference "#PWR036")
 					(unit 1)
 				)
@@
 		(on_board yes)
 		(dnp no)
-		(property "Reference" "C3"
+		(property "Reference" "C2"
 			(at 118.999 91.3384 0)
 			(effects
@@
 			(project "frank_rm2"
 				(path "/8c0b3d8b-46d3-4173-ab1e-a61765f77d61/8f57fa0b-80dc-4c8c-9148-33c48d230b70"
-					(reference "C3")
+					(reference "C2")
 					(unit 1)
 				)
@@
 		(on_board yes)
 		(dnp no)
-		(property "Reference" "R11"
+		(property "Reference" "R6"
 			(at 119.634 97.536 90)
 			(effects
@@
 			(project "frank_rm2"
 				(path "/8c0b3d8b-46d3-4173-ab1e-a61765f77d61/8f57fa0b-80dc-4c8c-9148-33c48d230b70"
-					(reference "R11")
+					(reference "R6")
 					(unit 1)
 				)
@@
 		(on_board yes)
 		(dnp no)
-		(property "Reference" "R13"
+		(property "Reference" "R8"
 			(at 119.634 112.776 90)
 			(effects
@@
 			(project "frank_rm2"
 				(path "/8c0b3d8b-46d3-4173-ab1e-a61765f77d61/8f57fa0b-80dc-4c8c-9148-33c48d230b70"
-					(reference "R13")
+					(reference "R8")
 					(unit 1)
 				)

Commit message: FRANK One WIP
Parts:
- renumbered J8 to J9
Changed lines of the file:
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@@
 		(on_board yes)
 		(dnp no)
-		(property "Reference" "J8"
+		(property "Reference" "J9"
 			(at 72.8981 101.4003 0)
 			(effects
@@
 			(project "minifrank_rm1"
 				(path "/8c0b3d8b-46d3-4173-ab1e-a61765f77d61/8f57fa0b-80dc-4c8c-9148-33c48d230b70"
-					(reference "J8")
+					(reference "J9")
 					(unit 1)
 				)
