File: lab/frank_one_rm2/frank_one_rm2.kicad_sch (KiCad schematic)
At the start: 14 parts, among them J1 PWR

Commit message: Board updates
Parts:
- added J1: EXT Sound, FRANK:PinHeader_2x10_P2.54mm_Vertical, symbol Connector_Generic:Conn_02x10_Odd_Even
- added JP4: MONO, FRANK:Pin Header (1x02), symbol Connector:Conn_01x02_Pin
- JP2: footprint FRANK:SW_DS05-127-2-04BK-SMT-TR -> FRANK:SW_DS05-127-2-05BK-SMT-TR
- renumbered J1 to J2
Connections:
- net +3V3: now also J1.19 (Pin_19)
- net AMP_OUT_L: now also J1.13 (Pin_13)
- net AMP_OUT_R: now also J1.15 (Pin_15)
- net GND: now also J1.10 (Pin_10), J1.12 (Pin_12), J1.14 (Pin_14), J1.16 (Pin_16), J1.18 (Pin_18), J1.2 (Pin_2), J1.20 (Pin_20), J1.4 (Pin_4), J1.6 (Pin_6), J1.8 (Pin_8)
- net MONO_L: now also JP4.1 (Pin_1); no longer JP2.3
- net MONO_R: now also JP4.2 (Pin_2); no longer JP2.6
- net PSW: now also JP2.3; no longer JP2.2
- net RP1_GPIO10: now also J1.9 (Pin_9)
- net RP1_GPIO11: now also J1.7 (Pin_7)
- net RP1_GPIO22: now also J1.17 (Pin_17)
- net RP1_GPIO9: now also J1.11 (Pin_11)
- net VBUS: now also JP2.6, J1.1 (Pin_1)
- net ASW renamed J_TDA
- new net EXT_L: J1.3 (Pin_3)
- new net EXT_R: J1.5 (Pin_5)
- new net J_EXT: JP2.2
Other:
- sheet Audio Multiplexer ports: added EXT_L, EXT_R, J_EXT, J_TDA; removed AUDIOSW

Commit message: FRANK One RM2 HW 1.01
Connections:
- net RP1_GPIO0: now also R1.1
- net RP1_GPIO1: now also R2.1
- net RP1_GPIO2: now also R3.1
- net RP1_GPIO3: now also R4.1
- net RP2_GPIO11: no longer R1.1
- net RP2_GPIO12: no longer R2.1
- net RP2_GPIO14: no longer R3.1
- net RP2_GPIO15: no longer R4.1
Changed lines of the file:
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@@
 		)
 	)
-	(label "RP2_GPIO11"
+	(label "RP1_GPIO0"
 		(at 207.01 129.54 90)
 		(effects
@@
 		)
 	)
-	(label "RP2_GPIO12"
+	(label "RP1_GPIO1"
 		(at 215.9 129.54 90)
 		(effects
@@
 		)
 	)
-	(label "RP2_GPIO15"
+	(label "RP1_GPIO3"
 		(at 233.68 129.54 90)
 		(effects
@@
 		)
 	)
-	(label "RP2_GPIO14"
+	(label "RP1_GPIO2"
 		(at 224.79 129.54 90)
 		(effects
@@
 		(dnp no)
 		(fields_autoplaced yes)
-		(property "Reference" "#PWR021"
+		(property "Reference" "#PWR025"
 			(at 231.14 88.9 0)
 			(effects
@@
 			(project "minifrank_rm1"
 				(path "/8c0b3d8b-46d3-4173-ab1e-a61765f77d61"
-					(reference "#PWR021")
+					(reference "#PWR025")
 					(unit 1)
 				)
@@
 		(dnp no)
 		(fields_autoplaced yes)
-		(property "Reference" "#PWR022"
+		(property "Reference" "#PWR017"
 			(at 219.71 35.56 0)
 			(effects
@@
 			(project ""
 				(path "/8c0b3d8b-46d3-4173-ab1e-a61765f77d61"
-					(reference "#PWR022")
+					(reference "#PWR017")
 					(unit 1)
 				)
@@
 		(dnp no)
 		(fields_autoplaced yes)
-		(property "Reference" "#PWR024"
+		(property "Reference" "#PWR019"
 			(at 219.71 40.64 0)
 			(effects
@@
 			(project "frank_one_rm2"
 				(path "/8c0b3d8b-46d3-4173-ab1e-a61765f77d61"
-					(reference "#PWR024")
+					(reference "#PWR019")
 					(unit 1)
 				)
@@
 		(dnp no)
 		(fields_autoplaced yes)
-		(property "Reference" "#PWR025"
+		(property "Reference" "#PWR020"
 			(at 229.87 43.18 0)
 			(effects
@@
 			(project "minifrank_rm1p2h"
 				(path "/8c0b3d8b-46d3-4173-ab1e-a61765f77d61"
-					(reference "#PWR025")
+					(reference "#PWR020")
 					(unit 1)
 				)
@@
 		(on_board yes)
 		(dnp no)
-		(property "Reference" "#PWR018"
+		(property "Reference" "#PWR022"
 			(at 233.68 113.03 0)
 			(effects
@@
 			(project "frank_one"
 				(path "/8c0b3d8b-46d3-4173-ab1e-a61765f77d61"
-					(reference "#PWR018")
+					(reference "#PWR022")
 					(unit 1)
 				)
@@
 		(dnp no)
 		(fields_autoplaced yes)
-		(property "Reference" "#PWR023"
+		(property "Reference" "#PWR018"
 			(at 219.71 38.1 0)
 			(effects
@@
 			(project "frank_one_rm2"
 				(path "/8c0b3d8b-46d3-4173-ab1e-a61765f77d61"
-					(reference "#PWR023")
+					(reference "#PWR018")
 					(unit 1)
 				)
@@
 		(on_board yes)
 		(dnp no)
-		(property "Reference" "#PWR017"
+		(property "Reference" "#PWR021"
 			(at 224.79 113.03 0)
 			(effects
@@
 			(project "frank_one"
 				(path "/8c0b3d8b-46d3-4173-ab1e-a61765f77d61"
-					(reference "#PWR017")
+					(reference "#PWR021")
 					(unit 1)
 				)
@@
 		(dnp no)
 		(fields_autoplaced yes)
-		(property "Reference" "#PWR019"
+		(property "Reference" "#PWR023"
 			(at 231.14 83.82 0)
 			(effects
@@
 			(project "minifrank_rm1"
 				(path "/8c0b3d8b-46d3-4173-ab1e-a61765f77d61"
-					(reference "#PWR019")
+					(reference "#PWR023")
 					(unit 1)
 				)
@@
 		(dnp no)
 		(fields_autoplaced yes)
-		(property "Reference" "#PWR020"
+		(property "Reference" "#PWR024"
 			(at 241.3 86.36 0)
 			(effects
@@
 			(project "minifrank_rm1"
 				(path "/8c0b3d8b-46d3-4173-ab1e-a61765f77d61"
-					(reference "#PWR020")
+					(reference "#PWR024")
 					(unit 1)
 				)

Commit message: Board updates
Parts:
- R1, R2, R3, R4: value 10K -> 4.7K
Other:
- moved on the sheet: H1, H2, H3, H4, J1, J2, JP1, JP3, JP4, R1, R2, R3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

Commit message: FRANK One WIP
Parts:
- removed JP4: MONO, FRANK:Pin Header (1x02), symbol Connector:Conn_01x02_Pin
- added JP1: UART, FRANK:Pin Header (1x03), symbol Connector:Conn_01x03_Pin
- JP2: footprint FRANK:SW_DS05-127-2-05BK-SMT-TR -> FRANK:DS05127208BKSMTTR; symbol Switch:SW_DIP_x04 -> Switch:SW_DIP_x08
- renumbered JP1 to JP3, JP3 to JP4
Connections:
- net PSW is gone; now on net SHND: JP2.3
- net +3V3: now also JP2.11; no longer R1.2, R2.2, R3.2, R4.2
- net GND: now also JP2.12, JP2.9, JP1.3 (Pin_3); no longer JP2.5
- net MONO_L: now also JP2.4
- net MONO_R: now also JP2.13
- net RP1_GPIO0: now also JP1.1 (Pin_1)
- net RP1_GPIO1: now also JP1.2 (Pin_2)
- net RP2_RUN: now also JP2.8
- net SHND: no longer JP2.4
- net VBUS: now also JP2.10, JP2.14, JP2.15, JP2.16; no longer JP2.6, JP2.7, JP2.8
- new net PUP3V3: JP2.6, R1.2, R2.2, R3.2, R4.2
- new net PUP5V: JP2.7
- new net VGA_BR: JP2.5
Other:
- removed sheet PS2 Mutliplexer
- removed sheet USB C 1
- removed sheet USB C 2
- added sheet Power (pwr_2usb.kicad_sch)
- sheet PS2 ports: added PUP5V; removed none
- sheet VGA ports: added VGA_BR; removed none
- moved on the sheet: J2, R1, R2, R3, R4, S1, S2

Commit message: FRANK One WIP
Parts:
- renumbered JP1 to J2, J2 to J3, JP2 to JP1, JP3 to JP2, JP4 to JP3
Changed lines of the file:
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@@
 		(dnp no)
 		(fields_autoplaced yes)
-		(property "Reference" "J2"
+		(property "Reference" "J3"
 			(at 217.805 64.77 0)
 			(effects
@@
 			(project "minifrank_rm1"
 				(path "/8c0b3d8b-46d3-4173-ab1e-a61765f77d61"
-					(reference "J2")
+					(reference "J3")
 					(unit 1)
 				)
@@
 		(dnp no)
 		(fields_autoplaced yes)
-		(property "Reference" "JP1"
+		(property "Reference" "J2"
 			(at 194.945 64.77 0)
 			(effects
@@
 			(project "frank_one_rm2"
 				(path "/8c0b3d8b-46d3-4173-ab1e-a61765f77d61"
-					(reference "JP1")
+					(reference "J2")
 					(unit 1)
 				)
@@
 		(dnp no)
 		(fields_autoplaced yes)
-		(property "Reference" "JP3"
+		(property "Reference" "JP2"
 			(at 250.825 27.94 0)
 			(effects
@@
 			(project "frank_one_rm2"
 				(path "/8c0b3d8b-46d3-4173-ab1e-a61765f77d61"
-					(reference "JP3")
+					(reference "JP2")
 					(unit 1)
 				)
@@
 		(dnp no)
 		(fields_autoplaced yes)
-		(property "Reference" "JP4"
+		(property "Reference" "JP3"
 			(at 250.825 41.91 0)
 			(effects
@@
 			(project "frank_one_rm2"
 				(path "/8c0b3d8b-46d3-4173-ab1e-a61765f77d61"
-					(reference "JP4")
+					(reference "JP3")
 					(unit 1)
 				)
@@
 		(on_board yes)
 		(dnp no)
-		(property "Reference" "JP2"
+		(property "Reference" "JP1"
 			(at 210.566 26.67 0)
 			(effects
@@
 			(project "frank_one_rm2"
 				(path "/8c0b3d8b-46d3-4173-ab1e-a61765f77d61"
-					(reference "JP2")
+					(reference "JP1")
 					(unit 1)
 				)

Commit message: FRANK One RM2 HW 1.03
Parts:
- added J19: DEBUG, FRANK:Pin Header (1x03), symbol Connector:Conn_01x03_Pin
Connections:
- net +3V3: no longer JP1.11
- net GND: now also JP1.14, J19.3 (Pin_3)
- net RP1_SWCLK: now also J19.1 (Pin_1)
- net RP1_SWD: now also J19.2 (Pin_2)
- net VBUS: no longer JP1.14
- new net +3V3_2350: JP1.11
- no-connect marks 32 -> 30
Other:
- moved on the sheet: J1, J2, J3, JP2, JP3, R1, R2, R3, R4, S1, S2
