File: lab/frank_one_rm2/usbstack.kicad_sch (KiCad schematic)
At the start: 7 parts, among them J11 SS-52100-004

Commit message: Board updates
Parts:
- renumbered J11 to J12
Changed lines of the file:
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@@
 		(dnp no)
 		(fields_autoplaced yes)
-		(property "Reference" "J11"
+		(property "Reference" "J12"
 			(at 121.92 68.58 0)
 			(effects
@@
 			(project "turbofrank"
 				(path "/8c0b3d8b-46d3-4173-ab1e-a61765f77d61/9f9f8cbe-7394-4892-9c0f-378226b1a9ff"
-					(reference "J11")
+					(reference "J12")
 					(unit 1)
 				)
@@
 		(on_board yes)
 		(dnp no)
-		(property "Reference" "#PWR053"
+		(property "Reference" "#PWR066"
 			(at 135.89 78.74 0)
 			(effects
@@
 			(project "turbofrank"
 				(path "/8c0b3d8b-46d3-4173-ab1e-a61765f77d61/9f9f8cbe-7394-4892-9c0f-378226b1a9ff"
-					(reference "#PWR053")
+					(reference "#PWR066")
 					(unit 1)
 				)
@@
 		(on_board yes)
 		(dnp no)
-		(property "Reference" "#PWR055"
+		(property "Reference" "#PWR068"
 			(at 165.1 95.25 0)
 			(effects
@@
 			(project "turbofrank"
 				(path "/8c0b3d8b-46d3-4173-ab1e-a61765f77d61/9f9f8cbe-7394-4892-9c0f-378226b1a9ff"
-					(reference "#PWR055")
+					(reference "#PWR068")
 					(unit 1)
 				)
@@
 		(on_board yes)
 		(dnp no)
-		(property "Reference" "#PWR056"
+		(property "Reference" "#PWR069"
 			(at 176.53 95.25 0)
 			(effects
@@
 			(project "turbofrank"
 				(path "/8c0b3d8b-46d3-4173-ab1e-a61765f77d61/9f9f8cbe-7394-4892-9c0f-378226b1a9ff"
-					(reference "#PWR056")
+					(reference "#PWR069")
 					(unit 1)
 				)
@@
 		(on_board yes)
 		(dnp no)
-		(property "Reference" "#PWR054"
+		(property "Reference" "#PWR067"
 			(at 142.24 78.74 0)
 			(effects
@@
 			(project "turbofrank"
 				(path "/8c0b3d8b-46d3-4173-ab1e-a61765f77d61/9f9f8cbe-7394-4892-9c0f-378226b1a9ff"
-					(reference "#PWR054")
+					(reference "#PWR067")
 					(unit 1)
 				)
@@
 		(dnp no)
 		(fields_autoplaced yes)
-		(property "Reference" "#PWR052"
+		(property "Reference" "#PWR065"
 			(at 121.92 111.76 0)
 			(effects
@@
 			(project "turbofrank"
 				(path "/8c0b3d8b-46d3-4173-ab1e-a61765f77d61/9f9f8cbe-7394-4892-9c0f-378226b1a9ff"
-					(reference "#PWR052")
+					(reference "#PWR065")
 					(unit 1)
 				)

Commit message: FRANK One WIP
Parts:
- renumbered C6 to C3, C7 to C4, J12 to J10, R21 to R10, R22 to R11, R23 to R12, R24 to R13
Changed lines of the file:
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@@
 		(dnp no)
 		(fields_autoplaced yes)
-		(property "Reference" "J12"
+		(property "Reference" "J10"
 			(at 121.92 68.58 0)
 			(effects
@@
 			(project "turbofrank"
 				(path "/8c0b3d8b-46d3-4173-ab1e-a61765f77d61/9f9f8cbe-7394-4892-9c0f-378226b1a9ff"
-					(reference "J12")
+					(reference "J10")
 					(unit 1)
 				)
@@
 		(on_board yes)
 		(dnp no)
-		(property "Reference" "C6"
+		(property "Reference" "C3"
 			(at 168.021 82.6516 0)
 			(effects
@@
 			(project "turbofrank"
 				(path "/8c0b3d8b-46d3-4173-ab1e-a61765f77d61/9f9f8cbe-7394-4892-9c0f-378226b1a9ff"
-					(reference "C6")
+					(reference "C3")
 					(unit 1)
 				)
@@
 		(on_board yes)
 		(dnp no)
-		(property "Reference" "R22"
+		(property "Reference" "R11"
 			(at 145.542 104.14 90)
 			(effects
@@
 			(project "turbofrank"
 				(path "/8c0b3d8b-46d3-4173-ab1e-a61765f77d61/9f9f8cbe-7394-4892-9c0f-378226b1a9ff"
-					(reference "R22")
+					(reference "R11")
 					(unit 1)
 				)
@@
 		(on_board yes)
 		(dnp no)
-		(property "Reference" "C7"
+		(property "Reference" "C4"
 			(at 179.451 82.6516 0)
 			(effects
@@
 			(project "turbofrank"
 				(path "/8c0b3d8b-46d3-4173-ab1e-a61765f77d61/9f9f8cbe-7394-4892-9c0f-378226b1a9ff"
-					(reference "C7")
+					(reference "C4")
 					(unit 1)
 				)
@@
 		(on_board yes)
 		(dnp no)
-		(property "Reference" "#PWR066"
+		(property "Reference" "#PWR043"
 			(at 135.89 78.74 0)
 			(effects
@@
 			(project "turbofrank"
 				(path "/8c0b3d8b-46d3-4173-ab1e-a61765f77d61/9f9f8cbe-7394-4892-9c0f-378226b1a9ff"
-					(reference "#PWR066")
+					(reference "#PWR043")
 					(unit 1)
 				)
@@
 		(on_board yes)
 		(dnp no)
-		(property "Reference" "#PWR068"
+		(property "Reference" "#PWR045"
 			(at 165.1 95.25 0)
 			(effects
@@
 			(project "turbofrank"
 				(path "/8c0b3d8b-46d3-4173-ab1e-a61765f77d61/9f9f8cbe-7394-4892-9c0f-378226b1a9ff"
-					(reference "#PWR068")
+					(reference "#PWR045")
 					(unit 1)
 				)
@@
 		(on_board yes)
 		(dnp no)
-		(property "Reference" "R23"
+		(property "Reference" "R12"
 			(at 154.432 102.87 90)
 			(effects
@@
 			(project "turbofrank"
 				(path "/8c0b3d8b-46d3-4173-ab1e-a61765f77d61/9f9f8cbe-7394-4892-9c0f-378226b1a9ff"
-					(reference "R23")
+					(reference "R12")
 					(unit 1)
 				)
@@
 		(on_board yes)
 		(dnp no)
-		(property "Reference" "#PWR069"
+		(property "Reference" "#PWR046"
 			(at 176.53 95.25 0)
 			(effects
@@
 			(project "turbofrank"
 				(path "/8c0b3d8b-46d3-4173-ab1e-a61765f77d61/9f9f8cbe-7394-4892-9c0f-378226b1a9ff"
-					(reference "#PWR069")
+					(reference "#PWR046")
 					(unit 1)
 				)
@@
 		(on_board yes)
 		(dnp no)
-		(property "Reference" "R21"
+		(property "Reference" "R10"
 			(at 141.732 97.79 90)
 			(effects
@@
 			(project "turbofrank"
 				(path "/8c0b3d8b-46d3-4173-ab1e-a61765f77d61/9f9f8cbe-7394-4892-9c0f-378226b1a9ff"
-					(reference "R21")
+					(reference "R10")
 					(unit 1)
 				)
@@
 		(on_board yes)
 		(dnp no)
-		(property "Reference" "#PWR067"
+		(property "Reference" "#PWR044"
 			(at 142.24 78.74 0)
 			(effects
@@
 			(project "turbofrank"
 				(path "/8c0b3d8b-46d3-4173-ab1e-a61765f77d61/9f9f8cbe-7394-4892-9c0f-378226b1a9ff"
-					(reference "#PWR067")
+					(reference "#PWR044")
 					(unit 1)
 				)
@@
 		(dnp no)
 		(fields_autoplaced yes)
-		(property "Reference" "#PWR065"
+		(property "Reference" "#PWR042"
 			(at 121.92 111.76 0)
 			(effects
@@
 			(project "turbofrank"
 				(path "/8c0b3d8b-46d3-4173-ab1e-a61765f77d61/9f9f8cbe-7394-4892-9c0f-378226b1a9ff"
-					(reference "#PWR065")
+					(reference "#PWR042")
 					(unit 1)
 				)
@@
 		(on_board yes)
 		(dnp no)
-		(property "Reference" "R24"
+		(property "Reference" "R13"
 			(at 158.242 109.22 90)
 			(effects
@@
 			(project "turbofrank"
 				(path "/8c0b3d8b-46d3-4173-ab1e-a61765f77d61/9f9f8cbe-7394-4892-9c0f-378226b1a9ff"
-					(reference "R24")
+					(reference "R13")
 					(unit 1)
 				)

Commit message: FRANK One WIP
Parts:
- renumbered J10 to J11
Changed lines of the file:
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@@
 		(dnp no)
 		(fields_autoplaced yes)
-		(property "Reference" "J10"
+		(property "Reference" "J11"
 			(at 121.92 68.58 0)
 			(effects
@@
 			(project "turbofrank"
 				(path "/8c0b3d8b-46d3-4173-ab1e-a61765f77d61/9f9f8cbe-7394-4892-9c0f-378226b1a9ff"
-					(reference "J10")
+					(reference "J11")
 					(unit 1)
 				)

Commit message: FRANK One RM2 HW 1.03
Other:
- moved on the sheet: C3, C4, J11, R10, R11, R12, R13
