File: hardware/frank_m1/gamepad.kicad_sch (KiCad schematic)
At the start: 3 parts, among them J7 D-SUB 9 Male

Commit message: FRANK M1 2.03 & xt8086 WIP
Parts:
- R27: renamed from R12; footprint FRANK:Resistor (0805) -> FRANK:R_0805_2012Metric
- renumbered D5 to D1, J7 to J6
Other:
- title: FRANK M1 -> ${NAME} ${MODEL}
- moved on the sheet: D1, J6, R27

Commit message: FRANK M1 WIP
Parts:
- renumbered D1 to D3, J6 to J13, R27 to R67
Other:
- title: ${NAME} ${MODEL} -> ${NAME} ${VARIANT}
Changed lines of the file:
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@@
 	(paper "A4")
 	(title_block
-		(title "${NAME} ${MODEL}")
+		(title "${NAME} ${VARIANT}")
 		(date "${DATE}")
 		(rev "${VERSION}")
@@
 		(on_board yes)
 		(dnp no)
-		(property "Reference" "#PWR054"
+		(property "Reference" "#PWR0119"
 			(at 147.32 119.38 0)
 			(effects
@@
 		)
 		(instances
-			(project ""
-				(path "/8c0b3d8b-46d3-4173-ab1e-a61765f77d61/91039a09-82d7-4099-8414-fc5647ada98f"
-					(reference "#PWR054")
-					(unit 1)
-				)
-				(path "/8c0b3d8b-46d3-4173-ab1e-a61765f77d61/e9da9b3c-e9c6-4677-bc99-391052f7625b"
-					(reference "#PWR057")
+			(project "frank_m1"
+				(path "/8c0b3d8b-46d3-4173-ab1e-a61765f77d61/b085e7bf-95c6-4d62-b8ec-fd94d25a70e5"
+					(reference "#PWR0119")
+					(unit 1)
+				)
+				(path "/8c0b3d8b-46d3-4173-ab1e-a61765f77d61/c50ad372-63d4-4886-82fc-368d1bd37a5f"
+					(reference "#PWR0122")
 					(unit 1)
 				)
@@
 		(on_board yes)
 		(dnp no)
-		(property "Reference" "D1"
+		(property "Reference" "D3"
 			(at 144.78 109.22 0)
 			(effects
@@
 		)
 		(instances
-			(project ""
-				(path "/8c0b3d8b-46d3-4173-ab1e-a61765f77d61/91039a09-82d7-4099-8414-fc5647ada98f"
-					(reference "D1")
-					(unit 1)
-				)
-				(path "/8c0b3d8b-46d3-4173-ab1e-a61765f77d61/e9da9b3c-e9c6-4677-bc99-391052f7625b"
-					(reference "D2")
+			(project "frank_m1"
+				(path "/8c0b3d8b-46d3-4173-ab1e-a61765f77d61/b085e7bf-95c6-4d62-b8ec-fd94d25a70e5"
+					(reference "D3")
+					(unit 1)
+				)
+				(path "/8c0b3d8b-46d3-4173-ab1e-a61765f77d61/c50ad372-63d4-4886-82fc-368d1bd37a5f"
+					(reference "D4")
 					(unit 1)
 				)
@@
 		(dnp no)
 		(fields_autoplaced yes)
-		(property "Reference" "#PWR055"
+		(property "Reference" "#PWR0120"
 			(at 160.02 102.87 0)
 			(effects
@@
 		)
 		(instances
-			(project ""
-				(path "/8c0b3d8b-46d3-4173-ab1e-a61765f77d61/91039a09-82d7-4099-8414-fc5647ada98f"
-					(reference "#PWR055")
-					(unit 1)
-				)
-				(path "/8c0b3d8b-46d3-4173-ab1e-a61765f77d61/e9da9b3c-e9c6-4677-bc99-391052f7625b"
-					(reference "#PWR058")
+			(project "frank_m1"
+				(path "/8c0b3d8b-46d3-4173-ab1e-a61765f77d61/b085e7bf-95c6-4d62-b8ec-fd94d25a70e5"
+					(reference "#PWR0120")
+					(unit 1)
+				)
+				(path "/8c0b3d8b-46d3-4173-ab1e-a61765f77d61/c50ad372-63d4-4886-82fc-368d1bd37a5f"
+					(reference "#PWR0123")
 					(unit 1)
 				)
@@
 		(on_board yes)
 		(dnp no)
-		(property "Reference" "J6"
+		(property "Reference" "J13"
 			(at 177.8 86.36 0)
 			(effects
@@
 		)
 		(instances
-			(project ""
-				(path "/8c0b3d8b-46d3-4173-ab1e-a61765f77d61/91039a09-82d7-4099-8414-fc5647ada98f"
-					(reference "J6")
-					(unit 1)
-				)
-				(path "/8c0b3d8b-46d3-4173-ab1e-a61765f77d61/e9da9b3c-e9c6-4677-bc99-391052f7625b"
-					(reference "J7")
+			(project "frank_m1"
+				(path "/8c0b3d8b-46d3-4173-ab1e-a61765f77d61/b085e7bf-95c6-4d62-b8ec-fd94d25a70e5"
+					(reference "J13")
+					(unit 1)
+				)
+				(path "/8c0b3d8b-46d3-4173-ab1e-a61765f77d61/c50ad372-63d4-4886-82fc-368d1bd37a5f"
+					(reference "J14")
 					(unit 1)
 				)
@@
 		(dnp no)
 		(fields_autoplaced yes)
-		(property "Reference" "#PWR056"
+		(property "Reference" "#PWR0121"
 			(at 154.94 96.52 0)
 			(effects
@@
 		)
 		(instances
-			(project ""
-				(path "/8c0b3d8b-46d3-4173-ab1e-a61765f77d61/91039a09-82d7-4099-8414-fc5647ada98f"
-					(reference "#PWR056")
-					(unit 1)
-				)
-				(path "/8c0b3d8b-46d3-4173-ab1e-a61765f77d61/e9da9b3c-e9c6-4677-bc99-391052f7625b"
-					(reference "#PWR059")
+			(project "frank_m1"
+				(path "/8c0b3d8b-46d3-4173-ab1e-a61765f77d61/b085e7bf-95c6-4d62-b8ec-fd94d25a70e5"
+					(reference "#PWR0121")
+					(unit 1)
+				)
+				(path "/8c0b3d8b-46d3-4173-ab1e-a61765f77d61/c50ad372-63d4-4886-82fc-368d1bd37a5f"
+					(reference "#PWR0124")
 					(unit 1)
 				)
@@
 		(on_board yes)
 		(dnp no)
-		(property "Reference" "R27"
+		(property "Reference" "R67"
 			(at 149.86 101.6 90)
 			(effects
@@
 		)
 		(instances
-			(project ""
-				(path "/8c0b3d8b-46d3-4173-ab1e-a61765f77d61/91039a09-82d7-4099-8414-fc5647ada98f"
-					(reference "R27")
-					(unit 1)
-				)
-				(path "/8c0b3d8b-46d3-4173-ab1e-a61765f77d61/e9da9b3c-e9c6-4677-bc99-391052f7625b"
-					(reference "R28")
-					(unit 1)
-				)
+			(project "frank_m1"
+				(path "/8c0b3d8b-46d3-4173-ab1e-a61765f77d61/b085e7bf-95c6-4d62-b8ec-fd94d25a70e5"
+					(reference "R67")
+					(unit 1)
+				)
+				(path "/8c0b3d8b-46d3-4173-ab1e-a61765f77d61/c50ad372-63d4-4886-82fc-368d1bd37a5f"
+					(reference "R68")
+					(unit 1)
+				)

Commit message: FRANK M1 2.04
Parts:
- R67: symbol Device:R -> FRANK:R
Other:
- title: ${NAME} ${VARIANT} -> ${NAME} ${MODEL}
Changed lines of the file:
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@@
 	(paper "A4")
 	(title_block
-		(title "${NAME} ${VARIANT}")
+		(title "${NAME} ${MODEL}")
 		(date "${DATE}")
 		(rev "${VERSION}")
@@
 	)
 	(symbol
-		(lib_id "Device:R")
+		(lib_id "FRANK:R")
 		(at 152.4 104.14 90)
 		(unit 1)
