File: hardware/frank_m1/vga.kicad_sch (KiCad schematic)
At the start: 9 parts, among them J13 D-SUB 15 Female

Commit message: FRANK M1 2.03 & xt8086 WIP
Parts:
- R57: renamed from R37; footprint FRANK:Resistor (0805) -> FRANK:R_0805_2012Metric
- R58: renamed from R38; footprint FRANK:Resistor (0805) -> FRANK:R_0805_2012Metric
- R59: renamed from R39; footprint FRANK:Resistor (0805) -> FRANK:R_0805_2012Metric
- R60: renamed from R40; footprint FRANK:Resistor (0805) -> FRANK:R_0805_2012Metric
- R61: renamed from R41; footprint FRANK:Resistor (0805) -> FRANK:R_0805_2012Metric
- R62: renamed from R42; footprint FRANK:Resistor (0805) -> FRANK:R_0805_2012Metric
- R63: renamed from R43; footprint FRANK:Resistor (0805) -> FRANK:R_0805_2012Metric
- R64: renamed from R44; footprint FRANK:Resistor (0805) -> FRANK:R_0805_2012Metric
- renumbered J13 to J14
Other:
- title: FRANK M1 -> ${NAME} ${MODEL}
- moved on the sheet: J14, R57, R58, R59, R60, R61, R62, R63, R64

Commit message: FRANK M1 WIP
Parts:
- renumbered J14 to J17, R57 to R73, R58 to R74, R59 to R75, R60 to R76, R61 to R77, R62 to R78, R63 to R79, R64 to R80
Other:
- title: ${NAME} ${MODEL} -> ${NAME} ${VARIANT}
Changed lines of the file:
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@@
 	(paper "A4")
 	(title_block
-		(title "${NAME} ${MODEL}")
+		(title "${NAME} ${VARIANT}")
 		(date "${DATE}")
 		(rev "${VERSION}")
@@
 		(on_board yes)
 		(dnp no)
-		(property "Reference" "R59"
+		(property "Reference" "R75"
 			(at 101.6 85.09 90)
 			(effects
@@
 		)
 		(instances
-			(project "turbofrank"
-				(path "/8c0b3d8b-46d3-4173-ab1e-a61765f77d61/24602416-4859-4434-98d4-6bf9d7e9b6c1"
-					(reference "R59")
+			(project "frank_m1"
+				(path "/8c0b3d8b-46d3-4173-ab1e-a61765f77d61/522a66a4-10b2-43ba-99ce-6cab39134d52"
+					(reference "R75")
 					(unit 1)
 				)
@@
 		(on_board yes)
 		(dnp no)
-		(property "Reference" "R64"
+		(property "Reference" "R80"
 			(at 184.15 106.68 90)
 			(effects
@@
 		)
 		(instances
-			(project "turbofrank"
-				(path "/8c0b3d8b-46d3-4173-ab1e-a61765f77d61/24602416-4859-4434-98d4-6bf9d7e9b6c1"
-					(reference "R64")
+			(project "frank_m1"
+				(path "/8c0b3d8b-46d3-4173-ab1e-a61765f77d61/522a66a4-10b2-43ba-99ce-6cab39134d52"
+					(reference "R80")
 					(unit 1)
 				)
@@
 		(dnp no)
 		(fields_autoplaced yes)
-		(property "Reference" "J14"
+		(property "Reference" "J17"
 			(at 157.48 80.01 0)
 			(effects
@@
 		)
 		(instances
-			(project "turbofrank"
-				(path "/8c0b3d8b-46d3-4173-ab1e-a61765f77d61/24602416-4859-4434-98d4-6bf9d7e9b6c1"
-					(reference "J14")
+			(project "frank_m1"
+				(path "/8c0b3d8b-46d3-4173-ab1e-a61765f77d61/522a66a4-10b2-43ba-99ce-6cab39134d52"
+					(reference "J17")
 					(unit 1)
 				)
@@
 		(on_board yes)
 		(dnp no)
-		(property "Reference" "R61"
+		(property "Reference" "R77"
 			(at 120.65 96.52 90)
 			(effects
@@
 		)
 		(instances
-			(project "turbofrank"
-				(path "/8c0b3d8b-46d3-4173-ab1e-a61765f77d61/24602416-4859-4434-98d4-6bf9d7e9b6c1"
-					(reference "R61")
+			(project "frank_m1"
+				(path "/8c0b3d8b-46d3-4173-ab1e-a61765f77d61/522a66a4-10b2-43ba-99ce-6cab39134d52"
+					(reference "R77")
 					(unit 1)
 				)
@@
 		(dnp no)
 		(fields_autoplaced yes)
-		(property "Reference" "#PWR0100"
+		(property "Reference" "#PWR0133"
 			(at 157.48 127 0)
 			(effects
@@
 		)
 		(instances
-			(project "turbofrank"
-				(path "/8c0b3d8b-46d3-4173-ab1e-a61765f77d61/24602416-4859-4434-98d4-6bf9d7e9b6c1"
-					(reference "#PWR0100")
+			(project "frank_m1"
+				(path "/8c0b3d8b-46d3-4173-ab1e-a61765f77d61/522a66a4-10b2-43ba-99ce-6cab39134d52"
+					(reference "#PWR0133")
 					(unit 1)
 				)
@@
 		(on_board yes)
 		(dnp no)
-		(property "Reference" "R60"
+		(property "Reference" "R76"
 			(at 120.65 91.44 90)
 			(effects
@@
 		)
 		(instances
-			(project "turbofrank"
-				(path "/8c0b3d8b-46d3-4173-ab1e-a61765f77d61/24602416-4859-4434-98d4-6bf9d7e9b6c1"
-					(reference "R60")
+			(project "frank_m1"
+				(path "/8c0b3d8b-46d3-4173-ab1e-a61765f77d61/522a66a4-10b2-43ba-99ce-6cab39134d52"
+					(reference "R76")
 					(unit 1)
 				)
@@
 		(on_board yes)
 		(dnp no)
-		(property "Reference" "R63"
+		(property "Reference" "R79"
 			(at 184.15 101.6 90)
 			(effects
@@
 		)
 		(instances
-			(project "turbofrank"
-				(path "/8c0b3d8b-46d3-4173-ab1e-a61765f77d61/24602416-4859-4434-98d4-6bf9d7e9b6c1"
-					(reference "R63")
+			(project "frank_m1"
+				(path "/8c0b3d8b-46d3-4173-ab1e-a61765f77d61/522a66a4-10b2-43ba-99ce-6cab39134d52"
+					(reference "R79")
 					(unit 1)
 				)
@@
 		(on_board yes)
 		(dnp no)
-		(property "Reference" "R58"
+		(property "Reference" "R74"
 			(at 101.6 80.01 90)
 			(effects
@@
 		)
 		(instances
-			(project "turbofrank"
-				(path "/8c0b3d8b-46d3-4173-ab1e-a61765f77d61/24602416-4859-4434-98d4-6bf9d7e9b6c1"
-					(reference "R58")
+			(project "frank_m1"
+				(path "/8c0b3d8b-46d3-4173-ab1e-a61765f77d61/522a66a4-10b2-43ba-99ce-6cab39134d52"
+					(reference "R74")
 					(unit 1)
 				)
@@
 		(on_board yes)
 		(dnp no)
-		(property "Reference" "R57"
+		(property "Reference" "R73"
 			(at 101.6 74.93 90)
 			(effects
@@
 		)
 		(instances
-			(project "turbofrank"
-				(path "/8c0b3d8b-46d3-4173-ab1e-a61765f77d61/24602416-4859-4434-98d4-6bf9d7e9b6c1"
-					(reference "R57")
+			(project "frank_m1"
+				(path "/8c0b3d8b-46d3-4173-ab1e-a61765f77d61/522a66a4-10b2-43ba-99ce-6cab39134d52"
+					(reference "R73")
 					(unit 1)
 				)
@@
 		(on_board yes)
 		(dnp no)
-		(property "Reference" "R62"
+		(property "Reference" "R78"
 			(at 120.65 101.6 90)
 			(effects
@@
 		)
 		(instances
-			(project "turbofrank"
-				(path "/8c0b3d8b-46d3-4173-ab1e-a61765f77d61/24602416-4859-4434-98d4-6bf9d7e9b6c1"
-					(reference "R62")
+			(project "frank_m1"
+				(path "/8c0b3d8b-46d3-4173-ab1e-a61765f77d61/522a66a4-10b2-43ba-99ce-6cab39134d52"
+					(reference "R78")
 					(unit 1)
 				)

Commit message: FRANK M1 2.04
Parts:
- R73, R74, R75, R76, R77, R78, R79, R80: symbol Device:R -> FRANK:R
Other:
- title: ${NAME} ${VARIANT} -> ${NAME} ${MODEL}
Changed lines of the file:
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@@
 	(paper "A4")
 	(title_block
-		(title "${NAME} ${VARIANT}")
+		(title "${NAME} ${MODEL}")
 		(date "${DATE}")
 		(rev "${VERSION}")
@@
 	)
 	(symbol
-		(lib_id "Device:R")
+		(lib_id "FRANK:R")
 		(at 105.41 86.36 90)
 		(unit 1)
@@
 	)
 	(symbol
-		(lib_id "Device:R")
+		(lib_id "FRANK:R")
 		(at 187.96 107.95 90)
 		(unit 1)
@@
 	)
 	(symbol
-		(lib_id "Device:R")
+		(lib_id "FRANK:R")
 		(at 124.46 97.79 90)
 		(unit 1)
@@
 	)
 	(symbol
-		(lib_id "Device:R")
+		(lib_id "FRANK:R")
 		(at 124.46 92.71 90)
 		(unit 1)
@@
 	)
 	(symbol
-		(lib_id "Device:R")
+		(lib_id "FRANK:R")
 		(at 187.96 102.87 90)
 		(unit 1)
@@
 	)
 	(symbol
-		(lib_id "Device:R")
+		(lib_id "FRANK:R")
 		(at 105.41 81.28 90)
 		(unit 1)
@@
 	)
 	(symbol
-		(lib_id "Device:R")
+		(lib_id "FRANK:R")
 		(at 105.41 76.2 90)
 		(unit 1)
@@
 	)
 	(symbol
-		(lib_id "Device:R")
+		(lib_id "FRANK:R")
 		(at 124.46 102.87 90)
 		(unit 1)
