File: hardware/frank_m1/hdmi.kicad_sch (KiCad schematic)
At the start: 10 parts, among them J9 DC3RX19JA2

Commit message: FRANK M1 2.03 & xt8086 WIP
Parts:
- added D3: 1N5819WS, FRANK:Diode (SOD-323), symbol Device:D_Schottky
- C24: renamed from C5; footprint FRANK:Capacitor (0805) -> FRANK:C_0805_2012Metric
- R37: renamed from R16; footprint FRANK:Resistor (0805) -> FRANK:R_0805_2012Metric
- R38: renamed from R20; footprint FRANK:Resistor (0805) -> FRANK:R_0805_2012Metric
- R39: renamed from R14; footprint FRANK:Resistor (0805) -> FRANK:R_0805_2012Metric
- R40: renamed from R17; footprint FRANK:Resistor (0805) -> FRANK:R_0805_2012Metric
- R41: renamed from R18; footprint FRANK:Resistor (0805) -> FRANK:R_0805_2012Metric
- R42: renamed from R21; footprint FRANK:Resistor (0805) -> FRANK:R_0805_2012Metric
- R43: renamed from R15; footprint FRANK:Resistor (0805) -> FRANK:R_0805_2012Metric
- R44: renamed from R19; footprint FRANK:Resistor (0805) -> FRANK:R_0805_2012Metric
- renumbered J9 to J8
Connections:
- net VBUS: now also D3.2 (A); no longer C24.1, J8.18 (+5V)
- new net: C24.1, D3.1 (K), J8.18 (+5V)
Other:
- title: FRANK M1 -> ${NAME} ${MODEL}
- moved on the sheet: C24, J8, R37, R38, R39, R40, R41, R42, R43, R44

Commit message: FRANK M1 WIP
Parts:
- renumbered C24 to C, D3 to D, J8 to J, R40 to R, R44 to R, R39 to R, R41 to R, R37 to R, R43 to R, R42 to R, R38 to R
Changed lines of the file:
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@@
 		(on_board yes)
 		(dnp no)
-		(property "Reference" "R40"
+		(property "Reference" "R"
 			(at 162.56 111.76 90)
 			(effects
@@
 		(pin "2"
 		)
-		(instances
-			(project "frank2"
-				(path "/8c0b3d8b-46d3-4173-ab1e-a61765f77d61/db853a64-9343-4a36-b5b8-71001392b936"
-					(reference "R40")
-					(unit 1)
-				)
-			)
-		)
+		(instances)
 	)
 	(symbol
@@
 		(on_board yes)
 		(dnp no)
-		(property "Reference" "R44"
+		(property "Reference" "R"
 			(at 172.72 119.38 90)
 			(effects
@@
 		(pin "2"
 		)
-		(instances
-			(project "frank2"
-				(path "/8c0b3d8b-46d3-4173-ab1e-a61765f77d61/db853a64-9343-4a36-b5b8-71001392b936"
-					(reference "R44")
-					(unit 1)
-				)
-			)
-		)
+		(instances)
 	)
 	(symbol
@@
 		(on_board yes)
 		(dnp no)
-		(property "Reference" "R39"
+		(property "Reference" "R"
 			(at 162.56 99.06 90)
 			(effects
@@
 		(pin "2"
 		)
-		(instances
-			(project "frank2"
-				(path "/8c0b3d8b-46d3-4173-ab1e-a61765f77d61/db853a64-9343-4a36-b5b8-71001392b936"
-					(reference "R39")
-					(unit 1)
-				)
-			)
-		)
+		(instances)
 	)
 	(symbol
@@
 		(dnp no)
 		(fields_autoplaced yes)
-		(property "Reference" "#PWR065"
+		(property "Reference" "#PWR"
 			(at 151.13 74.93 0)
 			(effects
@@
 		(pin "1"
 		)
-		(instances
-			(project ""
-				(path "/8c0b3d8b-46d3-4173-ab1e-a61765f77d61/db853a64-9343-4a36-b5b8-71001392b936"
-					(reference "#PWR065")
-					(unit 1)
-				)
-			)
-		)
+		(instances)
 	)
 	(symbol
@@
 		(on_board yes)
 		(dnp no)
-		(property "Reference" "R41"
+		(property "Reference" "R"
 			(at 162.56 114.3 90)
 			(effects
@@
 		(pin "2"
 		)
-		(instances
-			(project "frank2"
-				(path "/8c0b3d8b-46d3-4173-ab1e-a61765f77d61/db853a64-9343-4a36-b5b8-71001392b936"
-					(reference "R41")
-					(unit 1)
-				)
-			)
-		)
+		(instances)
 	)
 	(symbol
@@
 		(on_board yes)
 		(dnp no)
-		(property "Reference" "C24"
+		(property "Reference" "C"
 			(at 162.6616 82.169 0)
 			(effects
@@
 		(pin "2"
 		)
-		(instances
-			(project "frank2"
-				(path "/8c0b3d8b-46d3-4173-ab1e-a61765f77d61/db853a64-9343-4a36-b5b8-71001392b936"
-					(reference "C24")
-					(unit 1)
-				)
-			)
-		)
+		(instances)
 	)
 	(symbol
@@
 		(on_board yes)
 		(dnp no)
-		(property "Reference" "R37"
+		(property "Reference" "R"
 			(at 152.4 106.68 90)
 			(effects
@@
 		(pin "2"
 		)
-		(instances
-			(project "frank2"
-				(path "/8c0b3d8b-46d3-4173-ab1e-a61765f77d61/db853a64-9343-4a36-b5b8-71001392b936"
-					(reference "R37")
-					(unit 1)
-				)
-			)
-		)
+		(instances)
 	)
 	(symbol
@@
 		(dnp no)
 		(fields_autoplaced yes)
-		(property "Reference" "#PWR064"
+		(property "Reference" "#PWR"
 			(at 139.7 144.78 0)
 			(effects
@@
 		(pin "1"
 		)
-		(instances
-			(project "frank2"
-				(path "/8c0b3d8b-46d3-4173-ab1e-a61765f77d61/db853a64-9343-4a36-b5b8-71001392b936"
-					(reference "#PWR064")
-					(unit 1)
-				)
-			)
-		)
+		(instances)
 	)
 	(symbol
@@
 		(dnp no)
 		(fields_autoplaced yes)
-		(property "Reference" "#PWR066"
+		(property "Reference" "#PWR"
 			(at 173.99 85.09 0)
 			(effects
@@
 		(pin "1"
 		)
-		(instances
-			(project ""
-				(path "/8c0b3d8b-46d3-4173-ab1e-a61765f77d61/db853a64-9343-4a36-b5b8-71001392b936"
-					(reference "#PWR066")
-					(unit 1)
-				)
-			)
-		)
+		(instances)
 	)
 	(symbol
@@
 		(on_board yes)
 		(dnp no)
-		(property "Reference" "R43"
+		(property "Reference" "R"
 			(at 172.72 104.14 90)
 			(effects
@@
 		(pin "2"
 		)
-		(instances
-			(project "frank2"
-				(path "/8c0b3d8b-46d3-4173-ab1e-a61765f77d61/db853a64-9343-4a36-b5b8-71001392b936"
-					(reference "R43")
-					(unit 1)
-				)
-			)
-		)
+		(instances)
 	)
 	(symbol
@@
 		(dnp no)
 		(fields_autoplaced yes)
-		(property "Reference" "J8"
+		(property "Reference" "J"
 			(at 115.57 99.0599 0)
 			(effects
@@
 		(pin "9"
 		)
-		(instances
-			(project "frank2"
-				(path "/8c0b3d8b-46d3-4173-ab1e-a61765f77d61/db853a64-9343-4a36-b5b8-71001392b936"
-					(reference "J8")
-					(unit 1)
-				)
-			)
-		)
+		(instances)
 	)
 	(symbol
@@
 		(on_board yes)
 		(dnp no)
-		(property "Reference" "R42"
+		(property "Reference" "R"
 			(at 162.56 127 90)
 			(effects
@@
 		(pin "2"
 		)
-		(instances
-			(project "frank2"
-				(path "/8c0b3d8b-46d3-4173-ab1e-a61765f77d61/db853a64-9343-4a36-b5b8-71001392b936"
-					(reference "R42")
-					(unit 1)
-				)
-			)
-		)
+		(instances)
 	)
 	(symbol
@@
 		(on_board yes)
 		(dnp no)
-		(property "Reference" "D3"
+		(property "Reference" "D"
 			(at 153.67 77.47 0)
 			(effects
@@
 		(pin "2"
 		)
-		(instances
-			(project "frank_m2"
-				(path "/8c0b3d8b-46d3-4173-ab1e-a61765f77d61/db853a64-9343-4a36-b5b8-71001392b936"
-					(reference "D3")
-					(unit 1)
-				)
-			)
-		)
+		(instances)
 	)
 	(symbol
@@
 		(on_board yes)
 		(dnp no)
-		(property "Reference" "R38"
+		(property "Reference" "R"
 			(at 152.4 121.92 90)
 			(effects
@@
 		(pin "2"
 		)
-		(instances
-			(project "frank2"
-				(path "/8c0b3d8b-46d3-4173-ab1e-a61765f77d61/db853a64-9343-4a36-b5b8-71001392b936"
-					(reference "R38")
-					(unit 1)
-				)
-			)
-		)
+		(instances)
 	)
 )

Commit message: New HW releases, repository cleanup
Parts:
- C14: renamed from C; symbol Device:C -> FRANK:C
- D2: renamed from D; symbol Device:D_Schottky -> FRANK:D_Schottky
- R12, R13, R14, R15, R16, R17, R18, R19: renamed from R; symbol Device:R -> FRANK:R
- renumbered J to J5
Changed lines of the file:
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@@
 	)
 	(symbol
-		(lib_id "Device:R")
+		(lib_id "FRANK:R")
 		(at 166.37 113.03 90)
 		(unit 1)
@@
 		(on_board yes)
 		(dnp no)
-		(property "Reference" "R"
+		(property "Reference" "R15"
 			(at 162.56 111.76 90)
 			(effects
@@
 		(pin "2"
 		)
-		(instances)
-	)
-	(symbol
-		(lib_id "Device:R")
+		(instances
+			(project "frank2"
+				(path "/8c0b3d8b-46d3-4173-ab1e-a61765f77d61/db853a64-9343-4a36-b5b8-71001392b936"
+					(reference "R15")
+					(unit 1)
+				)
+			)
+		)
+	)
+	(symbol
+		(lib_id "FRANK:R")
 		(at 176.53 120.65 90)
 		(unit 1)
@@
 		(on_board yes)
 		(dnp no)
-		(property "Reference" "R"
+		(property "Reference" "R19"
 			(at 172.72 119.38 90)
 			(effects
@@
 		(pin "2"
 		)
-		(instances)
-	)
-	(symbol
-		(lib_id "Device:R")
+		(instances
+			(project "frank2"
+				(path "/8c0b3d8b-46d3-4173-ab1e-a61765f77d61/db853a64-9343-4a36-b5b8-71001392b936"
+					(reference "R19")
+					(unit 1)
+				)
+			)
+		)
+	)
+	(symbol
+		(lib_id "FRANK:R")
 		(at 166.37 100.33 90)
 		(unit 1)
@@
 		(on_board yes)
 		(dnp no)
-		(property "Reference" "R"
+		(property "Reference" "R14"
 			(at 162.56 99.06 90)
 			(effects
@@
 		(pin "2"
 		)
-		(instances)
+		(instances
+			(project "frank2"
+				(path "/8c0b3d8b-46d3-4173-ab1e-a61765f77d61/db853a64-9343-4a36-b5b8-71001392b936"
+					(reference "R14")
+					(unit 1)
+				)
+			)
+		)
 	)
 	(symbol
@@
 		(dnp no)
 		(fields_autoplaced yes)
-		(property "Reference" "#PWR"
+		(property "Reference" "#PWR041"
 			(at 151.13 74.93 0)
 			(effects
@@
 		(pin "1"
 		)
-		(instances)
-	)
-	(symbol
-		(lib_id "Device:R")
+		(instances
+			(project ""
+				(path "/8c0b3d8b-46d3-4173-ab1e-a61765f77d61/db853a64-9343-4a36-b5b8-71001392b936"
+					(reference "#PWR041")
+					(unit 1)
+				)
+			)
+		)
+	)
+	(symbol
+		(lib_id "FRANK:R")
 		(at 166.37 115.57 90)
 		(unit 1)
@@
 		(on_board yes)
 		(dnp no)
-		(property "Reference" "R"
+		(property "Reference" "R16"
 			(at 162.56 114.3 90)
 			(effects
@@
 		(pin "2"
 		)
-		(instances)
-	)
-	(symbol
-		(lib_id "Device:C")
+		(instances
+			(project "frank2"
+				(path "/8c0b3d8b-46d3-4173-ab1e-a61765f77d61/db853a64-9343-4a36-b5b8-71001392b936"
+					(reference "R16")
+					(unit 1)
+				)
+			)
+		)
+	)
+	(symbol
+		(lib_id "FRANK:C")
 		(at 163.83 85.09 90)
 		(unit 1)
@@
 		(on_board yes)
 		(dnp no)
-		(property "Reference" "C"
+		(property "Reference" "C14"
 			(at 162.6616 82.169 0)
 			(effects
@@
 		(pin "2"
 		)
-		(instances)
-	)
-	(symbol
-		(lib_id "Device:R")
+		(instances
+			(project "frank2"
+				(path "/8c0b3d8b-46d3-4173-ab1e-a61765f77d61/db853a64-9343-4a36-b5b8-71001392b936"
+					(reference "C14")
+					(unit 1)
+				)
+			)
+		)
+	)
+	(symbol
+		(lib_id "FRANK:R")
 		(at 156.21 107.95 90)
 		(unit 1)
@@
 		(on_board yes)
 		(dnp no)
-		(property "Reference" "R"
+		(property "Reference" "R12"
 			(at 152.4 106.68 90)
 			(effects
@@
 		(pin "2"
 		)
-		(instances)
+		(instances
+			(project "frank2"
+				(path "/8c0b3d8b-46d3-4173-ab1e-a61765f77d61/db853a64-9343-4a36-b5b8-71001392b936"
+					(reference "R12")
+					(unit 1)
+				)
+			)
+		)
 	)
 	(symbol
@@
 		(dnp no)
 		(fields_autoplaced yes)
-		(property "Reference" "#PWR"
+		(property "Reference" "#PWR040"
 			(at 139.7 144.78 0)
 			(effects
@@
 		(pin "1"
 		)
-		(instances)
+		(instances
+			(project "frank2"
+				(path "/8c0b3d8b-46d3-4173-ab1e-a61765f77d61/db853a64-9343-4a36-b5b8-71001392b936"
+					(reference "#PWR040")
+					(unit 1)
+				)
+			)
+		)
 	)
 	(symbol
@@
 		(dnp no)
 		(fields_autoplaced yes)
-		(property "Reference" "#PWR"
+		(property "Reference" "#PWR042"
 			(at 173.99 85.09 0)
 			(effects
@@
 		(pin "1"
 		)
-		(instances)
-	)
-	(symbol
-		(lib_id "Device:R")
+		(instances
+			(project ""
+				(path "/8c0b3d8b-46d3-4173-ab1e-a61765f77d61/db853a64-9343-4a36-b5b8-71001392b936"
+					(reference "#PWR042")
+					(unit 1)
+				)
+			)
+		)
+	)
+	(symbol
+		(lib_id "FRANK:R")
 		(at 176.53 105.41 90)
 		(unit 1)
@@
 		(on_board yes)
 		(dnp no)
-		(property "Reference" "R"
+		(property "Reference" "R18"
 			(at 172.72 104.14 90)
 			(effects
@@
 		(pin "2"
 		)
-		(instances)
+		(instances
+			(project "frank2"
+				(path "/8c0b3d8b-46d3-4173-ab1e-a61765f77d61/db853a64-9343-4a36-b5b8-71001392b936"
+					(reference "R18")
+					(unit 1)
+				)
+			)
+		)
 	)
 	(symbol
@@
 		(dnp no)
 		(fields_autoplaced yes)
-		(property "Reference" "J"
+		(property "Reference" "J5"
 			(at 115.57 99.0599 0)
 			(effects
@@
 		(pin "9"
 		)
-		(instances)
-	)
-	(symbol
-		(lib_id "Device:R")
+		(instances
+			(project "frank2"
+				(path "/8c0b3d8b-46d3-4173-ab1e-a61765f77d61/db853a64-9343-4a36-b5b8-71001392b936"
+					(reference "J5")
+					(unit 1)
+				)
+			)
+		)
+	)
+	(symbol
+		(lib_id "FRANK:R")
 		(at 166.37 128.27 90)
 		(unit 1)
@@
 		(on_board yes)
 		(dnp no)
-		(property "Reference" "R"
+		(property "Reference" "R17"
 			(at 162.56 127 90)
 			(effects
@@
 		(pin "2"
 		)
-		(instances)
-	)
-	(symbol
-		(lib_id "Device:D_Schottky")
+		(instances
+			(project "frank2"
+				(path "/8c0b3d8b-46d3-4173-ab1e-a61765f77d61/db853a64-9343-4a36-b5b8-71001392b936"
+					(reference "R17")
+					(unit 1)
+				)
+			)
+		)
+	)
+	(symbol
+		(lib_id "FRANK:D_Schottky")
 		(at 151.13 77.47 90)
 		(unit 1)
@@
 		(on_board yes)
 		(dnp no)
-		(property "Reference" "D"
+		(property "Reference" "D2"
 			(at 153.67 77.47 0)
 			(effects
@@
 		(pin "2"
 		)
-		(instances)
-	)
-	(symbol
-		(lib_id "Device:R")
+		(instances
+			(project "frank_m2"
+				(path "/8c0b3d8b-46d3-4173-ab1e-a61765f77d61/db853a64-9343-4a36-b5b8-71001392b936"
+					(reference "D2")
+					(unit 1)
+				)
+			)
+		)
+	)
+	(symbol
+		(lib_id "FRANK:R")
 		(at 156.21 123.19 90)
 		(unit 1)
@@
 		(on_board yes)
 		(dnp no)
-		(property "Reference" "R"
+		(property "Reference" "R13"
 			(at 152.4 121.92 90)
 			(effects
@@
 		(pin "2"
 		)
-		(instances)
+		(instances
+			(project "frank2"
+				(path "/8c0b3d8b-46d3-4173-ab1e-a61765f77d61/db853a64-9343-4a36-b5b8-71001392b936"
+					(reference "R13")
+					(unit 1)
+				)
+			)
+		)
 	)
 )
