File: hardware/frank_m1/tape.kicad_sch (KiCad schematic)
At the start: 11 parts, among them J11 SJ1-353XNG, Q1 BC850, Q2 BC850

Commit message: FRANK M1 2.03 & xt8086 WIP
Parts:
- removed C12, C13: 100n, FRANK:Capacitor (0805), symbol Device:C
- removed D7: 1N4148, FRANK:Diode (SOD-323), symbol Device:D
- removed Q1, Q2: BC850, FRANK:SOT-23, symbol Transistor_BJT:BC850
- removed R28, R30, R31: 10K, FRANK:Resistor (0805), symbol Device:R
- removed R29: 1K, FRANK:Resistor (0805), symbol Device:R
- removed R32: 100R, FRANK:Resistor (0805), symbol Device:R
- added C28: 100n, FRANK:C_0805_2012Metric, symbol Device:C
- added R47: 4.7K, FRANK:R_0805_2012Metric, symbol Device:R
- added R48, R49: 100K, FRANK:R_0805_2012Metric, symbol Device:R
- added U5: CD4069UBM, FRANK:SOIC127P600X175-14N, symbol FRANK:CD4069UBE
- J9: renamed from J11; value SJ1-353XNG -> PJ-320D; footprint FRANK:Jack (3.5mm) -> FRANK:Jack (3.5mm, PJ-320D); AliExpress https://www.aliexpress.com/item/1005006710837751.html -> https://www.aliexpress.com/item/4001158231104.html
Connections:
- net +3V3: now also U5.14 (VDD)
- net GND: now also U5.11 (E), U5.13 (F), U5.7 (VSS), U5.9 (D14)
- net LOAD_IN: now also U5.6 (I=*C)
- net TAPE: now reaches J9.T
- net TAPE: now also C28.2
- new net: R48.1, R49.2, U5.2 (G-*A)
- new net: R47.1, R48.2, U5.1 (A)
- new net: R49.1, U5.3 (B)
- new net: U5.4 (H=*B), U5.5 (C)
- new net: C28.1, R47.2
- no-connect marks 3 -> 5
Other:
- title: FRANK M1 -> ${NAME} ${MODEL}

Commit message: FRANK M1 WIP
Parts:
- added C17: 100n, FRANK:C_0805_2012Metric, symbol Device:C
- renumbered J9 to AJ1, C28 to C16, R47 to R37, R48 to R38, R49 to R39
Connections:
- net +3V3: now also C17.1
- net GND: now also C17.2
Other:
- title: ${NAME} ${MODEL} -> ${NAME} ${VARIANT}

Commit message: FRANK M1 2.04
Parts:
- C16, C17: symbol Device:C -> FRANK:C
- R37, R38, R39: symbol Device:R -> FRANK:R
Other:
- title: ${NAME} ${VARIANT} -> ${NAME} ${MODEL}
Changed lines of the file:
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@@
 	(paper "A4")
 	(title_block
-		(title "${NAME} ${VARIANT}")
+		(title "${NAME} ${MODEL}")
 		(date "${DATE}")
 		(rev "${VERSION}")
@@
 	)
 	(symbol
-		(lib_id "Device:R")
+		(lib_id "FRANK:R")
 		(at 121.92 105.41 180)
 		(unit 1)
@@
 	)
 	(symbol
-		(lib_id "Device:C")
+		(lib_id "FRANK:C")
 		(at 218.44 93.98 180)
 		(unit 1)
@@
 			)
 		)
-		(property "Datasheet" "https://eu.mouser.com/datasheet/2/40/KGM_X7R-3223212.pdf"
+		(property "Datasheet" "~"
 			(at 218.44 93.98 0)
 			(effects
@@
 			)
 		)
-		(property "Description" ""
+		(property "Description" "Unpolarized capacitor"
 			(at 218.44 93.98 0)
 			(effects
@@
 	)
 	(symbol
-		(lib_id "Device:C")
+		(lib_id "FRANK:C")
 		(at 121.92 90.17 180)
 		(unit 1)
@@
 	)
 	(symbol
-		(lib_id "Device:R")
+		(lib_id "FRANK:R")
 		(at 121.92 97.79 180)
 		(unit 1)
@@
 	)
 	(symbol
-		(lib_id "Device:R")
+		(lib_id "FRANK:R")
 		(at 121.92 113.03 180)
 		(unit 1)

Commit message: New HW releases, repository cleanup
Parts:
- renumbered AJ1 to J18
Changed lines of the file:
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@@
 		(on_board yes)
 		(dnp no)
-		(property "Reference" "AJ1"
+		(property "Reference" "J18"
 			(at 72.8981 101.4003 0)
 			(effects
@@
 			(project "frank_m1"
 				(path "/8c0b3d8b-46d3-4173-ab1e-a61765f77d61/101b4bd6-06a1-4cc1-900e-8806ee575034"
-					(reference "AJ1")
+					(reference "J18")
 					(unit 1)
 				)
