File: lab/frank_m2/tda.kicad_sch (KiCad schematic)
At the start: 6 parts, among them U4 TDA1387T

Commit message: FRANK M2 WIP
Parts:
- added R82: 100R, FRANK:R_0805_2012Metric, symbol FRANK:R_Small
- C20: renamed from C25; symbol Device:C_Small -> FRANK:C_Small
- C21: renamed from C26; symbol Device:C_Small -> FRANK:C_Small
- C22: renamed from C27; symbol Device:C_Small -> FRANK:C_Small
- R48: renamed from R45; symbol Device:R_Small -> FRANK:R_Small
- R49: renamed from R46; symbol Device:R_Small -> FRANK:R_Small
- renumbered U4 to U6
Connections:
- net VBUS: now also R82.2; no longer C20.1, C21.1, U6.5 (VA)
- new net: C20.1, C21.1, R82.1, U6.5 (VA)

Commit message: Frank boards WIP
Parts:
- renumbered R82 to R45, R48 to R46, R49 to R47
Changed lines of the file:
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@@
 		(dnp no)
 		(fields_autoplaced yes)
-		(property "Reference" "#PWR089"
+		(property "Reference" "#PWR071"
 			(at 166.37 73.66 0)
 			(effects
@@
 			(project "frank_m2"
 				(path "/8c0b3d8b-46d3-4173-ab1e-a61765f77d61/9d0ad236-240c-42bd-9e4a-79b0506e7ea9/0dccd710-fd54-4e53-9f08-059759dd7a75"
-					(reference "#PWR089")
+					(reference "#PWR071")
 					(unit 1)
 				)
@@
 		(on_board yes)
 		(dnp no)
-		(property "Reference" "R82"
+		(property "Reference" "R45"
 			(at 163.83 78.74 90)
 			(effects
@@
 			(project "frank_m2"
 				(path "/8c0b3d8b-46d3-4173-ab1e-a61765f77d61/9d0ad236-240c-42bd-9e4a-79b0506e7ea9/0dccd710-fd54-4e53-9f08-059759dd7a75"
-					(reference "R82")
+					(reference "R45")
 					(unit 1)
 				)
@@
 		(on_board yes)
 		(dnp no)
-		(property "Reference" "R49"
+		(property "Reference" "R47"
 			(at 184.15 97.79 90)
 			(effects
@@
 			(project "frank_m2"
 				(path "/8c0b3d8b-46d3-4173-ab1e-a61765f77d61/9d0ad236-240c-42bd-9e4a-79b0506e7ea9/0dccd710-fd54-4e53-9f08-059759dd7a75"
-					(reference "R49")
+					(reference "R47")
 					(unit 1)
 				)
@@
 		(dnp no)
 		(fields_autoplaced yes)
-		(property "Reference" "#PWR093"
+		(property "Reference" "#PWR075"
 			(at 186.69 109.22 0)
 			(effects
@@
 			(project "frank_m2"
 				(path "/8c0b3d8b-46d3-4173-ab1e-a61765f77d61/9d0ad236-240c-42bd-9e4a-79b0506e7ea9/0dccd710-fd54-4e53-9f08-059759dd7a75"
-					(reference "#PWR093")
+					(reference "#PWR075")
 					(unit 1)
 				)
@@
 		(dnp no)
 		(fields_autoplaced yes)
-		(property "Reference" "#PWR092"
+		(property "Reference" "#PWR074"
 			(at 186.69 68.58 0)
 			(effects
@@
 			(project "frank_m2"
 				(path "/8c0b3d8b-46d3-4173-ab1e-a61765f77d61/9d0ad236-240c-42bd-9e4a-79b0506e7ea9/0dccd710-fd54-4e53-9f08-059759dd7a75"
-					(reference "#PWR092")
+					(reference "#PWR074")
 					(unit 1)
 				)
@@
 		(on_board yes)
 		(dnp no)
-		(property "Reference" "R48"
+		(property "Reference" "R46"
 			(at 184.15 80.01 90)
 			(effects
@@
 			(project "frank_m2"
 				(path "/8c0b3d8b-46d3-4173-ab1e-a61765f77d61/9d0ad236-240c-42bd-9e4a-79b0506e7ea9/0dccd710-fd54-4e53-9f08-059759dd7a75"
-					(reference "R48")
+					(reference "R46")
 					(unit 1)
 				)
@@
 		(dnp no)
 		(fields_autoplaced yes)
-		(property "Reference" "#PWR087"
+		(property "Reference" "#PWR069"
 			(at 116.84 109.22 0)
 			(effects
@@
 			(project "frank_m2"
 				(path "/8c0b3d8b-46d3-4173-ab1e-a61765f77d61/9d0ad236-240c-42bd-9e4a-79b0506e7ea9/0dccd710-fd54-4e53-9f08-059759dd7a75"
-					(reference "#PWR087")
+					(reference "#PWR069")
 					(unit 1)
 				)
@@
 		(on_board yes)
 		(dnp no)
-		(property "Reference" "#PWR090"
+		(property "Reference" "#PWR072"
 			(at 166.37 121.92 0)
 			(effects
@@
 			(project "frank_m2"
 				(path "/8c0b3d8b-46d3-4173-ab1e-a61765f77d61/9d0ad236-240c-42bd-9e4a-79b0506e7ea9/0dccd710-fd54-4e53-9f08-059759dd7a75"
-					(reference "#PWR090")
+					(reference "#PWR072")
 					(unit 1)
 				)
@@
 		(dnp no)
 		(fields_autoplaced yes)
-		(property "Reference" "#PWR088"
+		(property "Reference" "#PWR070"
 			(at 157.48 121.92 0)
 			(effects
@@
 			(project "frank_m2"
 				(path "/8c0b3d8b-46d3-4173-ab1e-a61765f77d61/9d0ad236-240c-42bd-9e4a-79b0506e7ea9/0dccd710-fd54-4e53-9f08-059759dd7a75"
-					(reference "#PWR088")
+					(reference "#PWR070")
 					(unit 1)
 				)
@@
 		(dnp no)
 		(fields_autoplaced yes)
-		(property "Reference" "#PWR091"
+		(property "Reference" "#PWR073"
 			(at 176.53 121.92 0)
 			(effects
@@
 			(project "frank_m2"
 				(path "/8c0b3d8b-46d3-4173-ab1e-a61765f77d61/9d0ad236-240c-42bd-9e4a-79b0506e7ea9/0dccd710-fd54-4e53-9f08-059759dd7a75"
-					(reference "#PWR091")
+					(reference "#PWR073")
 					(unit 1)
 				)
