File: lab/frank_m2/vga.kicad_sch (KiCad schematic)
At the start: 9 parts, among them J14 D-SUB 15 Female

Commit message: FRANK M2 WIP
Parts:
- R73: renamed from R57; symbol Device:R -> FRANK:R
- R74: renamed from R58; symbol Device:R -> FRANK:R
- R75: renamed from R59; symbol Device:R -> FRANK:R
- R76: renamed from R60; symbol Device:R -> FRANK:R
- R77: renamed from R61; symbol Device:R -> FRANK:R
- R78: renamed from R62; symbol Device:R -> FRANK:R
- R79: renamed from R63; symbol Device:R -> FRANK:R
- R80: renamed from R64; symbol Device:R -> FRANK:R
- renumbered J14 to J17
Changed lines of the file:
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@@
 	)
 	(symbol
-		(lib_id "Device:R")
+		(lib_id "FRANK:R")
 		(at 105.41 86.36 90)
 		(unit 1)
@@
 		(on_board yes)
 		(dnp no)
-		(property "Reference" "R59"
+		(property "Reference" "R75"
 			(at 101.6 85.09 90)
 			(effects
@@
 		)
 		(instances
-			(project "turbofrank"
-				(path "/8c0b3d8b-46d3-4173-ab1e-a61765f77d61/24602416-4859-4434-98d4-6bf9d7e9b6c1"
-					(reference "R59")
-					(unit 1)
-				)
-			)
-		)
-	)
-	(symbol
-		(lib_id "Device:R")
+			(project "frank_m2"
+				(path "/8c0b3d8b-46d3-4173-ab1e-a61765f77d61/522a66a4-10b2-43ba-99ce-6cab39134d52"
+					(reference "R75")
+					(unit 1)
+				)
+			)
+		)
+	)
+	(symbol
+		(lib_id "FRANK:R")
 		(at 187.96 107.95 90)
 		(unit 1)
@@
 		(on_board yes)
 		(dnp no)
-		(property "Reference" "R64"
+		(property "Reference" "R80"
 			(at 184.15 106.68 90)
 			(effects
@@
 		)
 		(instances
-			(project "turbofrank"
-				(path "/8c0b3d8b-46d3-4173-ab1e-a61765f77d61/24602416-4859-4434-98d4-6bf9d7e9b6c1"
-					(reference "R64")
+			(project "frank_m2"
+				(path "/8c0b3d8b-46d3-4173-ab1e-a61765f77d61/522a66a4-10b2-43ba-99ce-6cab39134d52"
+					(reference "R80")
 					(unit 1)
 				)
@@
 		(dnp no)
 		(fields_autoplaced yes)
-		(property "Reference" "J14"
+		(property "Reference" "J17"
 			(at 157.48 80.01 0)
 			(effects
@@
 		)
 		(instances
-			(project "turbofrank"
-				(path "/8c0b3d8b-46d3-4173-ab1e-a61765f77d61/24602416-4859-4434-98d4-6bf9d7e9b6c1"
-					(reference "J14")
-					(unit 1)
-				)
-			)
-		)
-	)
-	(symbol
-		(lib_id "Device:R")
+			(project "frank_m2"
+				(path "/8c0b3d8b-46d3-4173-ab1e-a61765f77d61/522a66a4-10b2-43ba-99ce-6cab39134d52"
+					(reference "J17")
+					(unit 1)
+				)
+			)
+		)
+	)
+	(symbol
+		(lib_id "FRANK:R")
 		(at 124.46 97.79 90)
 		(unit 1)
@@
 		(on_board yes)
 		(dnp no)
-		(property "Reference" "R61"
+		(property "Reference" "R77"
 			(at 120.65 96.52 90)
 			(effects
@@
 		)
 		(instances
-			(project "turbofrank"
-				(path "/8c0b3d8b-46d3-4173-ab1e-a61765f77d61/24602416-4859-4434-98d4-6bf9d7e9b6c1"
-					(reference "R61")
+			(project "frank_m2"
+				(path "/8c0b3d8b-46d3-4173-ab1e-a61765f77d61/522a66a4-10b2-43ba-99ce-6cab39134d52"
+					(reference "R77")
 					(unit 1)
 				)
@@
 		(dnp no)
 		(fields_autoplaced yes)
-		(property "Reference" "#PWR0100"
+		(property "Reference" "#PWR0133"
 			(at 157.48 127 0)
 			(effects
@@
 		)
 		(instances
-			(project "turbofrank"
-				(path "/8c0b3d8b-46d3-4173-ab1e-a61765f77d61/24602416-4859-4434-98d4-6bf9d7e9b6c1"
-					(reference "#PWR0100")
-					(unit 1)
-				)
-			)
-		)
-	)
-	(symbol
-		(lib_id "Device:R")
+			(project "frank_m2"
+				(path "/8c0b3d8b-46d3-4173-ab1e-a61765f77d61/522a66a4-10b2-43ba-99ce-6cab39134d52"
+					(reference "#PWR0133")
+					(unit 1)
+				)
+			)
+		)
+	)
+	(symbol
+		(lib_id "FRANK:R")
 		(at 124.46 92.71 90)
 		(unit 1)
@@
 		(on_board yes)
 		(dnp no)
-		(property "Reference" "R60"
+		(property "Reference" "R76"
 			(at 120.65 91.44 90)
 			(effects
@@
 		)
 		(instances
-			(project "turbofrank"
-				(path "/8c0b3d8b-46d3-4173-ab1e-a61765f77d61/24602416-4859-4434-98d4-6bf9d7e9b6c1"
-					(reference "R60")
-					(unit 1)
-				)
-			)
-		)
-	)
-	(symbol
-		(lib_id "Device:R")
+			(project "frank_m2"
+				(path "/8c0b3d8b-46d3-4173-ab1e-a61765f77d61/522a66a4-10b2-43ba-99ce-6cab39134d52"
+					(reference "R76")
+					(unit 1)
+				)
+			)
+		)
+	)
+	(symbol
+		(lib_id "FRANK:R")
 		(at 187.96 102.87 90)
 		(unit 1)
@@
 		(on_board yes)
 		(dnp no)
-		(property "Reference" "R63"
+		(property "Reference" "R79"
 			(at 184.15 101.6 90)
 			(effects
@@
 		)
 		(instances
-			(project "turbofrank"
-				(path "/8c0b3d8b-46d3-4173-ab1e-a61765f77d61/24602416-4859-4434-98d4-6bf9d7e9b6c1"
-					(reference "R63")
-					(unit 1)
-				)
-			)
-		)
-	)
-	(symbol
-		(lib_id "Device:R")
+			(project "frank_m2"
+				(path "/8c0b3d8b-46d3-4173-ab1e-a61765f77d61/522a66a4-10b2-43ba-99ce-6cab39134d52"
+					(reference "R79")
+					(unit 1)
+				)
+			)
+		)
+	)
+	(symbol
+		(lib_id "FRANK:R")
 		(at 105.41 81.28 90)
 		(unit 1)
@@
 		(on_board yes)
 		(dnp no)
-		(property "Reference" "R58"
+		(property "Reference" "R74"
 			(at 101.6 80.01 90)
 			(effects
@@
 		)
 		(instances
-			(project "turbofrank"
-				(path "/8c0b3d8b-46d3-4173-ab1e-a61765f77d61/24602416-4859-4434-98d4-6bf9d7e9b6c1"
-					(reference "R58")
-					(unit 1)
-				)
-			)
-		)
-	)
-	(symbol
-		(lib_id "Device:R")
+			(project "frank_m2"
+				(path "/8c0b3d8b-46d3-4173-ab1e-a61765f77d61/522a66a4-10b2-43ba-99ce-6cab39134d52"
+					(reference "R74")
+					(unit 1)
+				)
+			)
+		)
+	)
+	(symbol
+		(lib_id "FRANK:R")
 		(at 105.41 76.2 90)
 		(unit 1)
@@
 		(on_board yes)
 		(dnp no)
-		(property "Reference" "R57"
+		(property "Reference" "R73"
 			(at 101.6 74.93 90)
 			(effects
@@
 		)
 		(instances
-			(project "turbofrank"
-				(path "/8c0b3d8b-46d3-4173-ab1e-a61765f77d61/24602416-4859-4434-98d4-6bf9d7e9b6c1"
-					(reference "R57")
-					(unit 1)
-				)
-			)
-		)
-	)
-	(symbol
-		(lib_id "Device:R")
+			(project "frank_m2"
+				(path "/8c0b3d8b-46d3-4173-ab1e-a61765f77d61/522a66a4-10b2-43ba-99ce-6cab39134d52"
+					(reference "R73")
+					(unit 1)
+				)
+			)
+		)
+	)
+	(symbol
+		(lib_id "FRANK:R")
 		(at 124.46 102.87 90)
 		(unit 1)
@@
 		(on_board yes)
 		(dnp no)
-		(property "Reference" "R62"
+		(property "Reference" "R78"
 			(at 120.65 101.6 90)
 			(effects
@@
 		)
 		(instances
-			(project "turbofrank"
-				(path "/8c0b3d8b-46d3-4173-ab1e-a61765f77d61/24602416-4859-4434-98d4-6bf9d7e9b6c1"
-					(reference "R62")
-					(unit 1)
-				)
+			(project "frank_m2"
+				(path "/8c0b3d8b-46d3-4173-ab1e-a61765f77d61/522a66a4-10b2-43ba-99ce-6cab39134d52"
+					(reference "R78")
+					(unit 1)
+				)

Commit message: Frank boards WIP
Parts:
- J16: renamed from J17; value D-SUB 15 Female -> VGA
- renumbered R73 to R71, R74 to R72, R75 to R73, R76 to R74, R77 to R75, R78 to R76, R79 to R77, R80 to R78
Changed lines of the file:
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@@
 		(on_board yes)
 		(dnp no)
-		(property "Reference" "R75"
+		(property "Reference" "R73"
 			(at 101.6 85.09 90)
 			(effects
@@
 			(project "frank_m2"
 				(path "/8c0b3d8b-46d3-4173-ab1e-a61765f77d61/522a66a4-10b2-43ba-99ce-6cab39134d52"
-					(reference "R75")
+					(reference "R73")
 					(unit 1)
 				)
@@
 		(on_board yes)
 		(dnp no)
-		(property "Reference" "R80"
+		(property "Reference" "R78"
 			(at 184.15 106.68 90)
 			(effects
@@
 			(project "frank_m2"
 				(path "/8c0b3d8b-46d3-4173-ab1e-a61765f77d61/522a66a4-10b2-43ba-99ce-6cab39134d52"
-					(reference "R80")
+					(reference "R78")
 					(unit 1)
 				)
@@
 		(dnp no)
 		(fields_autoplaced yes)
-		(property "Reference" "J17"
+		(property "Reference" "J16"
 			(at 157.48 80.01 0)
 			(effects
@@
 			)
 		)
-		(property "Value" "D-SUB 15 Female"
+		(property "Value" "VGA"
 			(at 157.48 82.55 0)
 			(effects
@@
 			(project "frank_m2"
 				(path "/8c0b3d8b-46d3-4173-ab1e-a61765f77d61/522a66a4-10b2-43ba-99ce-6cab39134d52"
-					(reference "J17")
+					(reference "J16")
 					(unit 1)
 				)
@@
 		(on_board yes)
 		(dnp no)
-		(property "Reference" "R77"
+		(property "Reference" "R75"
 			(at 120.65 96.52 90)
 			(effects
@@
 			(project "frank_m2"
 				(path "/8c0b3d8b-46d3-4173-ab1e-a61765f77d61/522a66a4-10b2-43ba-99ce-6cab39134d52"
-					(reference "R77")
+					(reference "R75")
 					(unit 1)
 				)
@@
 		(dnp no)
 		(fields_autoplaced yes)
-		(property "Reference" "#PWR0133"
+		(property "Reference" "#PWR0117"
 			(at 157.48 127 0)
 			(effects
@@
 			(project "frank_m2"
 				(path "/8c0b3d8b-46d3-4173-ab1e-a61765f77d61/522a66a4-10b2-43ba-99ce-6cab39134d52"
-					(reference "#PWR0133")
+					(reference "#PWR0117")
 					(unit 1)
 				)
@@
 		(on_board yes)
 		(dnp no)
-		(property "Reference" "R76"
+		(property "Reference" "R74"
 			(at 120.65 91.44 90)
 			(effects
@@
 			(project "frank_m2"
 				(path "/8c0b3d8b-46d3-4173-ab1e-a61765f77d61/522a66a4-10b2-43ba-99ce-6cab39134d52"
-					(reference "R76")
+					(reference "R74")
 					(unit 1)
 				)
@@
 		(on_board yes)
 		(dnp no)
-		(property "Reference" "R79"
+		(property "Reference" "R77"
 			(at 184.15 101.6 90)
 			(effects
@@
 			(project "frank_m2"
 				(path "/8c0b3d8b-46d3-4173-ab1e-a61765f77d61/522a66a4-10b2-43ba-99ce-6cab39134d52"
-					(reference "R79")
+					(reference "R77")
 					(unit 1)
 				)
@@
 		(on_board yes)
 		(dnp no)
-		(property "Reference" "R74"
+		(property "Reference" "R72"
 			(at 101.6 80.01 90)
 			(effects
@@
 			(project "frank_m2"
 				(path "/8c0b3d8b-46d3-4173-ab1e-a61765f77d61/522a66a4-10b2-43ba-99ce-6cab39134d52"
-					(reference "R74")
+					(reference "R72")
 					(unit 1)
 				)
@@
 		(on_board yes)
 		(dnp no)
-		(property "Reference" "R73"
+		(property "Reference" "R71"
 			(at 101.6 74.93 90)
 			(effects
@@
 			(project "frank_m2"
 				(path "/8c0b3d8b-46d3-4173-ab1e-a61765f77d61/522a66a4-10b2-43ba-99ce-6cab39134d52"
-					(reference "R73")
+					(reference "R71")
 					(unit 1)
 				)
@@
 		(on_board yes)
 		(dnp no)
-		(property "Reference" "R78"
+		(property "Reference" "R76"
 			(at 120.65 101.6 90)
 			(effects
@@
 			(project "frank_m2"
 				(path "/8c0b3d8b-46d3-4173-ab1e-a61765f77d61/522a66a4-10b2-43ba-99ce-6cab39134d52"
-					(reference "R78")
-					(unit 1)
-				)
+					(reference "R76")
+					(unit 1)
+				)
