File: hardware/minifrank_rm2/audio.kicad_sch (KiCad schematic)
At the start: 1 part, among them J2 PJ-320D

Commit message: Board updates
Parts:
- renumbered J2 to J11
Connections:
- no-connect marks 0 -> 1
Other:
- removed sheet PWM
- title: ${NAME} -> ${NAME} ${MODEL}
