File: lab/minifrank_rm2_pro/usb.kicad_sch (KiCad schematic)
At the start: 17 parts, among them J10 SS-52100-004, J9 USB4215-03-A, U12 MW7211A, U13 USBLC6-2SC6

Commit message: MiniFRANK RM2 WIP
Parts:
- renumbered C54 to C50, C57 to C53, C58 to C54, J9 to J8, J10 to J9, R41 to R37, R42 to R38, R43 to R39, R44 to R40, R45 to R41, R48 to R44, R49 to R45, R50 to R46, R51 to R47, U12 to U11, U13 to U12
