File: lab/minifrank_rm2_pro/usb2ttl.kicad_sch (KiCad schematic)
At the start: 6 parts, among them U11 CH340C

Commit message: MiniFRANK RM2 WIP
Parts:
- C49: renamed from C53; footprint FRANK:Capacitor (0603, S) -> FRANK:C_0603_1608Metric
- LD3, LD4: footprint FRANK:LED (0805) -> FRANK:LED_0603_1608Metric
- renumbered R39 to R35, R40 to R36, U11 to U10
Changed lines of the file:
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@@
 			)
 		)
-		(property "Footprint" "FRANK:LED (0805)"
+		(property "Footprint" "FRANK:LED_0603_1608Metric"
 			(at 176.53 95.25 90)
 			(effects
@@
 		(on_board yes)
 		(dnp no)
-		(property "Reference" "U11"
+		(property "Reference" "U10"
 			(at 134.62 75.946 0)
 			(effects
@@
 			(project "echo"
 				(path "/8c0b3d8b-46d3-4173-ab1e-a61765f77d61/ac94f22c-2cf6-40d7-be87-268997e0aba1"
-					(reference "U11")
+					(reference "U10")
 					(unit 1)
 				)
@@
 		(on_board yes)
 		(dnp no)
-		(property "Reference" "R40"
+		(property "Reference" "R36"
 			(at 189.484 87.63 90)
 			(effects
@@
 			(project "echo"
 				(path "/8c0b3d8b-46d3-4173-ab1e-a61765f77d61/ac94f22c-2cf6-40d7-be87-268997e0aba1"
-					(reference "R40")
+					(reference "R36")
 					(unit 1)
 				)
@@
 		(on_board yes)
 		(dnp no)
-		(property "Reference" "#PWR0109"
+		(property "Reference" "#PWR094"
 			(at 190.5 80.01 0)
 			(effects
@@
 			(project ""
 				(path "/8c0b3d8b-46d3-4173-ab1e-a61765f77d61/ac94f22c-2cf6-40d7-be87-268997e0aba1"
-					(reference "#PWR0109")
+					(reference "#PWR094")
 					(unit 1)
 				)
@@
 		(on_board yes)
 		(dnp no)
-		(property "Reference" "#PWR0107"
+		(property "Reference" "#PWR092"
 			(at 113.03 87.63 0)
 			(effects
@@
 			(project "protea"
 				(path "/8c0b3d8b-46d3-4173-ab1e-a61765f77d61/ac94f22c-2cf6-40d7-be87-268997e0aba1"
-					(reference "#PWR0107")
+					(reference "#PWR092")
 					(unit 1)
 				)
@@
 		(on_board yes)
 		(dnp no)
-		(property "Reference" "R39"
+		(property "Reference" "R35"
 			(at 179.07 87.63 90)
 			(effects
@@
 			(project "echo"
 				(path "/8c0b3d8b-46d3-4173-ab1e-a61765f77d61/ac94f22c-2cf6-40d7-be87-268997e0aba1"
-					(reference "R39")
+					(reference "R35")
 					(unit 1)
 				)
@@
 		(dnp no)
 		(fields_autoplaced yes)
-		(property "Reference" "#PWR0106"
+		(property "Reference" "#PWR091"
 			(at 102.87 80.01 0)
 			(effects
@@
 			(project ""
 				(path "/8c0b3d8b-46d3-4173-ab1e-a61765f77d61/ac94f22c-2cf6-40d7-be87-268997e0aba1"
-					(reference "#PWR0106")
+					(reference "#PWR091")
 					(unit 1)
 				)
@@
 		(on_board yes)
 		(dnp no)
-		(property "Reference" "#PWR0108"
+		(property "Reference" "#PWR093"
 			(at 165.1 97.79 0)
 			(effects
@@
 			(project "echo"
 				(path "/8c0b3d8b-46d3-4173-ab1e-a61765f77d61/ac94f22c-2cf6-40d7-be87-268997e0aba1"
-					(reference "#PWR0108")
+					(reference "#PWR093")
 					(unit 1)
 				)
@@
 			)
 		)
-		(property "Footprint" "FRANK:LED (0805)"
+		(property "Footprint" "FRANK:LED_0603_1608Metric"
 			(at 186.69 95.25 90)
 			(effects
@@
 		(on_board yes)
 		(dnp no)
-		(property "Reference" "C53"
+		(property "Reference" "C49"
 			(at 165.608 83.82 0)
 			(effects
@@
 			)
 		)
-		(property "Footprint" "FRANK:Capacitor (0603, S)"
+		(property "Footprint" "FRANK:C_0603_1608Metric"
 			(at 165.1 86.36 0)
 			(effects
@@
 			(project "echo"
 				(path "/8c0b3d8b-46d3-4173-ab1e-a61765f77d61/ac94f22c-2cf6-40d7-be87-268997e0aba1"
-					(reference "C53")
-					(unit 1)
-				)
+					(reference "C49")
+					(unit 1)
+				)
