File: hardware/minifrank_rm2p2/minifrank_rm2p2.kicad_pcb (KiCad board)
At the start: 4 copper layers, 85.6 x 54 mm, 133 parts, among them J1 PWR, J10 VGA, J11 PJ-320D, J12 104031-0811, J2 DEBUG, J3 UART, J4 SS-52100-004, J5 USB4215-03-A, J6 MDC-036, J7 PJ-320D, J8 DC3RX19JA2, J9 GP2, U1 TS3USB221RSER, U10 TDA1387T, U11 LM358, U2 USBLC6-2SC6, U3 MW7211A, U4 ME6211C33M5, U5 TXS0104ERGYR, U6 ESP-PSRAM32, U7 W25Q128JVS, U8 CD4069UBM, U9 RP2350, Y1 ASE-12MHz

Commit message: MiniFRANK RM2P2 WIP
Parts:
- removed the S4 at (214.8, 77.5)
- added S3: ESP Reset, FRANK:KMR_2, F.Cu at (172.8, 96.0)
- added S5: RP Reset, FRANK:TS-1234VW, F.Cu at (214.5, 77.6)
- added U10: ESP-01v090, FRANK:ESP-01, F.Cu at (165.2, 80.4)
- C4: value 10u -> 22u; footprint FRANK:C_0603_1608Metric -> FRANK:Capacitor (3528, tantalum, polar)
- C7: value 100n -> 22u; footprint FRANK:C_0603_1608Metric -> FRANK:Capacitor (3528, tantalum, polar)
- C9: value 10u -> 100n
- J2: value DEBUG -> UART; footprint FRANK:Pin Header (1x03) -> FRANK:JST_SH_BM04B-SRSS-TB_1x04-1MP_P1.00mm_Vertical
- J3: value UART -> DEBUG; footprint FRANK:Pin Header (1x03) -> FRANK:JST_SH_BM03B-SRSS-TB_1x03-1MP_P1.00mm_Vertical
- S2: value Reset RP2530A -> RP Reset; footprint FRANK:TACT-SIDE-4623 -> FRANK:TS-1234VW
- U4: value ME6211C33M5 -> NCP1117-3.3_SOT223; footprint FRANK:SOT-23-5 -> Package_TO_SOT_SMD:SOT-223-3_TabPin2
- moved J1 16.7 mm to (175.6, 79.0)
- moved C9 13.9 mm to (213.2, 95.2)
- moved R17 13.4 mm to (169.5, 88.9), turned to -90 degrees
- moved R12 13.3 mm to (213.2, 82.9)
- moved C7 12.8 mm to (213.3, 97.7)
- moved J3 7.23 mm to (178.6, 99.9)
- moved D1 5.36 mm to (209.5, 101.9)
- moved C5 5.27 mm to (200.7, 103.5)
- moved L1 3.26 mm to (208.9, 105.0)
- moved C15 1.79 mm to (171.2, 92.1), turned to 90 degrees
- moved U4 1.56 mm to (204.1, 97.2)
- moved C4 1.50 mm to (205.2, 102.6), turned to 180 degrees
- moved J2 1.14 mm to (171.9, 100.7), turned to 180 degrees
- moved S2 0.56 mm to (132.5, 106.8), turned to -90 degrees
- renumbered L2 to L1, L1 to L2, S3 to S4, U10 to U11, U11 to U12
Connections:
- C7 pad 1: +3V3 -> GND
- C7 pad 2: GND -> +3V3
- C9 pad 1: +3V3 -> GND
- C9 pad 2: GND -> +3V3
- J2 pad 1: /SWCLK -> GND
- J2 pad 2: /SWD -> +3V3
- J2 pad 3: GND -> /GPIO0
- J3 pad 1: /GPIO0 -> /SWCLK
- J3 pad 2: /GPIO1 -> GND
- J3 pad 3: GND -> /SWD
- U4 pad 1: VBUS -> GND
- U4 pad 2: GND -> +3V3
Routing:
- net /GPIO20: track 113.2 -> 146.7 mm
- net /ESP_RST: track 0.00 -> 24.5 mm, vias 0 -> 1
- net /GPIO21: track 122.6 -> 143.4 mm
- net GND: track 0.00 -> 11.5 mm, vias 10 -> 12
- net /SWCLK: track 31.5 -> 20.8 mm
- net VBUS: track 207.7 -> 217.5 mm, vias 10 -> 13
- net +3V3: track 62.9 -> 69.7 mm, vias 25 -> 28
- net /Power/VBUS_IN: track 11.2 -> 4.73 mm, vias 0 -> 1
- net Net-(D1-A): track 9.71 -> 13.6 mm
- net /RUN: track 95.0 -> 98.6 mm
- net Net-(C8-Pad1): track 8.76 -> 5.67 mm, vias 0 -> 1
- net /RP2350A/~{USB_BOOT}: track 3.82 -> 6.42 mm
- net /RP2350A/FLASH_SS: track 13.6 -> 15.0 mm
- net /SWD: track 26.9 -> 25.9 mm
- net /GPIO0: track 58.2 -> 59.2 mm, vias 2 -> 3
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Other:
- board text removed: "3V3"
- board text removed: "5V"
- board text removed: "CLK SWD GND"
- board text removed: "GND"
- board text removed: "IO0 IO1 GND"

Commit message: Bugfixes
Parts:
- added S6: RP Reset, FRANK:KMR_2, F.Cu at (152.2, 86.7)
- added S7: RP Reset, FRANK:KMR_2, F.Cu at (199.2, 85.5)
Connections:
- S3 pad 1: /ESP_RST -> GND
- S3 pad 4: GND -> /ESP_RST
Routing:
- net /RUN: track 98.6 -> 133.5 mm, vias 2 -> 6
- net /RP2350A/~{USB_BOOT}: track 6.42 -> 24.2 mm, vias 0 -> 2
- net VBUS: track 217.5 -> 214.7 mm
- net /ESP_RST: track 24.5 -> 27.0 mm
- net /GPIO1: track 66.8 -> 65.7 mm
- net /SWCLK: track 20.8 -> 20.1 mm
- net GND: vias 12 -> 15
Other:
- board text added: "3V3"
- board text added: "5V"
- board text added: "DBG"
- board text added: "ERS"
- board text added: "ESP-01"
- board text added: "GND"
- board text added: "UART"

Commit message: Bugfixes
Parts:
- turned C39 to 0 degrees
- turned C4 to 0 degrees
- turned C7 to 0 degrees
Connections:
- C39 pad 1: GND -> Net-(U12C-V+)
- C39 pad 2: Net-(U12C-V+) -> GND
- C4 pad 1: GND -> VBUS
- C4 pad 2: VBUS -> GND
- C7 pad 1: GND -> +3V3
- C7 pad 2: +3V3 -> GND
