File: lab/frank_m2_pro/amp.kicad_sch (KiCad schematic)
At the start: 30 parts, among them U10 PAM8403D, U11 LM358

Commit message: FRANK M2 Pro WIP
Parts:
- renumbered R38 to R39, R39 to R40, R40 to R41, R41 to R42, R42 to R43, R43 to R44, R44 to R45, R45 to R46, R46 to R47, R47 to R48, R48 to R49, R49 to R50, R50 to R51, R51 to R52, R52 to R53, R53 to R54
