File: lab/frank_m2_pro/tape.kicad_sch (KiCad schematic)
At the start: 7 parts, among them J9 PJ-320D, U8 CD4069UBM

Commit message: FRANK M2 Pro WIP
Parts:
- renumbered R24 to R25, R25 to R26, R26 to R27
Changed lines of the file:
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@@
 		(on_board yes)
 		(dnp no)
-		(property "Reference" "R25"
+		(property "Reference" "R26"
 			(at 119.634 105.156 90)
 			(effects
@@
 			(project "frank_m2"
 				(path "/8c0b3d8b-46d3-4173-ab1e-a61765f77d61/101b4bd6-06a1-4cc1-900e-8806ee575034"
-					(reference "R25")
+					(reference "R26")
 					(unit 1)
 				)
@@
 		(dnp no)
 		(fields_autoplaced yes)
-		(property "Reference" "#PWR078"
+		(property "Reference" "#PWR083"
 			(at 140.97 116.84 0)
 			(effects
@@
 			(project "frank_m2"
 				(path "/8c0b3d8b-46d3-4173-ab1e-a61765f77d61/101b4bd6-06a1-4cc1-900e-8806ee575034"
-					(reference "#PWR078")
+					(reference "#PWR083")
 					(unit 1)
 				)
@@
 		(dnp no)
 		(fields_autoplaced yes)
-		(property "Reference" "#PWR083"
+		(property "Reference" "#PWR088"
 			(at 226.06 114.3 0)
 			(effects
@@
 			(project "frank_m2"
 				(path "/8c0b3d8b-46d3-4173-ab1e-a61765f77d61/101b4bd6-06a1-4cc1-900e-8806ee575034"
-					(reference "#PWR083")
+					(reference "#PWR088")
 					(unit 1)
 				)
@@
 		(dnp no)
 		(fields_autoplaced yes)
-		(property "Reference" "#PWR082"
+		(property "Reference" "#PWR087"
 			(at 226.06 109.22 0)
 			(effects
@@
 			(project "frank_m2"
 				(path "/8c0b3d8b-46d3-4173-ab1e-a61765f77d61/101b4bd6-06a1-4cc1-900e-8806ee575034"
-					(reference "#PWR082")
+					(reference "#PWR087")
 					(unit 1)
 				)
@@
 		(on_board yes)
 		(dnp no)
-		(property "Reference" "#PWR079"
+		(property "Reference" "#PWR084"
 			(at 218.44 85.09 0)
 			(effects
@@
 			(project "frank_m2"
 				(path "/8c0b3d8b-46d3-4173-ab1e-a61765f77d61/101b4bd6-06a1-4cc1-900e-8806ee575034"
-					(reference "#PWR079")
+					(reference "#PWR084")
 					(unit 1)
 				)
@@
 		(dnp no)
 		(fields_autoplaced yes)
-		(property "Reference" "#PWR077"
+		(property "Reference" "#PWR082"
 			(at 91.44 107.95 0)
 			(effects
@@
 			(project "frank_m2"
 				(path "/8c0b3d8b-46d3-4173-ab1e-a61765f77d61/101b4bd6-06a1-4cc1-900e-8806ee575034"
-					(reference "#PWR077")
+					(reference "#PWR082")
 					(unit 1)
 				)
@@
 		(on_board yes)
 		(dnp no)
-		(property "Reference" "#PWR080"
+		(property "Reference" "#PWR085"
 			(at 215.9 101.6 0)
 			(effects
@@
 			(project "frank_m2"
 				(path "/8c0b3d8b-46d3-4173-ab1e-a61765f77d61/101b4bd6-06a1-4cc1-900e-8806ee575034"
-					(reference "#PWR080")
+					(reference "#PWR085")
 					(unit 1)
 				)
@@
 		(dnp no)
 		(fields_autoplaced yes)
-		(property "Reference" "#PWR081"
+		(property "Reference" "#PWR086"
 			(at 226.06 104.14 0)
 			(effects
@@
 			(project "frank_m2"
 				(path "/8c0b3d8b-46d3-4173-ab1e-a61765f77d61/101b4bd6-06a1-4cc1-900e-8806ee575034"
-					(reference "#PWR081")
+					(reference "#PWR086")
 					(unit 1)
 				)
@@
 		(on_board yes)
 		(dnp no)
-		(property "Reference" "R24"
+		(property "Reference" "R25"
 			(at 119.634 97.536 90)
 			(effects
@@
 			(project "frank_m2"
 				(path "/8c0b3d8b-46d3-4173-ab1e-a61765f77d61/101b4bd6-06a1-4cc1-900e-8806ee575034"
-					(reference "R24")
+					(reference "R25")
 					(unit 1)
 				)
@@
 		(on_board yes)
 		(dnp no)
-		(property "Reference" "R26"
+		(property "Reference" "R27"
 			(at 119.634 112.776 90)
 			(effects
@@
 			(project "frank_m2"
 				(path "/8c0b3d8b-46d3-4173-ab1e-a61765f77d61/101b4bd6-06a1-4cc1-900e-8806ee575034"
-					(reference "R26")
+					(reference "R27")
 					(unit 1)
 				)
