File: lab/frank_m2_pro/usb_hub.kicad_sch (KiCad schematic)
At the start: 2 parts, among them U5 MW7211A

Commit message: FRANK M1 Pro HW 1.00
Other:
- title: ${NAME} -> ${NAME} ${MODEL}
Changed lines of the file:
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@@
 	(paper "A4")
 	(title_block
-		(title "${NAME}")
-		(date "2025-04-24")
+		(title "${NAME} ${MODEL}")
+		(date "${DATE}")
 		(rev "${VERSION}")
 		(company "Mikhail Matveev")
-		(comment 1 "https://github.com/xtremespb/frank")
+		(comment 1 "https://github.com/rh1tech/frank")
 	)
 	(junction
