File: lab/frank_pro_m2/audio_multiplexer.kicad_sch (KiCad schematic)
At the start: 3 parts, among them U13 74HC4052D

Commit message: Rename footprints, 3D models to KiCad standard naming
lab/xt8086:
- Renamed 22 footprints (spaces/parens/IPNs -> KiCad style)
- Renamed 13 3D models, normalized all to .step
- Fixed FRANK: prefix -> xt8086: in symbol/schematic refs
- Fixed bare 3D model path without ${KIPRJMOD} prefix

lab/frank_pro_m2:
- Removed 11 unused footprints
- Renamed 32 footprints to KiCad standard naming
- Renamed 33 3D models, normalized all to .step
- Fixed wrong library prefixes (LIBS:, DC-005-5A-2.0:, MSK12C02:, etc.)
Parts:
- U13: footprint FRANK:SOP-16 -> FRANK:SOP-16_P1.27mm
Changed lines of the file:
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@@
 			)
 		)
-		(property "Footprint" "FRANK:SOP-16"
+		(property "Footprint" "FRANK:SOP-16_P1.27mm"
 			(at 156.21 188.9 0)
 			(hide yes)
