File: lab/frank_pro_m2/display.kicad_sch (KiCad schematic)
At the start: 1 part, among them J8 Pin Header 1x08

Commit message: LAB WIP
Parts:
- renumbered J8 to J9
Changed lines of the file:
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@@
 		(dnp no)
 		(fields_autoplaced yes)
-		(property "Reference" "#PWR076"
+		(property "Reference" "#PWR089"
 			(at 166.37 95.25 0)
 			(effects
@@
 			(project "frank_m2"
 				(path "/8c0b3d8b-46d3-4173-ab1e-a61765f77d61/3504beb8-2939-46b0-9c32-2648908a1056"
-					(reference "#PWR076")
+					(reference "#PWR089")
 					(unit 1)
 				)
@@
 		(dnp no)
 		(fields_autoplaced yes)
-		(property "Reference" "#PWR075"
+		(property "Reference" "#PWR088"
 			(at 156.21 92.71 0)
 			(effects
@@
 			(project "frank_m2"
 				(path "/8c0b3d8b-46d3-4173-ab1e-a61765f77d61/3504beb8-2939-46b0-9c32-2648908a1056"
-					(reference "#PWR075")
+					(reference "#PWR088")
 					(unit 1)
 				)
@@
 		(dnp no)
 		(fields_autoplaced yes)
-		(property "Reference" "J8"
+		(property "Reference" "J9"
 			(at 135.255 87.63 0)
 			(effects
@@
 			(project "frank_m2"
 				(path "/8c0b3d8b-46d3-4173-ab1e-a61765f77d61/3504beb8-2939-46b0-9c32-2648908a1056"
-					(reference "J8")
+					(reference "J9")
 					(unit 1)
 				)

Commit message: Rename footprints, 3D models to KiCad standard naming
lab/xt8086:
- Renamed 22 footprints (spaces/parens/IPNs -> KiCad style)
- Renamed 13 3D models, normalized all to .step
- Fixed FRANK: prefix -> xt8086: in symbol/schematic refs
- Fixed bare 3D model path without ${KIPRJMOD} prefix

lab/frank_pro_m2:
- Removed 11 unused footprints
- Renamed 32 footprints to KiCad standard naming
- Renamed 33 3D models, normalized all to .step
- Fixed wrong library prefixes (LIBS:, DC-005-5A-2.0:, MSK12C02:, etc.)
Parts:
- J9: footprint FRANK:Connector Female 1.25 JST 8P -> FRANK:JST_GH_1x08_P1.25mm
Changed lines of the file:
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@@
 			)
 		)
-		(property "Footprint" "FRANK:Connector Female 1.25 JST 8P"
+		(property "Footprint" "FRANK:JST_GH_1x08_P1.25mm"
 			(at 134.62 100.33 0)
 			(hide yes)
