File: lab/frank_pro_m2/power.kicad_sch (KiCad schematic)
At the start: 30 parts, among them J3 DC-005-5A-2.0, J4 USB4215-03-A, U1 MP1584EN-LF-Z, U2 USBLC6-2SC6, U3 AMS1117 3.3

Commit message: LAB WIP
Parts:
- renumbered J3 to J4, J4 to J5, S2 to S7
Changed lines of the file:
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@@
 		(dnp no)
 		(fields_autoplaced yes)
-		(property "Reference" "#PWR014"
+		(property "Reference" "#PWR027"
 			(at 78.74 82.55 0)
 			(effects
@@
 			(project "fastbeta_pwt"
 				(path "/8c0b3d8b-46d3-4173-ab1e-a61765f77d61/84d5e8f7-bda8-4f18-8ff8-1a8273c38b01"
-					(reference "#PWR014")
+					(reference "#PWR027")
 					(unit 1)
 				)
@@
 		(on_board yes)
 		(dnp no)
-		(property "Reference" "#PWR022"
+		(property "Reference" "#PWR035"
 			(at 148.59 135.89 0)
 			(effects
@@
 			(project "frank_m2_pro"
 				(path "/8c0b3d8b-46d3-4173-ab1e-a61765f77d61/84d5e8f7-bda8-4f18-8ff8-1a8273c38b01"
-					(reference "#PWR022")
+					(reference "#PWR035")
 					(unit 1)
 				)
@@
 		(dnp no)
 		(fields_autoplaced yes)
-		(property "Reference" "#PWR034"
+		(property "Reference" "#PWR047"
 			(at 214.63 91.44 0)
 			(effects
@@
 			(project "frank2"
 				(path "/8c0b3d8b-46d3-4173-ab1e-a61765f77d61/84d5e8f7-bda8-4f18-8ff8-1a8273c38b01"
-					(reference "#PWR034")
+					(reference "#PWR047")
 					(unit 1)
 				)
@@
 		(on_board yes)
 		(dnp no)
-		(property "Reference" "#PWR012"
+		(property "Reference" "#PWR025"
 			(at 55.88 116.84 0)
 			(effects
@@
 			(project "frank_pro_m2"
 				(path "/8c0b3d8b-46d3-4173-ab1e-a61765f77d61/84d5e8f7-bda8-4f18-8ff8-1a8273c38b01"
-					(reference "#PWR012")
+					(reference "#PWR025")
 					(unit 1)
 				)
@@
 		(dnp no)
 		(fields_autoplaced yes)
-		(property "Reference" "#PWR031"
+		(property "Reference" "#PWR044"
 			(at 191.77 85.09 0)
 			(effects
@@
 			(project "fastbeta_pwt"
 				(path "/8c0b3d8b-46d3-4173-ab1e-a61765f77d61/84d5e8f7-bda8-4f18-8ff8-1a8273c38b01"
-					(reference "#PWR031")
+					(reference "#PWR044")
 					(unit 1)
 				)
@@
 		(dnp no)
 		(fields_autoplaced yes)
-		(property "Reference" "#PWR017"
+		(property "Reference" "#PWR030"
 			(at 110.49 97.79 0)
 			(effects
@@
 			(project "fastbeta_pwt"
 				(path "/8c0b3d8b-46d3-4173-ab1e-a61765f77d61/84d5e8f7-bda8-4f18-8ff8-1a8273c38b01"
-					(reference "#PWR017")
+					(reference "#PWR030")
 					(unit 1)
 				)
@@
 		(on_board yes)
 		(dnp no)
-		(property "Reference" "#PWR023"
+		(property "Reference" "#PWR036"
 			(at 151.13 140.97 0)
 			(effects
@@
 			(project "frank_m2_pro"
 				(path "/8c0b3d8b-46d3-4173-ab1e-a61765f77d61/84d5e8f7-bda8-4f18-8ff8-1a8273c38b01"
-					(reference "#PWR023")
+					(reference "#PWR036")
 					(unit 1)
 				)
@@
 		(on_board yes)
 		(dnp no)
-		(property "Reference" "J4"
+		(property "Reference" "J5"
 			(at 128.27 116.84 0)
 			(effects
@@
 			(project "frank_m2_pro"
 				(path "/8c0b3d8b-46d3-4173-ab1e-a61765f77d61/84d5e8f7-bda8-4f18-8ff8-1a8273c38b01"
-					(reference "J4")
+					(reference "J5")
 					(unit 1)
 				)
@@
 		(dnp no)
 		(fields_autoplaced yes)
-		(property "Reference" "#PWR024"
+		(property "Reference" "#PWR037"
 			(at 152.4 86.36 0)
 			(effects
@@
 			(project "fastbeta_pwt"
 				(path "/8c0b3d8b-46d3-4173-ab1e-a61765f77d61/84d5e8f7-bda8-4f18-8ff8-1a8273c38b01"
-					(reference "#PWR024")
+					(reference "#PWR037")
 					(unit 1)
 				)
@@
 		(dnp no)
 		(fields_autoplaced yes)
-		(property "Reference" "#PWR015"
+		(property "Reference" "#PWR028"
 			(at 86.36 82.55 0)
 			(effects
@@
 			(project "fastbeta_pwt"
 				(path "/8c0b3d8b-46d3-4173-ab1e-a61765f77d61/84d5e8f7-bda8-4f18-8ff8-1a8273c38b01"
-					(reference "#PWR015")
+					(reference "#PWR028")
 					(unit 1)
 				)
@@
 		(on_board yes)
 		(dnp no)
-		(property "Reference" "#PWR021"
+		(property "Reference" "#PWR034"
 			(at 148.59 120.65 0)
 			(effects
@@
 			(project "frank_m2_pro"
 				(path "/8c0b3d8b-46d3-4173-ab1e-a61765f77d61/84d5e8f7-bda8-4f18-8ff8-1a8273c38b01"
-					(reference "#PWR021")
+					(reference "#PWR034")
 					(unit 1)
 				)
@@
 		(dnp no)
 		(fields_autoplaced yes)
-		(property "Reference" "#PWR033"
+		(property "Reference" "#PWR046"
 			(at 198.12 85.09 0)
 			(effects
@@
 			(project "fastbeta_pwt"
 				(path "/8c0b3d8b-46d3-4173-ab1e-a61765f77d61/84d5e8f7-bda8-4f18-8ff8-1a8273c38b01"
-					(reference "#PWR033")
+					(reference "#PWR046")
 					(unit 1)
 				)
@@
 		(on_board yes)
 		(dnp no)
-		(property "Reference" "#PWR030"
+		(property "Reference" "#PWR043"
 			(at 186.69 139.7 0)
 			(effects
@@
 			(project "frank_pro_m2"
 				(path "/8c0b3d8b-46d3-4173-ab1e-a61765f77d61/84d5e8f7-bda8-4f18-8ff8-1a8273c38b01"
-					(reference "#PWR030")
+					(reference "#PWR043")
 					(unit 1)
 				)
@@
 		(dnp no)
 		(fields_autoplaced yes)
-		(property "Reference" "#PWR028"
+		(property "Reference" "#PWR041"
 			(at 185.42 85.09 0)
 			(effects
@@
 			(project "fastbeta_pwt"
 				(path "/8c0b3d8b-46d3-4173-ab1e-a61765f77d61/84d5e8f7-bda8-4f18-8ff8-1a8273c38b01"
-					(reference "#PWR028")
+					(reference "#PWR041")
 					(unit 1)
 				)
@@
 		(on_board yes)
 		(dnp no)
-		(property "Reference" "S2"
+		(property "Reference" "S7"
 			(at 86.36 107.9501 0)
 			(effects
@@
 			(project "frank_m2_pro"
 				(path "/8c0b3d8b-46d3-4173-ab1e-a61765f77d61/84d5e8f7-bda8-4f18-8ff8-1a8273c38b01"
-					(reference "S2")
+					(reference "S7")
 					(unit 1)
 				)
@@
 		(on_board yes)
 		(dnp no)
-		(property "Reference" "#PWR020"
+		(property "Reference" "#PWR033"
 			(at 148.59 113.03 0)
 			(effects
@@
 			(project "frank_m2_pro"
 				(path "/8c0b3d8b-46d3-4173-ab1e-a61765f77d61/84d5e8f7-bda8-4f18-8ff8-1a8273c38b01"
-					(reference "#PWR020")
+					(reference "#PWR033")
 					(unit 1)
 				)
@@
 		(dnp no)
 		(fields_autoplaced yes)
-		(property "Reference" "#PWR025"
+		(property "Reference" "#PWR038"
 			(at 162.56 41.91 0)
 			(effects
@@
 			(project "fastbeta_pwt"
 				(path "/8c0b3d8b-46d3-4173-ab1e-a61765f77d61/84d5e8f7-bda8-4f18-8ff8-1a8273c38b01"
-					(reference "#PWR025")
+					(reference "#PWR038")
 					(unit 1)
 				)
@@
 		(dnp no)
 		(fields_autoplaced yes)
-		(property "Reference" "J3"
+		(property "Reference" "J4"
 			(at 47.4889 97.79 0)
 			(effects
@@
 			(project "frank_m1"
 				(path "/8c0b3d8b-46d3-4173-ab1e-a61765f77d61/84d5e8f7-bda8-4f18-8ff8-1a8273c38b01"
-					(reference "J3")
+					(reference "J4")
 					(unit 1)
 				)
@@
 		(dnp no)
 		(fields_autoplaced yes)
-		(property "Reference" "#PWR026"
+		(property "Reference" "#PWR039"
 			(at 160.02 115.57 0)
 			(effects
@@
 			(project ""
 				(path "/8c0b3d8b-46d3-4173-ab1e-a61765f77d61/84d5e8f7-bda8-4f18-8ff8-1a8273c38b01"
-					(reference "#PWR026")
+					(reference "#PWR039")
 					(unit 1)
 				)
@@
 		(dnp no)
 		(fields_autoplaced yes)
-		(property "Reference" "#PWR018"
+		(property "Reference" "#PWR031"
 			(at 119.38 97.79 0)
 			(effects
@@
 			(project "fastbeta_pwt"
 				(path "/8c0b3d8b-46d3-4173-ab1e-a61765f77d61/84d5e8f7-bda8-4f18-8ff8-1a8273c38b01"
-					(reference "#PWR018")
+					(reference "#PWR031")
 					(unit 1)
 				)
@@
 		(dnp no)
 		(fields_autoplaced yes)
-		(property "Reference" "#PWR027"
+		(property "Reference" "#PWR040"
 			(at 171.45 143.51 0)
 			(effects
@@
 			(project "frank_pro_m2"
 				(path "/8c0b3d8b-46d3-4173-ab1e-a61765f77d61/84d5e8f7-bda8-4f18-8ff8-1a8273c38b01"
-					(reference "#PWR027")
+					(reference "#PWR040")
 					(unit 1)
 				)
@@
 		(dnp no)
 		(fields_autoplaced yes)
-		(property "Reference" "#PWR036"
+		(property "Reference" "#PWR049"
 			(at 236.22 63.5 0)
 			(effects
@@
 			(project "fastbeta_pwt"
 				(path "/8c0b3d8b-46d3-4173-ab1e-a61765f77d61/84d5e8f7-bda8-4f18-8ff8-1a8273c38b01"
-					(reference "#PWR036")
+					(reference "#PWR049")
 					(unit 1)
 				)
@@
 		(dnp no)
 		(fields_autoplaced yes)
-		(property "Reference" "#PWR032"
+		(property "Reference" "#PWR045"
 			(at 198.12 58.42 0)
 			(effects
@@
 			(project ""
 				(path "/8c0b3d8b-46d3-4173-ab1e-a61765f77d61/84d5e8f7-bda8-4f18-8ff8-1a8273c38b01"
-					(reference "#PWR032")
+					(reference "#PWR045")
 					(unit 1)
 				)
@@
 		(dnp no)
 		(fields_autoplaced yes)
-		(property "Reference" "#PWR019"
+		(property "Reference" "#PWR032"
 			(at 132.08 97.79 0)
 			(effects
@@
 			(project "fastbeta_pwt"
 				(path "/8c0b3d8b-46d3-4173-ab1e-a61765f77d61/84d5e8f7-bda8-4f18-8ff8-1a8273c38b01"
-					(reference "#PWR019")
+					(reference "#PWR032")
 					(unit 1)
 				)
@@
 		(dnp no)
 		(fields_autoplaced yes)
-		(property "Reference" "#PWR013"
+		(property "Reference" "#PWR026"
 			(at 71.12 82.55 0)
 			(effects
@@
 			(project "fastbeta_pwt"
 				(path "/8c0b3d8b-46d3-4173-ab1e-a61765f77d61/84d5e8f7-bda8-4f18-8ff8-1a8273c38b01"
-					(reference "#PWR013")
+					(reference "#PWR026")
 					(unit 1)
 				)
@@
 		(on_board yes)
 		(dnp no)
-		(property "Reference" "#PWR029"
+		(property "Reference" "#PWR042"
 			(at 186.69 121.92 0)
 			(effects
@@
 			(project "frank_pro_m2"
 				(path "/8c0b3d8b-46d3-4173-ab1e-a61765f77d61/84d5e8f7-bda8-4f18-8ff8-1a8273c38b01"
-					(reference "#PWR029")
+					(reference "#PWR042")
 					(unit 1)
 				)
@@
 		(dnp no)
 		(fields_autoplaced yes)
-		(property "Reference" "#PWR016"
+		(property "Reference" "#PWR029"
 			(at 104.14 80.01 0)
 			(effects
@@
 			(project "fastbeta_pwt"
 				(path "/8c0b3d8b-46d3-4173-ab1e-a61765f77d61/84d5e8f7-bda8-4f18-8ff8-1a8273c38b01"
-					(reference "#PWR016")
+					(reference "#PWR029")
 					(unit 1)
 				)
@@
 		(dnp no)
 		(fields_autoplaced yes)
-		(property "Reference" "#PWR035"
+		(property "Reference" "#PWR048"
 			(at 234.95 91.44 0)
 			(effects
@@
 			(project ""
 				(path "/8c0b3d8b-46d3-4173-ab1e-a61765f77d61/84d5e8f7-bda8-4f18-8ff8-1a8273c38b01"
-					(reference "#PWR035")
+					(reference "#PWR048")
 					(unit 1)
 				)
@@
 		(dnp no)
 		(fields_autoplaced yes)
-		(property "Reference" "#PWR037"
+		(property "Reference" "#PWR050"
 			(at 246.38 73.66 0)
 			(effects
@@
 			(project "fastbeta_pwt"
 				(path "/8c0b3d8b-46d3-4173-ab1e-a61765f77d61/84d5e8f7-bda8-4f18-8ff8-1a8273c38b01"
-					(reference "#PWR037")
+					(reference "#PWR050")
 					(unit 1)
 				)

Commit message: Rename footprints, 3D models to KiCad standard naming
lab/xt8086:
- Renamed 22 footprints (spaces/parens/IPNs -> KiCad style)
- Renamed 13 3D models, normalized all to .step
- Fixed FRANK: prefix -> xt8086: in symbol/schematic refs
- Fixed bare 3D model path without ${KIPRJMOD} prefix

lab/frank_pro_m2:
- Removed 11 unused footprints
- Renamed 32 footprints to KiCad standard naming
- Renamed 33 3D models, normalized all to .step
- Fixed wrong library prefixes (LIBS:, DC-005-5A-2.0:, MSK12C02:, etc.)
Parts:
- C1: footprint FRANK:Capacitor (Radial_D8.0mm_P3.50mm) -> FRANK:C_Radial_D8.0mm_P3.50mm
- C8: footprint FRANK:Capacitor (Radial_D6.3mm_P2.50mm) -> FRANK:C_Radial_D6.3mm_P2.50mm
- D1: footprint FRANK:SS34 -> FRANK:D_SMA_SS34
- J4: footprint FRANK:XKB_DC-005-5A-2.0 -> FRANK:BarrelJack_DC-005
- J5: footprint FRANK:USB Type C -> FRANK:USB_C_Receptacle
- L1: footprint FRANK:CDRH104RNP -> FRANK:Inductor_CDRH104RNP
- LD1: footprint FRANK:LED (0805) -> FRANK:LED_0805
- S7: footprint FRANK:SK12D07VG3NS -> FRANK:Switch_Slide_SK12D07VG3NS
- U1: footprint FRANK:SOIC127P600X170-9N -> FRANK:SOIC-9_P1.27mm
Changed lines of the file:
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@@
 			)
 		)
-		(property "Footprint" "FRANK:SOIC127P600X170-9N"
+		(property "Footprint" "FRANK:SOIC-9_P1.27mm"
 			(at 143.51 153.34 0)
 			(hide yes)
@@
 			)
 		)
-		(property "Footprint" "FRANK:LED (0805)"
+		(property "Footprint" "FRANK:LED_0805"
 			(at 224.79 91.44 0)
 			(hide yes)
@@
 			)
 		)
-		(property "Footprint" "FRANK:USB Type C"
+		(property "Footprint" "FRANK:USB_C_Receptacle"
 			(at 138.43 128.27 0)
 			(hide yes)
@@
 			)
 		)
-		(property "Footprint" "FRANK:SS34"
+		(property "Footprint" "FRANK:D_SMA_SS34"
 			(at 162.56 54.61 0)
 			(hide yes)
@@
 			)
 		)
-		(property "Footprint" "FRANK:SK12D07VG3NS"
+		(property "Footprint" "FRANK:Switch_Slide_SK12D07VG3NS"
 			(at 86.36 16.84 0)
 			(hide yes)
@@
 			)
 		)
-		(property "Footprint" "FRANK:XKB_DC-005-5A-2.0"
+		(property "Footprint" "FRANK:BarrelJack_DC-005"
 			(at 48.26 106.68 0)
 			(hide yes)
@@
 			)
 		)
-		(property "Footprint" "FRANK:Capacitor (Radial_D6.3mm_P2.50mm)"
+		(property "Footprint" "FRANK:C_Radial_D6.3mm_P2.50mm"
 			(at 198.12 72.39 0)
 			(hide yes)
@@
 			)
 		)
-		(property "Footprint" "FRANK:CDRH104RNP"
+		(property "Footprint" "FRANK:Inductor_CDRH104RNP"
 			(at 171.45 63.5 0)
 			(hide yes)
@@
 			)
 		)
-		(property "Footprint" "FRANK:Capacitor (Radial_D8.0mm_P3.50mm)"
+		(property "Footprint" "FRANK:C_Radial_D8.0mm_P3.50mm"
 			(at 71.12 73.66 0)
 			(hide yes)

Commit message: Rename footprints and 3D models in lab/tinyfrank_m2p2
- Removed 2 unused footprints (ESP-01, SO-16)
- Renamed 18 footprints to KiCad standard naming
- Renamed 15 3D models, normalized all to .step
- Fixed wrong library prefixes (FRANK:, LIBS:, MSK12C02:, etc.)
Parts:
- U3: footprint FRANK:SOT-223 -> Package_TO_SOT_SMD:SOT-223-3_TabPin2
Changed lines of the file:
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@@
 			)
 		)
-		(property "Description" ""
+		(property "Description" "DC Power Receptacle Jack, Through Hole，Right Angle"
 			(at 48.26 106.68 0)
 			(hide yes)
@@
 			)
 		)
-		(property "Footprint" "FRANK:SOT-223"
+		(property "Footprint" "Package_TO_SOT_SMD:SOT-223-3_TabPin2"
 			(at 217.17 58.42 0)
 			(hide yes)
@@
 			)
 		)
-		(property "Description" ""
+		(property "Description" "1A Low drop-out regulator, Fixed Output 3.3V, SOT-223"
 			(at 217.17 63.5 0)
 			(hide yes)
