File: hardware/frank_m2/audio_multiplexer.kicad_sch (KiCad schematic)
At the start: 3 parts, among them U9 74HC4052D

Commit message: Rename and localize hardware/frank_m2 footprints, 3D models
- Removed 5 unused footprints, 1 unused 3D model
- Renamed 28 footprints to KiCad standard naming
- Renamed 30 3D models, normalized all to .step
- Copied 12 system 3D models (KiCad built-in) to local 3d/ dir
- Replaced all ${KICADx_3DMODEL_DIR} refs with ${KIPRJMOD}/3d/
- Fixed wrong library prefixes (LIBS:, DC-005-5A-2.0:, etc.)
- Project is now fully self-contained (no external 3D model dependencies)
Parts:
- U9: footprint FRANK:SOP-16 -> FRANK:SOP-16_P1.27mm

Commit message: Move hardware/frank_m2 to frank-lab repo, restore v2.06 from master
Parts:
- U9: footprint FRANK:SOP-16_P1.27mm -> FRANK:SOP-16
