File: hardware/megafrank/usbstack.kicad_sch (KiCad schematic)
At the start: 7 parts, among them J19 SS-52100-004

Commit message: Add Megafrank-1
- Two stacked USB-A ports were added on front board edge. 4 USB-A host ports total
- Power barrel 5mm connector was moved to right edge of the board
- ESP-RESET connected to PGPIO36 (optional, available if S11 jumper is closed)
Parts:
- renumbered C50 to C52, C51 to C53, J19 to J21, R121 to R133, R122 to R134, R123 to R135, R124 to R136
Changed lines of the file:
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@@
 		(dnp no)
 		(fields_autoplaced yes)
-		(property "Reference" "J19"
+		(property "Reference" "J21"
 			(at 121.92 68.58 0)
 			(show_name no)
@@
 		(instances
 			(project "megafrank"
+				(path "/8c0b3d8b-46d3-4173-ab1e-a61765f77d61/3817edc5-ec38-47b6-a331-73c18c09aca9"
+					(reference "J21")
+					(unit 1)
+				)
 				(path "/8c0b3d8b-46d3-4173-ab1e-a61765f77d61/cc3b493c-84ed-45fe-8a9e-a3bf2d009620"
 					(reference "J19")
@@
 		(in_pos_files yes)
 		(dnp no)
-		(property "Reference" "C50"
+		(property "Reference" "C52"
 			(at 168.021 82.6516 0)
 			(show_name no)
@@
 		(instances
 			(project "megafrank"
+				(path "/8c0b3d8b-46d3-4173-ab1e-a61765f77d61/3817edc5-ec38-47b6-a331-73c18c09aca9"
+					(reference "C52")
+					(unit 1)
+				)
 				(path "/8c0b3d8b-46d3-4173-ab1e-a61765f77d61/cc3b493c-84ed-45fe-8a9e-a3bf2d009620"
 					(reference "C50")
@@
 		(in_pos_files yes)
 		(dnp no)
-		(property "Reference" "R122"
+		(property "Reference" "R134"
 			(at 145.542 104.14 90)
 			(show_name no)
@@
 		(instances
 			(project "megafrank"
+				(path "/8c0b3d8b-46d3-4173-ab1e-a61765f77d61/3817edc5-ec38-47b6-a331-73c18c09aca9"
+					(reference "R134")
+					(unit 1)
+				)
 				(path "/8c0b3d8b-46d3-4173-ab1e-a61765f77d61/cc3b493c-84ed-45fe-8a9e-a3bf2d009620"
 					(reference "R122")
@@
 		(in_pos_files yes)
 		(dnp no)
-		(property "Reference" "C51"
+		(property "Reference" "C53"
 			(at 179.451 82.6516 0)
 			(show_name no)
@@
 		(instances
 			(project "megafrank"
+				(path "/8c0b3d8b-46d3-4173-ab1e-a61765f77d61/3817edc5-ec38-47b6-a331-73c18c09aca9"
+					(reference "C53")
+					(unit 1)
+				)
 				(path "/8c0b3d8b-46d3-4173-ab1e-a61765f77d61/cc3b493c-84ed-45fe-8a9e-a3bf2d009620"
 					(reference "C51")
@@
 		(in_pos_files yes)
 		(dnp no)
-		(property "Reference" "#PWR0192"
+		(property "Reference" "#PWR0198"
 			(at 135.89 78.74 0)
 			(hide yes)
@@
 		(instances
 			(project "megafrank"
+				(path "/8c0b3d8b-46d3-4173-ab1e-a61765f77d61/3817edc5-ec38-47b6-a331-73c18c09aca9"
+					(reference "#PWR0198")
+					(unit 1)
+				)
 				(path "/8c0b3d8b-46d3-4173-ab1e-a61765f77d61/cc3b493c-84ed-45fe-8a9e-a3bf2d009620"
 					(reference "#PWR0192")
@@
 		(in_pos_files yes)
 		(dnp no)
-		(property "Reference" "#PWR0194"
+		(property "Reference" "#PWR0200"
 			(at 165.1 95.25 0)
 			(hide yes)
@@
 		(instances
 			(project "megafrank"
+				(path "/8c0b3d8b-46d3-4173-ab1e-a61765f77d61/3817edc5-ec38-47b6-a331-73c18c09aca9"
+					(reference "#PWR0200")
+					(unit 1)
+				)
 				(path "/8c0b3d8b-46d3-4173-ab1e-a61765f77d61/cc3b493c-84ed-45fe-8a9e-a3bf2d009620"
 					(reference "#PWR0194")
@@
 		(in_pos_files yes)
 		(dnp no)
-		(property "Reference" "R123"
+		(property "Reference" "R135"
 			(at 154.432 102.87 90)
 			(show_name no)
@@
 		(instances
 			(project "megafrank"
+				(path "/8c0b3d8b-46d3-4173-ab1e-a61765f77d61/3817edc5-ec38-47b6-a331-73c18c09aca9"
+					(reference "R135")
+					(unit 1)
+				)
 				(path "/8c0b3d8b-46d3-4173-ab1e-a61765f77d61/cc3b493c-84ed-45fe-8a9e-a3bf2d009620"
 					(reference "R123")
@@
 		(in_pos_files yes)
 		(dnp no)
-		(property "Reference" "#PWR0195"
+		(property "Reference" "#PWR0201"
 			(at 176.53 95.25 0)
 			(hide yes)
@@
 		(instances
 			(project "megafrank"
+				(path "/8c0b3d8b-46d3-4173-ab1e-a61765f77d61/3817edc5-ec38-47b6-a331-73c18c09aca9"
+					(reference "#PWR0201")
+					(unit 1)
+				)
 				(path "/8c0b3d8b-46d3-4173-ab1e-a61765f77d61/cc3b493c-84ed-45fe-8a9e-a3bf2d009620"
 					(reference "#PWR0195")
@@
 		(in_pos_files yes)
 		(dnp no)
-		(property "Reference" "R121"
+		(property "Reference" "R133"
 			(at 141.732 97.79 90)
 			(show_name no)
@@
 		(instances
 			(project "megafrank"
+				(path "/8c0b3d8b-46d3-4173-ab1e-a61765f77d61/3817edc5-ec38-47b6-a331-73c18c09aca9"
+					(reference "R133")
+					(unit 1)
+				)
 				(path "/8c0b3d8b-46d3-4173-ab1e-a61765f77d61/cc3b493c-84ed-45fe-8a9e-a3bf2d009620"
 					(reference "R121")
@@
 		(in_pos_files yes)
 		(dnp no)
-		(property "Reference" "#PWR0193"
+		(property "Reference" "#PWR0199"
 			(at 142.24 78.74 0)
 			(hide yes)
@@
 		(instances
 			(project "megafrank"
+				(path "/8c0b3d8b-46d3-4173-ab1e-a61765f77d61/3817edc5-ec38-47b6-a331-73c18c09aca9"
+					(reference "#PWR0199")
+					(unit 1)
+				)
 				(path "/8c0b3d8b-46d3-4173-ab1e-a61765f77d61/cc3b493c-84ed-45fe-8a9e-a3bf2d009620"
 					(reference "#PWR0193")
@@
 		(dnp no)
 		(fields_autoplaced yes)
-		(property "Reference" "#PWR0191"
+		(property "Reference" "#PWR0197"
 			(at 121.92 111.76 0)
 			(hide yes)
@@
 		(instances
 			(project "megafrank"
+				(path "/8c0b3d8b-46d3-4173-ab1e-a61765f77d61/3817edc5-ec38-47b6-a331-73c18c09aca9"
+					(reference "#PWR0197")
+					(unit 1)
+				)
 				(path "/8c0b3d8b-46d3-4173-ab1e-a61765f77d61/cc3b493c-84ed-45fe-8a9e-a3bf2d009620"
 					(reference "#PWR0191")
@@
 		(in_pos_files yes)
 		(dnp no)
-		(property "Reference" "R124"
+		(property "Reference" "R136"
 			(at 158.242 109.22 90)
 			(show_name no)
@@
 		(instances
 			(project "megafrank"
+				(path "/8c0b3d8b-46d3-4173-ab1e-a61765f77d61/3817edc5-ec38-47b6-a331-73c18c09aca9"
+					(reference "R136")
+					(unit 1)
+				)
 				(path "/8c0b3d8b-46d3-4173-ab1e-a61765f77d61/cc3b493c-84ed-45fe-8a9e-a3bf2d009620"
 					(reference "R124")
