File: hardware/dino_z80/sd.kicad_sch (KiCad schematic)
At the start: 2 parts, among them J3 104031-0811

Commit message: feat: dino_z80 stereo audio with a PAM8403 speaker amp
Replace the buzzer with a Sound sheet: RC filters on GP46/GP44, an LM358
buffer, a 3-way DIP switch (HDMI L, HDMI R, speaker) and a stereo jack.
The Speaker sub-sheet mixes L+R into a PAM8403 driving a CVS-2308 speaker.

Libraries: fix the mirrored SOT-23 land pattern, replace the SOIC-8 land
pattern with the standard 4.95 mm span, add PAM8403D, LM358 and CVS-2308,
and rename the MS9288A footprint to QFN-48 6x6 to match its package.
Parts:
- renumbered C9 to C21
Changed lines of the file:
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@@
 		(in_pos_files yes)
 		(dnp no)
-		(property "Reference" "C9"
+		(property "Reference" "C21"
 			(at 120.7516 94.869 0)
 			(show_name no)
@@
 			(project "dino_z80"
 				(path "/8c0b3d8b-46d3-4173-ab1e-a61765f77d61/2e81912e-397c-4129-8da5-abf37a4f2667"
-					(reference "C9")
+					(reference "C21")
 					(unit 1)
 				)
@@
 		(dnp no)
 		(fields_autoplaced yes)
-		(property "Reference" "#PWR044"
+		(property "Reference" "#PWR066"
 			(at 132.08 99.06 0)
 			(hide yes)
@@
 			(project "dino_z80"
 				(path "/8c0b3d8b-46d3-4173-ab1e-a61765f77d61/2e81912e-397c-4129-8da5-abf37a4f2667"
-					(reference "#PWR044")
+					(reference "#PWR066")
 					(unit 1)
 				)
@@
 		(dnp no)
 		(fields_autoplaced yes)
-		(property "Reference" "#PWR040"
+		(property "Reference" "#PWR065"
 			(at 111.76 97.79 0)
 			(hide yes)
@@
 			(project "dino_z80"
 				(path "/8c0b3d8b-46d3-4173-ab1e-a61765f77d61/2e81912e-397c-4129-8da5-abf37a4f2667"
-					(reference "#PWR040")
+					(reference "#PWR065")
 					(unit 1)
 				)
@@
 		(dnp no)
 		(fields_autoplaced yes)
-		(property "Reference" "#PWR047"
+		(property "Reference" "#PWR068"
 			(at 194.31 113.03 0)
 			(hide yes)
@@
 			(project "dino_z80"
 				(path "/8c0b3d8b-46d3-4173-ab1e-a61765f77d61/2e81912e-397c-4129-8da5-abf37a4f2667"
-					(reference "#PWR047")
+					(reference "#PWR068")
 					(unit 1)
 				)
@@
 		(dnp no)
 		(fields_autoplaced yes)
-		(property "Reference" "#PWR045"
+		(property "Reference" "#PWR067"
 			(at 138.43 102.87 0)
 			(hide yes)
@@
 			(project "dino_z80"
 				(path "/8c0b3d8b-46d3-4173-ab1e-a61765f77d61/2e81912e-397c-4129-8da5-abf37a4f2667"
-					(reference "#PWR045")
-					(unit 1)
-				)
+					(reference "#PWR067")
+					(unit 1)
+				)

Commit message: chore: dino_z80 standard values, Y2 for the oscillator, datasheet links checked
- Values in SI form: 10kΩ, 200Ω, 100nF, 10µF, 3.3µH, 220Ω@100MHz beads,
  12MHz / 24.576MHz clocks. Schematic and board agree.
- X1 (12 MHz oscillator) renamed Y2, crystals and oscillators both Y.
- Links: Y2 datasheet is the ASE series (was ASV, a 7x5 part); S1/S5 and
  S3/S4 point at the Littelfuse C&K datasheets (KMR2 link was dead);
  J4 gets the JST SH datasheet instead of 2.54 mm header links; D5 gets
  the listing that has 1N5819WS; the Vishay datasheet on R1/R2/R35/R36/
  R41/R42 moves from AliExpress to Datasheet; Y1 loses the LCSC record of
  a 12 MHz 3225 crystal; datasheets added for U1, U4, U7, D3.
- LS1 and U11 descriptions tidied.

DRC: 0 errors, 0 unconnected, 0 schematic parity. ERC: 0.
Parts:
- C21: value 100n -> 100nF
Changed lines of the file:
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@@
 			)
 		)
-		(property "Value" "100n"
+		(property "Value" "100nF"
 			(at 123.063 94.869 0)
 			(show_name no)
