File: hardware/dino_z80/usb_hub.kicad_sch (KiCad schematic)
At the start: 5 parts, among them U4 MW7211A

Commit message: feat: dino_z80 stereo audio with a PAM8403 speaker amp
Replace the buzzer with a Sound sheet: RC filters on GP46/GP44, an LM358
buffer, a 3-way DIP switch (HDMI L, HDMI R, speaker) and a stereo jack.
The Speaker sub-sheet mixes L+R into a PAM8403 driving a CVS-2308 speaker.

Libraries: fix the mirrored SOT-23 land pattern, replace the SOIC-8 land
pattern with the standard 4.95 mm span, add PAM8403D, LM358 and CVS-2308,
and rename the MS9288A footprint to QFN-48 6x6 to match its package.
Parts:
- renumbered C6 to C10, C7 to C11, C8 to C12, C5 to C9, U4 to U5
Changed lines of the file:
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@@
 		(dnp no)
 		(fields_autoplaced yes)
-		(property "Reference" "#PWR034"
+		(property "Reference" "#PWR039"
 			(at 176.53 109.22 0)
 			(hide yes)
@@
 			(project "dino_z80"
 				(path "/8c0b3d8b-46d3-4173-ab1e-a61765f77d61/fc69669c-5428-4356-8e92-0aa932a39979/8c675c61-7675-483d-9014-57cd80e2c617"
-					(reference "#PWR034")
+					(reference "#PWR039")
 					(unit 1)
 				)
@@
 		(in_pos_files yes)
 		(dnp no)
-		(property "Reference" "C5"
+		(property "Reference" "C9"
 			(at 174.625 63.5 0)
 			(show_name no)
@@
 			(project "dino_z80"
 				(path "/8c0b3d8b-46d3-4173-ab1e-a61765f77d61/fc69669c-5428-4356-8e92-0aa932a39979/8c675c61-7675-483d-9014-57cd80e2c617"
-					(reference "C5")
+					(reference "C9")
 					(unit 1)
 				)
@@
 		(in_pos_files yes)
 		(dnp no)
-		(property "Reference" "C7"
+		(property "Reference" "C11"
 			(at 182.245 63.5 0)
 			(show_name no)
@@
 			(project "dino_z80"
 				(path "/8c0b3d8b-46d3-4173-ab1e-a61765f77d61/fc69669c-5428-4356-8e92-0aa932a39979/8c675c61-7675-483d-9014-57cd80e2c617"
-					(reference "C7")
+					(reference "C11")
 					(unit 1)
 				)
@@
 		(dnp no)
 		(fields_autoplaced yes)
-		(property "Reference" "#PWR035"
+		(property "Reference" "#PWR040"
 			(at 175.26 85.09 0)
 			(hide yes)
@@
 			(project "dino_z80"
 				(path "/8c0b3d8b-46d3-4173-ab1e-a61765f77d61/fc69669c-5428-4356-8e92-0aa932a39979/8c675c61-7675-483d-9014-57cd80e2c617"
-					(reference "#PWR035")
+					(reference "#PWR040")
 					(unit 1)
 				)
@@
 		(dnp no)
 		(fields_autoplaced yes)
-		(property "Reference" "#PWR032"
+		(property "Reference" "#PWR037"
 			(at 170.18 77.47 0)
 			(hide yes)
@@
 			(project "dino_z80"
 				(path "/8c0b3d8b-46d3-4173-ab1e-a61765f77d61/fc69669c-5428-4356-8e92-0aa932a39979/8c675c61-7675-483d-9014-57cd80e2c617"
-					(reference "#PWR032")
+					(reference "#PWR037")
 					(unit 1)
 				)
@@
 		(in_pos_files yes)
 		(dnp no)
-		(property "Reference" "C8"
+		(property "Reference" "C12"
 			(at 186.055 97.79 0)
 			(show_name no)
@@
 			(project "dino_z80"
 				(path "/8c0b3d8b-46d3-4173-ab1e-a61765f77d61/fc69669c-5428-4356-8e92-0aa932a39979/8c675c61-7675-483d-9014-57cd80e2c617"
-					(reference "C8")
+					(reference "C12")
 					(unit 1)
 				)
@@
 		(dnp no)
 		(fields_autoplaced yes)
-		(property "Reference" "#PWR036"
+		(property "Reference" "#PWR041"
 			(at 180.34 64.77 0)
 			(hide yes)
@@
 			(project "dino_z80"
 				(path "/8c0b3d8b-46d3-4173-ab1e-a61765f77d61/fc69669c-5428-4356-8e92-0aa932a39979/8c675c61-7675-483d-9014-57cd80e2c617"
-					(reference "#PWR036")
+					(reference "#PWR041")
 					(unit 1)
 				)
@@
 		(dnp no)
 		(fields_autoplaced yes)
-		(property "Reference" "#PWR037"
+		(property "Reference" "#PWR042"
 			(at 184.15 99.06 0)
 			(hide yes)
@@
 			(project "dino_z80"
 				(path "/8c0b3d8b-46d3-4173-ab1e-a61765f77d61/fc69669c-5428-4356-8e92-0aa932a39979/8c675c61-7675-483d-9014-57cd80e2c617"
-					(reference "#PWR037")
+					(reference "#PWR042")
 					(unit 1)
 				)
@@
 		(dnp no)
 		(fields_autoplaced yes)
-		(property "Reference" "#PWR033"
+		(property "Reference" "#PWR038"
 			(at 172.72 64.77 0)
 			(hide yes)
@@
 			(project "dino_z80"
 				(path "/8c0b3d8b-46d3-4173-ab1e-a61765f77d61/fc69669c-5428-4356-8e92-0aa932a39979/8c675c61-7675-483d-9014-57cd80e2c617"
-					(reference "#PWR033")
+					(reference "#PWR038")
 					(unit 1)
 				)
@@
 		(in_pos_files yes)
 		(dnp no)
-		(property "Reference" "C6"
+		(property "Reference" "C10"
 			(at 179.578 99.314 90)
 			(show_name no)
@@
 			(project "dino_z80"
 				(path "/8c0b3d8b-46d3-4173-ab1e-a61765f77d61/fc69669c-5428-4356-8e92-0aa932a39979/8c675c61-7675-483d-9014-57cd80e2c617"
-					(reference "C6")
+					(reference "C10")
 					(unit 1)
 				)
@@
 		(dnp no)
 		(fields_autoplaced yes)
-		(property "Reference" "U4"
+		(property "Reference" "U5"
 			(at 134.62 67.31 0)
 			(show_name no)
@@
 			(project "dino_z80"
 				(path "/8c0b3d8b-46d3-4173-ab1e-a61765f77d61/fc69669c-5428-4356-8e92-0aa932a39979/8c675c61-7675-483d-9014-57cd80e2c617"
-					(reference "U4")
-					(unit 1)
-				)
+					(reference "U5")
+					(unit 1)
+				)

Commit message: chore: dino_z80 standard values, Y2 for the oscillator, datasheet links checked
- Values in SI form: 10kΩ, 200Ω, 100nF, 10µF, 3.3µH, 220Ω@100MHz beads,
  12MHz / 24.576MHz clocks. Schematic and board agree.
- X1 (12 MHz oscillator) renamed Y2, crystals and oscillators both Y.
- Links: Y2 datasheet is the ASE series (was ASV, a 7x5 part); S1/S5 and
  S3/S4 point at the Littelfuse C&K datasheets (KMR2 link was dead);
  J4 gets the JST SH datasheet instead of 2.54 mm header links; D5 gets
  the listing that has 1N5819WS; the Vishay datasheet on R1/R2/R35/R36/
  R41/R42 moves from AliExpress to Datasheet; Y1 loses the LCSC record of
  a 12 MHz 3225 crystal; datasheets added for U1, U4, U7, D3.
- LS1 and U11 descriptions tidied.

DRC: 0 errors, 0 unconnected, 0 schematic parity. ERC: 0.
Parts:
- C10: value 4.7u -> 4.7µF
- C11, C12: value 100n -> 100nF
- C9: value 1u -> 1µF
Changed lines of the file:
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@@
 			)
 		)
-		(property "Value" "1u"
+		(property "Value" "1µF"
 			(at 174.625 66.04 0)
 			(show_name no)
@@
 			)
 		)
-		(property "Value" "100n"
+		(property "Value" "100nF"
 			(at 182.245 66.04 0)
 			(show_name no)
@@
 			)
 		)
-		(property "Value" "100n"
+		(property "Value" "100nF"
 			(at 186.055 100.33 0)
 			(show_name no)
@@
 			)
 		)
-		(property "Value" "4.7u"
+		(property "Value" "4.7µF"
 			(at 173.736 99.314 90)
 			(show_name no)
